Commit message: modify link params

File: aero_description/aero_four_legs/models/gen/aero_upper.urdf (robot description, URDF)
Before this commit: robot AeroUpperRobot, 29 links, 28 joints
Joints:
- joint LARM_INDEX_P1: origin xyz=-0.00825 0.001 -0.1363 rpy=0 -0 0  -> xyz=0 0.001 -0.1363 rpy=0 -0 0 
- joint LARM_SHOULDER_P: origin xyz=-0.02 0.134 0.3049 rpy=0 -0 0  -> xyz=-0.02 0.1342 0.3049 rpy=0 -0 0 
- joint LARM_THUMB_P: origin xyz=-0.00825 -0.0344 -0.1 rpy=0 -0 0  -> xyz=0 -0.0344 -0.1 rpy=0 -0 0 
- joint RARM_INDEX_P1: origin xyz=-0.00825 -0.001 -0.1358 rpy=0 -0 0  -> xyz=0 -0.001 -0.1358 rpy=0 -0 0 
- joint RARM_THUMB_P: origin xyz=-0.00825 0.0344 -0.1 rpy=0 -0 0  -> xyz=0 0.0344 -0.1 rpy=0 -0 0 
