Commit message: fixed urdfs

File: aero_description/aero_four_legs/models/urdf/aero_upper.urdf (robot description, URDF)
Before this commit: robot AeroUpperRobot, 29 links, 28 joints
Joints:
- joint LARM_ELBOW: origin xyz=0 0 -0.17 rpy=0 -0 0  -> xyz=0.014 0 -0.171 rpy=0 -0 0 
- joint LARM_INDEX_P1: origin xyz=0 0.013 -0.1363 rpy=0 -0 0  -> xyz=0 0.001 -0.1363 rpy=0 -0 0 
- joint LARM_SHOULDER_P: origin xyz=-0.02 0.134 0.31 rpy=0 -0 0  -> xyz=-0.02 0.1342 0.3049 rpy=0 -0 0 
- joint LARM_SHOULDER_R: origin xyz=0 0.055 0.002 rpy=0 -0 0  -> xyz=0 0.0549 0.0023 rpy=0 -0 0 
- joint LARM_SHOULDER_Y: origin xyz=0 -0.012 -0.123 rpy=0 -0 0  -> xyz=0 -0.012 -0.1255 rpy=0 -0 0 
- joint LARM_THUMB_P: origin xyz=0 -0.0224 -0.1 rpy=0 -0 0  -> xyz=0 -0.0344 -0.1 rpy=0 -0 0 
- joint LARM_WRIST_P: origin xyz=0 0 -0.137 rpy=0 -0 0  -> xyz=0 0 -0.1337 rpy=0 -0 0 
- joint LARM_WRIST_Y: origin xyz=0 0 -0.121 rpy=0 -0 0  -> xyz=-0.014 0 -0.1235 rpy=0 -0 0 
- joint NECK_P: origin xyz=0.015 0 0.1025 rpy=0 -0 0  -> xyz=0 0 0.105 rpy=0 -0 0 
- joint NECK_Y: origin xyz=0 0 0.3585 rpy=0 -0 0  -> xyz=0 0 0.351 rpy=0 -0 0 
- joint RARM_ELBOW: origin xyz=0 0 -0.17 rpy=0 -0 0  -> xyz=0.014 0 -0.171 rpy=0 -0 0 
- joint RARM_INDEX_P1: origin xyz=0 -0.013 -0.1358 rpy=0 -0 0  -> xyz=0 -0.001 -0.1358 rpy=0 -0 0 
- joint RARM_SHOULDER_P: origin xyz=-0.02 -0.134 0.312 rpy=0 -0 0  -> xyz=-0.02 -0.134 0.3049 rpy=0 -0 0 
- joint RARM_SHOULDER_R: origin xyz=0 -0.055 0.002 rpy=0 -0 0  -> xyz=0 -0.0549 0.0023 rpy=0 -0 0 
- joint RARM_SHOULDER_Y: origin xyz=0 0.012 -0.123 rpy=0 -0 0  -> xyz=0 0.012 -0.1255 rpy=0 -0 0 
- joint RARM_THUMB_P: origin xyz=0 0.0224 -0.1 rpy=0 -0 0  -> xyz=0 0.0344 -0.1 rpy=0 -0 0 
- joint RARM_WRIST_P: origin xyz=0 0 -0.137 rpy=0 -0 0  -> xyz=0 0 -0.1337 rpy=0 -0 0 
- joint RARM_WRIST_Y: origin xyz=0 0 -0.121 rpy=0 -0 0  -> xyz=-0.014 0 -0.1235 rpy=0 -0 0 
- joint WAIST_P: origin xyz=0 0 0.11 rpy=0 -0 0  -> xyz=0 0 0.1367 rpy=0 -0 0 
- joint WAIST_Y: origin xyz=0.01175 0 0.0347 rpy=0 -0 0  -> xyz=0 0 0.0103 rpy=0 -0 0 
