Commit message: 1.5708 > M_PI/2.0, so max limit was over 90 degrees

File: aero_description/typeF/models/urdf/aero_upper.urdf (robot description, URDF)
Before this commit: robot AeroUpperRobot, 29 links, 28 joints
Joints:
- joint LARM_SHOULDER_P: limit lower=-1.5708 upper=0 effort=100 velocity=0.5 -> lower=-1.5707 upper=0 effort=100 velocity=0.5
- joint LARM_SHOULDER_R: limit lower=0 upper=1.5708 effort=100 velocity=0.5 -> lower=0 upper=1.5707 effort=100 velocity=0.5
- joint RARM_SHOULDER_P: limit lower=-1.5708 upper=0 effort=100 velocity=0.5 -> lower=-1.5707 upper=0 effort=100 velocity=0.5
- joint RARM_SHOULDER_R: limit lower=-1.5708 upper=0 effort=100 velocity=0.5 -> lower=-1.5707 upper=0 effort=100 velocity=0.5
- joint WAIST_P: limit lower=0 upper=1.5708 effort=100 velocity=0.5 -> lower=0 upper=1.5707 effort=100 velocity=0.5
