Commit message: new setup script with xacro

File: aero_description/typeF/urdf/aero-wheels/lifter.urdf.xacro (robot description, xacro)
@@ -21,5 +21,5 @@
         <origin xyz="0 0 0" rpy="0 -0 0"/>
         <geometry>
-          <mesh filename="package://aero_description/models/aero-lower_meshes/WAIST_LINK1_mesh.dae" scale="1 1 1" />
+          <mesh filename="package://aero_description/meshes/aero-lower_meshes/WAIST_LINK1_mesh.dae" scale="1 1 1" />
         </geometry>
       </visual>
@@ -27,5 +27,5 @@
         <origin xyz="0 0 0" rpy="0 -0 0"/>
         <geometry>
-          <mesh filename="package://aero_description/models/aero-lower_meshes/WAIST_LINK1_mesh.dae" scale="1 1 1" />
+          <mesh filename="package://aero_description/meshes/aero-lower_meshes/WAIST_LINK1_mesh.dae" scale="1 1 1" />
         </geometry>
       </collision>
@@ -44,5 +44,5 @@
         <origin xyz="0.0 0.0 0.29009" rpy="0 -0 0"/>
         <geometry>
-          <mesh filename="package://aero_description/models/aero-lower_meshes/wheel_upper_mesh.dae" scale="1 1 1" />
+          <mesh filename="package://aero_description/meshes/aero-lower_meshes/wheel_upper_mesh.dae" scale="1 1 1" />
         </geometry>
       </visual>
@@ -50,5 +50,5 @@
         <origin xyz="0.0 0.0 0.0" rpy="0 -0 0"/>
         <geometry>
-          <mesh filename="package://aero_description/models/aero-lower_meshes/wheel_upper_mesh.dae" scale="1 1 1" />
+          <mesh filename="package://aero_description/meshes/aero-lower_meshes/wheel_upper_mesh.dae" scale="1 1 1" />
         </geometry>
       </collision>
@@ -67,5 +67,5 @@
         <origin xyz="0.0 0.0 0.29009" rpy="0 -0 0"/>
         <geometry>
-          <mesh filename="package://aero_description/models/aero-lower_meshes/wheel_lower_mesh.dae" scale="1 1 1" />
+          <mesh filename="package://aero_description/meshes/aero-lower_meshes/wheel_lower_mesh.dae" scale="1 1 1" />
         </geometry>
       </visual>
@@ -73,5 +73,5 @@
         <origin xyz="0.0 0.0 0.0" rpy="0 -0 0"/>
         <geometry>
-          <mesh filename="package://aero_description/models/aero-lower_meshes/wheel_lower_mesh.dae" scale="1 1 1" />
+          <mesh filename="package://aero_description/meshes/aero-lower_meshes/wheel_lower_mesh.dae" scale="1 1 1" />
         </geometry>
       </collision>

File: aero_description/typeF/urdf/aero-wheels/wheels.urdf.xacro (robot description, xacro)
@@ -21,5 +21,5 @@
         <origin xyz="0.0 0.0 0.0" rpy="0 -0 0"/>
         <geometry>
-          <mesh filename="package://aero_description/models/aero-lower_meshes/wheels_base.dae" scale="1 1 1" />
+          <mesh filename="package://aero_description/meshes/aero-lower_meshes/wheels_base.dae" scale="1 1 1" />
         </geometry>
       </visual>
@@ -27,5 +27,5 @@
         <origin xyz="0.0 0.0 0.0" rpy="0 -0 0"/>
         <geometry>
-          <mesh filename="package://aero_description/models/aero-lower_meshes/wheels_base.dae" scale="1 1 1" />
+          <mesh filename="package://aero_description/meshes/aero-lower_meshes/wheels_base.dae" scale="1 1 1" />
         </geometry>
       </collision>

File: aero_description/typeF/urdf/aero_upper/aero_upper.urdf.xacro (robot description, xacro)
@@ -14,11 +14,11 @@
       <origin xyz="0 0 0" rpy="0 -0 0"/>
       <geometry>
-        <mesh filename="package://aero_description/models/aero_upper_meshes/WAIST_LINK0_mesh.dae" scale="1 1 1" />
-      </geometry>
-    </visual>
-    <collision>
-      <origin xyz="0 0 0" rpy="0 -0 0"/>
-      <geometry>
-        <mesh filename="package://aero_description/models/aero_upper_meshes/WAIST_LINK0_mesh.dae" scale="1 1 1" />
+        <mesh filename="package://aero_description/meshes/aero_upper_meshes/WAIST_LINK0_mesh.dae" scale="1 1 1" />
+      </geometry>
+    </visual>
+    <collision>
+      <origin xyz="0 0 0" rpy="0 -0 0"/>
+      <geometry>
+        <mesh filename="package://aero_description/meshes/aero_upper_meshes/WAIST_LINK0_mesh.dae" scale="1 1 1" />
       </geometry>
     </collision>
@@ -37,11 +37,11 @@
       <origin xyz="0 0 0" rpy="0 -0 0"/>
       <geometry>
-        <mesh filename="package://aero_description/models/aero_upper_meshes/WAIST_LINK1_mesh.dae" scale="1 1 1" />
-      </geometry>
-    </visual>
-    <collision>
-      <origin xyz="0 0 0" rpy="0 -0 0"/>
-      <geometry>
-        <mesh filename="package://aero_description/models/aero_upper_meshes/WAIST_LINK1_mesh.dae" scale="1 1 1" />
+        <mesh filename="package://aero_description/meshes/aero_upper_meshes/WAIST_LINK1_mesh.dae" scale="1 1 1" />
+      </geometry>
+    </visual>
+    <collision>
+      <origin xyz="0 0 0" rpy="0 -0 0"/>
+      <geometry>
+        <mesh filename="package://aero_description/meshes/aero_upper_meshes/WAIST_LINK1_mesh.dae" scale="1 1 1" />
       </geometry>
     </collision>
@@ -71,11 +71,11 @@
       <origin xyz="0 0 0" rpy="0 -0 0"/>
       <geometry>
-        <mesh filename="package://aero_description/models/aero_upper_meshes/WAIST_LINK3_mesh.dae" scale="1 1 1" />
-      </geometry>
-    </visual>
-    <collision>
-      <origin xyz="0 0 0" rpy="0 -0 0"/>
-      <geometry>
-        <mesh filename="package://aero_description/models/aero_upper_meshes/WAIST_LINK3_mesh.dae" scale="1 1 1" />
+        <mesh filename="package://aero_description/meshes/aero_upper_meshes/WAIST_LINK3_mesh.dae" scale="1 1 1" />
+      </geometry>
+    </visual>
+    <collision>
+      <origin xyz="0 0 0" rpy="0 -0 0"/>
+      <geometry>
+        <mesh filename="package://aero_description/meshes/aero_upper_meshes/WAIST_LINK3_mesh.dae" scale="1 1 1" />
       </geometry>
     </collision>
@@ -94,5 +94,5 @@
       <origin xyz="0 0 0" rpy="-0.174532925 -0 0"/>
       <geometry>
-        <mesh filename="package://aero_description/models/aero_upper_meshes/LARM_LINK1_mesh.dae" scale="1 1 1" />
+        <mesh filename="package://aero_description/meshes/aero_upper_meshes/LARM_LINK1_mesh.dae" scale="1 1 1" />
       </geometry>
     </visual>
@@ -100,5 +100,5 @@
       <origin xyz="0 0 0" rpy="-0.174532925 -0 0"/>
       <geometry>
-        <mesh filename="package://aero_description/models/aero_upper_meshes/LARM_LINK1_mesh.dae" scale="1 1 1" />
+        <mesh filename="package://aero_description/meshes/aero_upper_meshes/LARM_LINK1_mesh.dae" scale="1 1 1" />
       </geometry>
     </collision>
@@ -117,11 +117,11 @@
       <origin xyz="0 0 0" rpy="0 -0 0"/>
       <geometry>
-        <mesh filename="package://aero_description/models/aero_upper_meshes/LARM_LINK2_mesh.dae" scale="1 1 1" />
-      </geometry>
-    </visual>
-    <collision>
-      <origin xyz="0 0 0" rpy="0 -0 0"/>
-      <geometry>
-        <mesh filename="package://aero_description/models/aero_upper_meshes/LARM_LINK2_mesh.dae" scale="1 1 1" />
+        <mesh filename="package://aero_description/meshes/aero_upper_meshes/LARM_LINK2_mesh.dae" scale="1 1 1" />
+      </geometry>
+    </visual>
+    <collision>
+      <origin xyz="0 0 0" rpy="0 -0 0"/>
+      <geometry>
+        <mesh filename="package://aero_description/meshes/aero_upper_meshes/LARM_LINK2_mesh.dae" scale="1 1 1" />
       </geometry>
     </collision>
@@ -140,11 +140,11 @@
       <origin xyz="0 0 0" rpy="0 -0 0"/>
       <geometry>
-        <mesh filename="package://aero_description/models/aero_upper_meshes/LARM_LINK3_mesh.dae" scale="1 1 1" />
-      </geometry>
-    </visual>
-    <collision>
-      <origin xyz="0 0 0" rpy="0 -0 0"/>
-      <geometry>
-        <mesh filename="package://aero_description/models/aero_upper_meshes/LARM_LINK3_mesh.dae" scale="1 1 1" />
+        <mesh filename="package://aero_description/meshes/aero_upper_meshes/LARM_LINK3_mesh.dae" scale="1 1 1" />
+      </geometry>
+    </visual>
+    <collision>
+      <origin xyz="0 0 0" rpy="0 -0 0"/>
+      <geometry>
+        <mesh filename="package://aero_description/meshes/aero_upper_meshes/LARM_LINK3_mesh.dae" scale="1 1 1" />
       </geometry>
     </collision>
@@ -163,5 +163,5 @@
       <origin xyz="-0.035 0 -0.035" rpy="0 -0 0"/>
       <geometry>
-        <mesh filename="package://aero_description/models/aero_upper_meshes/LARM_LINK4_mesh.dae" scale="1 1 1" />
+        <mesh filename="package://aero_description/meshes/aero_upper_meshes/LARM_LINK4_mesh.dae" scale="1 1 1" />
       </geometry>
     </visual>
@@ -169,5 +169,5 @@
       <origin xyz="-0.035 0 -0.035" rpy="0 -0 0"/>
       <geometry>
-        <mesh filename="package://aero_description/models/aero_upper_meshes/LARM_LINK4_mesh.dae" scale="1 1 1" />
+        <mesh filename="package://aero_description/meshes/aero_upper_meshes/LARM_LINK4_mesh.dae" scale="1 1 1" />
       </geometry>
     </collision>
@@ -186,11 +186,11 @@
       <origin xyz="0 0 0" rpy="0 -0 0"/>
       <geometry>
-        <mesh filename="package://aero_description/models/aero_upper_meshes/LARM_LINK5_mesh.dae" scale="1 1 1" />
-      </geometry>
-    </visual>
-    <collision>
-      <origin xyz="0 0 0" rpy="0 -0 0"/>
-      <geometry>
-        <mesh filename="package://aero_description/models/aero_upper_meshes/LARM_LINK5_mesh.dae" scale="1 1 1" />
+        <mesh filename="package://aero_description/meshes/aero_upper_meshes/LARM_LINK5_mesh.dae" scale="1 1 1" />
+      </geometry>
+    </visual>
+    <collision>
+      <origin xyz="0 0 0" rpy="0 -0 0"/>
+      <geometry>
+        <mesh filename="package://aero_description/meshes/aero_upper_meshes/LARM_LINK5_mesh.dae" scale="1 1 1" />
       </geometry>
     </collision>
@@ -220,11 +220,11 @@
       <origin xyz="0 0 0" rpy="0 -0 0"/>
       <geometry>
-        <mesh filename="package://aero_description/models/aero_upper_meshes/LARM_LINK7_mesh.dae" scale="1 1 1" />
-      </geometry>
-    </visual>
-    <collision>
-      <origin xyz="0 0 0" rpy="0 -0 0"/>
-      <geometry>
-        <mesh filename="package://aero_description/models/aero_upper_meshes/LARM_LINK7_mesh.dae" scale="1 1 1" />
+        <mesh filename="package://aero_description/meshes/aero_upper_meshes/LARM_LINK7_mesh.dae" scale="1 1 1" />
+      </geometry>
+    </visual>
+    <collision>
+      <origin xyz="0 0 0" rpy="0 -0 0"/>
+      <geometry>
+        <mesh filename="package://aero_description/meshes/aero_upper_meshes/LARM_LINK7_mesh.dae" scale="1 1 1" />
       </geometry>
     </collision>
@@ -243,5 +243,5 @@
       <origin xyz="0 -0.013 0.115" rpy="0 -0 0 "/>
       <geometry>
-        <mesh filename="package://aero_description/models/aero_upper_meshes/LARM_INDEX_LINK1_mesh.dae" scale="1 1 1" />
+        <mesh filename="package://aero_description/meshes/aero_upper_meshes/LARM_INDEX_LINK1_mesh.dae" scale="1 1 1" />
       </geometry>
     </visual>
@@ -249,5 +249,5 @@
       <origin xyz="0 -0.013 0.115" rpy="0 -0 0 "/>
       <geometry>
-        <mesh filename="package://aero_description/models/aero_upper_meshes/LARM_INDEX_LINK1_mesh.dae" scale="1 1 1" />
+        <mesh filename="package://aero_description/meshes/aero_upper_meshes/LARM_INDEX_LINK1_mesh.dae" scale="1 1 1" />
       </geometry>
     </collision>
@@ -266,5 +266,5 @@
       <origin xyz="0 0.015754 0.149615" rpy="0 -0 0"/>
       <geometry>
-        <mesh filename="package://aero_description/models/aero_upper_meshes/LARM_INDEX_LINK2_mesh.dae" scale="1 1 1" />
+        <mesh filename="package://aero_description/meshes/aero_upper_meshes/LARM_INDEX_LINK2_mesh.dae" scale="1 1 1" />
       </geometry>
     </visual>
@@ -272,5 +272,5 @@
       <origin xyz="0 0.015754 0.149615" rpy="0 -0 0"/>
       <geometry>
-        <mesh filename="package://aero_description/models/aero_upper_meshes/LARM_INDEX_LINK2_mesh.dae" scale="1 1 1" />
+        <mesh filename="package://aero_description/meshes/aero_upper_meshes/LARM_INDEX_LINK2_mesh.dae" scale="1 1 1" />
       </geometry>
     </collision>
@@ -289,5 +289,5 @@
       <origin xyz="0 0.03747 0.162972" rpy="0 -0 0"/>
       <geometry>
-        <mesh filename="package://aero_description/models/aero_upper_meshes/LARM_INDEX_LINK3_mesh.dae" scale="1 1 1" />
+        <mesh filename="package://aero_description/meshes/aero_upper_meshes/LARM_INDEX_LINK3_mesh.dae" scale="1 1 1" />
       </geometry>
     </visual>
@@ -295,5 +295,5 @@
       <origin xyz="0 0.03747 0.162972" rpy="0 -0 0"/>
       <geometry>
-        <mesh filename="package://aero_description/models/aero_upper_meshes/LARM_INDEX_LINK3_mesh.dae" scale="1 1 1" />
+        <mesh filename="package://aero_description/meshes/aero_upper_meshes/LARM_INDEX_LINK3_mesh.dae" scale="1 1 1" />
       </geometry>
     </collision>
@@ -312,5 +312,5 @@
       <origin xyz="0 0.022355 0.079645" rpy="0 -0 0 "/>
       <geometry>
-        <mesh filename="package://aero_description/models/aero_upper_meshes/LARM_THUMB_LINK_mesh.dae" scale="1 1 1" />
+        <mesh filename="package://aero_description/meshes/aero_upper_meshes/LARM_THUMB_LINK_mesh.dae" scale="1 1 1" />
       </geometry>
     </visual>
@@ -318,5 +318,5 @@
       <origin xyz="0 0.022355 0.079645" rpy="0 -0 0 "/>
       <geometry>
-        <mesh filename="package://aero_description/models/aero_upper_meshes/LARM_THUMB_LINK_mesh.dae" scale="1 1 1" />
+        <mesh filename="package://aero_description/meshes/aero_upper_meshes/LARM_THUMB_LINK_mesh.dae" scale="1 1 1" />
       </geometry>
     </collision>
@@ -335,11 +335,11 @@
       <origin xyz="0 0 0" rpy="0 -0 0"/>
       <geometry>
-        <mesh filename="package://aero_description/models/aero_upper_meshes/NECK_LINK1_mesh.dae" scale="1 1 1" />
-      </geometry>
-    </visual>
-    <collision>
-      <origin xyz="0 0 0" rpy="0 -0 0"/>
-      <geometry>
-        <mesh filename="package://aero_description/models/aero_upper_meshes/NECK_LINK1_mesh.dae" scale="1 1 1" />
+        <mesh filename="package://aero_description/meshes/aero_upper_meshes/NECK_LINK1_mesh.dae" scale="1 1 1" />
+      </geometry>
+    </visual>
+    <collision>
+      <origin xyz="0 0 0" rpy="0 -0 0"/>
+      <geometry>
+        <mesh filename="package://aero_description/meshes/aero_upper_meshes/NECK_LINK1_mesh.dae" scale="1 1 1" />
       </geometry>
     </collision>
@@ -358,11 +358,11 @@
       <origin xyz="0 0 0" rpy="0 -0 0"/>
       <geometry>
-        <mesh filename="package://aero_description/models/aero_upper_meshes/NECK_LINK2_mesh.dae" scale="1 1 1" />
-      </geometry>
-    </visual>
-    <collision>
-      <origin xyz="0 0 0" rpy="0 -0 0"/>
-      <geometry>
-        <mesh filename="package://aero_description/models/aero_upper_meshes/NECK_LINK2_mesh.dae" scale="1 1 1" />
+        <mesh filename="package://aero_description/meshes/aero_upper_meshes/NECK_LINK2_mesh.dae" scale="1 1 1" />
+      </geometry>
+    </visual>
+    <collision>
+      <origin xyz="0 0 0" rpy="0 -0 0"/>
+      <geometry>
+        <mesh filename="package://aero_description/meshes/aero_upper_meshes/NECK_LINK2_mesh.dae" scale="1 1 1" />
       </geometry>
     </collision>
@@ -381,11 +381,11 @@
       <origin xyz="0 0 0" rpy="0 -0 0"/>
       <geometry>
-        <mesh filename="package://aero_description/models/aero_upper_meshes/NECK_LINK3_mesh.dae" scale="1 1 1" />
-      </geometry>
-    </visual>
-    <collision>
-      <origin xyz="0 0 0" rpy="0 -0 0"/>
-      <geometry>
-        <mesh filename="package://aero_description/models/aero_upper_meshes/NECK_LINK3_mesh.dae" scale="1 1 1" />
+        <mesh filename="package://aero_description/meshes/aero_upper_meshes/NECK_LINK3_mesh.dae" scale="1 1 1" />
+      </geometry>
+    </visual>
+    <collision>
+      <origin xyz="0 0 0" rpy="0 -0 0"/>
+      <geometry>
+        <mesh filename="package://aero_description/meshes/aero_upper_meshes/NECK_LINK3_mesh.dae" scale="1 1 1" />
       </geometry>
     </collision>
@@ -404,11 +404,11 @@
       <origin xyz="0 0 0" rpy="0.174532925 -0 0"/>
       <geometry>
-        <mesh filename="package://aero_description/models/aero_upper_meshes/RARM_LINK1_mesh.dae" scale="1 1 1" />
-      </geometry>
-    </visual>
-    <collision>
-      <origin xyz="0 0 0" rpy="0 -0 0"/>
-      <geometry>
-        <mesh filename="package://aero_description/models/aero_upper_meshes/RARM_LINK1_mesh.dae" scale="1 1 1" />
+        <mesh filename="package://aero_description/meshes/aero_upper_meshes/RARM_LINK1_mesh.dae" scale="1 1 1" />
+      </geometry>
+    </visual>
+    <collision>
+      <origin xyz="0 0 0" rpy="0 -0 0"/>
+      <geometry>
+        <mesh filename="package://aero_description/meshes/aero_upper_meshes/RARM_LINK1_mesh.dae" scale="1 1 1" />
       </geometry>
     </collision>
@@ -427,11 +427,11 @@
       <origin xyz="0 0 0" rpy="0 -0 0"/>
       <geometry>
-        <mesh filename="package://aero_description/models/aero_upper_meshes/RARM_LINK2_mesh.dae" scale="1 1 1" />
-      </geometry>
-    </visual>
-    <collision>
-      <origin xyz="0 0 0" rpy="0 -0 0"/>
-      <geometry>
-        <mesh filename="package://aero_description/models/aero_upper_meshes/RARM_LINK2_mesh.dae" scale="1 1 1" />
+        <mesh filename="package://aero_description/meshes/aero_upper_meshes/RARM_LINK2_mesh.dae" scale="1 1 1" />
+      </geometry>
+    </visual>
+    <collision>
+      <origin xyz="0 0 0" rpy="0 -0 0"/>
+      <geometry>
+        <mesh filename="package://aero_description/meshes/aero_upper_meshes/RARM_LINK2_mesh.dae" scale="1 1 1" />
       </geometry>
     </collision>
@@ -450,11 +450,11 @@
       <origin xyz="0 0 0" rpy="0 -0 0"/>
       <geometry>
-        <mesh filename="package://aero_description/models/aero_upper_meshes/RARM_LINK3_mesh.dae" scale="1 1 1" />
-      </geometry>
-    </visual>
-    <collision>
-      <origin xyz="0 0 0" rpy="0 -0 0"/>
-      <geometry>
-        <mesh filename="package://aero_description/models/aero_upper_meshes/RARM_LINK3_mesh.dae" scale="1 1 1" />
+        <mesh filename="package://aero_description/meshes/aero_upper_meshes/RARM_LINK3_mesh.dae" scale="1 1 1" />
+      </geometry>
+    </visual>
+    <collision>
+      <origin xyz="0 0 0" rpy="0 -0 0"/>
+      <geometry>
+        <mesh filename="package://aero_description/meshes/aero_upper_meshes/RARM_LINK3_mesh.dae" scale="1 1 1" />
       </geometry>
     </collision>
@@ -473,5 +473,5 @@
       <origin xyz="-0.035 0 -0.035" rpy="0 -0 0"/>
       <geometry>
-        <mesh filename="package://aero_description/models/aero_upper_meshes/RARM_LINK4_mesh.dae" scale="1 1 1" />
+        <mesh filename="package://aero_description/meshes/aero_upper_meshes/RARM_LINK4_mesh.dae" scale="1 1 1" />
       </geometry>
     </visual>
@@ -479,5 +479,5 @@
       <origin xyz="-0.035 0 -0.070" rpy="0 -0 0"/>
       <geometry>
-        <mesh filename="package://aero_description/models/aero_upper_meshes/RARM_LINK4_mesh.dae" scale="1 1 1" />
+        <mesh filename="package://aero_description/meshes/aero_upper_meshes/RARM_LINK4_mesh.dae" scale="1 1 1" />
       </geometry>
     </collision>
@@ -496,11 +496,11 @@
       <origin xyz="0 0 0" rpy="0 -0 0"/>
       <geometry>
-        <mesh filename="package://aero_description/models/aero_upper_meshes/RARM_LINK5_mesh.dae" scale="1 1 1" />
-      </geometry>
-    </visual>
-    <collision>
-      <origin xyz="0 0 0" rpy="0 -0 0"/>
-      <geometry>
-        <mesh filename="package://aero_description/models/aero_upper_meshes/RARM_LINK5_mesh.dae" scale="1 1 1" />
+        <mesh filename="package://aero_description/meshes/aero_upper_meshes/RARM_LINK5_mesh.dae" scale="1 1 1" />
+      </geometry>
+    </visual>
+    <collision>
+      <origin xyz="0 0 0" rpy="0 -0 0"/>
+      <geometry>
+        <mesh filename="package://aero_description/meshes/aero_upper_meshes/RARM_LINK5_mesh.dae" scale="1 1 1" />
       </geometry>
     </collision>
@@ -530,11 +530,11 @@
       <origin xyz="0 0 0" rpy="0 -0 0"/>
       <geometry>
-        <mesh filename="package://aero_description/models/aero_upper_meshes/RARM_LINK7_mesh.dae" scale="1 1 1" />
-      </geometry>
-    </visual>
-    <collision>
-      <origin xyz="0 0 0" rpy="0 -0 0"/>
-      <geometry>
-        <mesh filename="package://aero_description/models/aero_upper_meshes/RARM_LINK7_mesh.dae" scale="1 1 1" />
+        <mesh filename="package://aero_description/meshes/aero_upper_meshes/RARM_LINK7_mesh.dae" scale="1 1 1" />
+      </geometry>
+    </visual>
+    <collision>
+      <origin xyz="0 0 0" rpy="0 -0 0"/>
+      <geometry>
+        <mesh filename="package://aero_description/meshes/aero_upper_meshes/RARM_LINK7_mesh.dae" scale="1 1 1" />
       </geometry>
     </collision>
@@ -553,5 +553,5 @@
       <origin xyz="0 0.013 0.115" rpy="0 -0 0 "/>
       <geometry>
-        <mesh filename="package://aero_description/models/aero_upper_meshes/RARM_INDEX_LINK1_mesh.dae" scale="1 1 1" />
+        <mesh filename="package://aero_description/meshes/aero_upper_meshes/RARM_INDEX_LINK1_mesh.dae" scale="1 1 1" />
       </geometry>
     </visual>
@@ -559,5 +559,5 @@
       <origin xyz="0 0.013 0.115" rpy="0 -0 0 "/>
       <geometry>
-        <mesh filename="package://aero_description/models/aero_upper_meshes/RARM_INDEX_LINK1_mesh.dae" scale="1 1 1" />
+        <mesh filename="package://aero_description/meshes/aero_upper_meshes/RARM_INDEX_LINK1_mesh.dae" scale="1 1 1" />
       </geometry>
     </collision>
@@ -576,5 +576,5 @@
       <origin xyz="0 -0.015754 0.149615" rpy="0 -0 0"/>
       <geometry>
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