Commit message: remove urdfs from typeF/models

File: aero_description/typeF/urdf/aero-wheels/lifter.urdf.xacro (robot description, xacro)
@@ -110,5 +110,5 @@
     </transmission>
     <gazebo reference="hip_joint">
-      <cfmDamping>0.4</cfmDamping>
+      <implicitSpringDamper>0.4</implicitSpringDamper>
     </gazebo>
     <joint name="knee_joint" type="revolute">
@@ -127,5 +127,5 @@
     </transmission>
     <gazebo reference="knee_joint">
-      <cfmDamping>0.4</cfmDamping>
+      <implicitSpringDamper>0.4</implicitSpringDamper>
     </gazebo>
     <joint name="ankle_joint" type="revolute">
@@ -144,5 +144,5 @@
     </transmission>
     <gazebo reference="hip_joint">
-      <cfmDamping>0.4</cfmDamping>
+      <implicitSpringDamper>0.4</implicitSpringDamper>
     </gazebo>
   </xacro:macro>

File: aero_description/typeF/urdf/aero_upper/aero_upper.urdf.xacro (robot description, xacro)
@@ -24,7 +24,7 @@
     </collision> </xacro:unless>
     <inertial>
-      <mass value="0" />
-      <origin xyz="0 0 0" rpy="0 -0 0"/>
-      <inertia ixx="0" ixy="0" ixz="0" iyy="0" iyz="0" izz="0"/>
+      <mass value="1.257" />
+      <origin xyz="0 0 0.0" rpy="0 -0 0"/>
+      <inertia ixx="0.0034" ixy="0" ixz="0" iyy="0.0036" iyz="0" izz="0.0017"/>
     </inertial>
   </link>
@@ -58,7 +58,7 @@
   <link name="hip_center">
     <inertial>
-      <mass value="0" />
-      <origin xyz="0 0 0" rpy="0 -0 0"/>
-      <inertia ixx="0" ixy="0" ixz="0" iyy="0" iyz="0" izz="0"/>
+      <mass value="0.01" />
+      <origin xyz="0 0 0" rpy="0 -0 0"/>
+      <inertia ixx="0.01" ixy="0" ixz="0" iyy="0.01" iyz="0" izz="0.01"/>
     </inertial>
   </link>
@@ -207,7 +207,7 @@
   <link name="l_wrist_center">
     <inertial>
-      <mass value="0" />
-      <origin xyz="0 0 0" rpy="0 -0 0"/>
-      <inertia ixx="0" ixy="0" ixz="0" iyy="0" iyz="0" izz="0"/>
+      <mass value="0.01" />
+      <origin xyz="0 0 0" rpy="0 -0 0"/>
+      <inertia ixx="0.00001" ixy="0" ixz="0" iyy="0.00001" iyz="0" izz="0.00001"/>
     </inertial>
   </link>
@@ -368,7 +368,7 @@
     </collision> </xacro:unless>
     <inertial>
-      <mass value="0" />
-      <origin xyz="0 0 0" rpy="0 -0 0"/>
-      <inertia ixx="0" ixy="0" ixz="0" iyy="0" iyz="0" izz="0"/>
+      <mass value="0.01" />
+      <origin xyz="0 0 0" rpy="0 -0 0"/>
+      <inertia ixx="0.00001" ixy="0" ixz="0" iyy="0.00001" iyz="0" izz="0.00001"/>
     </inertial>
   </link>
@@ -517,7 +517,7 @@
   <link name="r_wrist_center">
     <inertial>
-      <mass value="0" />
-      <origin xyz="0 0 0" rpy="0 -0 0"/>
-      <inertia ixx="0" ixy="0" ixz="0" iyy="0" iyz="0" izz="0"/>
+      <mass value="0.01" />
+      <origin xyz="0 0 0" rpy="0 -0 0"/>
+      <inertia ixx="0.00001" ixy="0" ixz="0" iyy="0.00001" iyz="0" izz="0.00001"/>
     </inertial>
   </link>
@@ -665,5 +665,5 @@
   </transmission>
   <gazebo reference="waist_y_joint">
-    <cfmDamping>0.4</cfmDamping>
+    <implicitSpringDamper>0.4</implicitSpringDamper>
   </gazebo>
   <joint name="waist_p_joint" type="revolute">
@@ -681,5 +681,5 @@
   </transmission>
   <gazebo reference="waist_p_joint">
-    <cfmDamping>0.4</cfmDamping>
+    <implicitSpringDamper>0.4</implicitSpringDamper>
   </gazebo>
   <joint name="waist_r_joint" type="revolute">
@@ -697,5 +697,5 @@
   </transmission>
   <gazebo reference="waist_r_joint">
-    <cfmDamping>0.4</cfmDamping>
+    <implicitSpringDamper>0.4</implicitSpringDamper>
   </gazebo>
   <joint name="l_shoulder_p_joint" type="revolute">
@@ -713,5 +713,5 @@
   </transmission>
   <gazebo reference="l_shoulder_p_joint">
-    <cfmDamping>0.4</cfmDamping>
+    <implicitSpringDamper>0.4</implicitSpringDamper>
   </gazebo>
   <joint name="l_shoulder_r_joint" type="revolute">
@@ -729,5 +729,5 @@
   </transmission>
   <gazebo reference="l_shoulder_r_joint">
-    <cfmDamping>0.4</cfmDamping>
+    <implicitSpringDamper>0.4</implicitSpringDamper>
   </gazebo>
   <joint name="l_shoulder_y_joint" type="revolute">
@@ -745,5 +745,5 @@
   </transmission>
   <gazebo reference="l_shoulder_y_joint">
-    <cfmDamping>0.4</cfmDamping>
+    <implicitSpringDamper>0.4</implicitSpringDamper>
   </gazebo>
   <joint name="l_elbow_joint" type="revolute">
@@ -761,5 +761,5 @@
   </transmission>
   <gazebo reference="l_elbow_joint">
-    <cfmDamping>0.4</cfmDamping>
+    <implicitSpringDamper>0.4</implicitSpringDamper>
   </gazebo>
   <joint name="l_wrist_y_joint" type="revolute">
@@ -777,5 +777,5 @@
   </transmission>
   <gazebo reference="l_wrist_y_joint">
-    <cfmDamping>0.4</cfmDamping>
+    <implicitSpringDamper>0.4</implicitSpringDamper>
   </gazebo>
   <joint name="l_wrist_p_joint" type="revolute">
@@ -793,5 +793,5 @@
   </transmission>
   <gazebo reference="l_wrist_p_joint">
-    <cfmDamping>0.4</cfmDamping>
+    <implicitSpringDamper>0.4</implicitSpringDamper>
   </gazebo>
   <joint name="l_wrist_r_joint" type="revolute">
@@ -809,5 +809,5 @@
   </transmission>
   <gazebo reference="l_wrist_r_joint">
-    <cfmDamping>0.4</cfmDamping>
+    <implicitSpringDamper>0.4</implicitSpringDamper>
   </gazebo>
   <joint name="l_indexbase_joint" type="revolute">
@@ -820,5 +820,5 @@
   </joint>
   <gazebo reference="l_indexbase_joint">
-    <cfmDamping>0.4</cfmDamping>
+    <implicitSpringDamper>0.4</implicitSpringDamper>
   </gazebo>
   <joint name="l_indexmid_joint" type="revolute">
@@ -831,5 +831,5 @@
   </joint>
   <gazebo reference="l_indexmid_joint">
-    <cfmDamping>0.4</cfmDamping>
+    <implicitSpringDamper>0.4</implicitSpringDamper>
   </gazebo>
   <joint name="l_indexend_joint" type="revolute">
@@ -842,5 +842,5 @@
   </joint>
   <gazebo reference="l_indexend_joint">
-    <cfmDamping>0.4</cfmDamping>
+    <implicitSpringDamper>0.4</implicitSpringDamper>
   </gazebo>
   <joint name="l_thumb_joint" type="revolute">
@@ -858,5 +858,5 @@
   </transmission>
   <gazebo reference="l_thumb_joint">
-    <cfmDamping>0.4</cfmDamping>
+    <implicitSpringDamper>0.4</implicitSpringDamper>
   </gazebo>
   <joint name="neck_y_joint" type="revolute">
@@ -874,5 +874,5 @@
   </transmission>
   <gazebo reference="neck_y_joint">
-    <cfmDamping>0.4</cfmDamping>
+    <implicitSpringDamper>0.4</implicitSpringDamper>
   </gazebo>
   <joint name="neck_p_joint" type="revolute">
@@ -890,5 +890,5 @@
   </transmission>
   <gazebo reference="neck_p_joint">
-    <cfmDamping>0.4</cfmDamping>
+    <implicitSpringDamper>0.4</implicitSpringDamper>
   </gazebo>
   <joint name="neck_r_joint" type="revolute">
@@ -906,5 +906,5 @@
   </transmission>
   <gazebo reference="neck_r_joint">
-    <cfmDamping>0.4</cfmDamping>
+    <implicitSpringDamper>0.4</implicitSpringDamper>
   </gazebo>
   <joint name="r_shoulder_p_joint" type="revolute">
@@ -922,5 +922,5 @@
   </transmission>
   <gazebo reference="r_shoulder_p_joint">
-    <cfmDamping>0.4</cfmDamping>
+    <implicitSpringDamper>0.4</implicitSpringDamper>
   </gazebo>
   <joint name="r_shoulder_r_joint" type="revolute">
@@ -938,5 +938,5 @@
   </transmission>
   <gazebo reference="r_shoulder_r_joint">
-    <cfmDamping>0.4</cfmDamping>
+    <implicitSpringDamper>0.4</implicitSpringDamper>
   </gazebo>
   <joint name="r_shoulder_y_joint" type="revolute">
@@ -954,5 +954,5 @@
   </transmission>
   <gazebo reference="r_shoulder_y_joint">
-    <cfmDamping>0.4</cfmDamping>
+    <implicitSpringDamper>0.4</implicitSpringDamper>
   </gazebo>
   <joint name="r_elbow_joint" type="revolute">
@@ -970,5 +970,5 @@
   </transmission>
   <gazebo reference="r_elbow_joint">
-    <cfmDamping>0.4</cfmDamping>
+    <implicitSpringDamper>0.4</implicitSpringDamper>
   </gazebo>
   <joint name="r_wrist_y_joint" type="revolute">
@@ -986,5 +986,5 @@
   </transmission>
   <gazebo reference="r_wrist_y_joint">
-    <cfmDamping>0.4</cfmDamping>
+    <implicitSpringDamper>0.4</implicitSpringDamper>
   </gazebo>
   <joint name="r_wrist_p_joint" type="revolute">
@@ -1002,5 +1002,5 @@
   </transmission>
   <gazebo reference="r_wrist_p_joint">
-    <cfmDamping>0.4</cfmDamping>
+    <implicitSpringDamper>0.4</implicitSpringDamper>
   </gazebo>
   <joint name="r_wrist_r_joint" type="revolute">
@@ -1018,5 +1018,5 @@
   </transmission>
   <gazebo reference="r_wrist_r_joint">
-    <cfmDamping>0.4</cfmDamping>
+    <implicitSpringDamper>0.4</implicitSpringDamper>
   </gazebo>
   <joint name="r_indexbase_joint" type="revolute">
@@ -1029,5 +1029,5 @@
   </joint>
   <gazebo reference="r_indexbase_joint">
-    <cfmDamping>0.4</cfmDamping>
+    <implicitSpringDamper>0.4</implicitSpringDamper>
   </gazebo>
   <joint name="r_indexmid_joint" type="revolute">
@@ -1040,5 +1040,5 @@
   </joint>
   <gazebo reference="r_indexmid_joint">
-    <cfmDamping>0.4</cfmDamping>
+    <implicitSpringDamper>0.4</implicitSpringDamper>
   </gazebo>
   <joint name="r_indexend_joint" type="revolute">
@@ -1056,5 +1056,5 @@
   </transmission>
   <gazebo reference="r_indexend_joint">
-    <cfmDamping>0.4</cfmDamping>
+    <implicitSpringDamper>0.4</implicitSpringDamper>
   </gazebo>
   <joint name="r_thumb_joint" type="revolute">
@@ -1072,5 +1072,5 @@
   </transmission>
   <gazebo reference="r_thumb_joint">
-    <cfmDamping>0.4</cfmDamping>
+    <implicitSpringDamper>0.4</implicitSpringDamper>
   </gazebo>
   <!-- for ik eef connector-->

Commit message: added pseudo mass in order for gazebo

File: aero_description/typeF/urdf/aero-wheels/lifter.urdf.xacro (robot description, xacro)
@@ -16,10 +16,9 @@
   <xacro:include filename="$(find aero_description)/urdf/common.xacro" />
   <xacro:macro name="lifter" params="base_link">
-    <link name="${base_link}" />
-    <link name="leg_base_link">
-<!--      <visual>
+    <link name="${base_link}">
+      <visual>
         <origin xyz="0 0 0" rpy="0 -0 0"/>
         <geometry>
-          <mesh filename="package://aero_description/meshes/aero-lower_meshes/WAIST_LINK1_mesh.dae" scale="1 1 1" />
+          <mesh filename="package://aero_description/meshes/aero-lower_meshes/lifter_base.dae" scale="1 1 1" />
         </geometry>
       </visual>
@@ -27,5 +26,5 @@
         <origin xyz="0 0 0" rpy="0 -0 0"/>
         <geometry>
-          <mesh filename="package://aero_description/meshes/aero-lower_meshes/WAIST_LINK1_mesh.dae" scale="1 1 1" />
+          <mesh filename="package://aero_description/meshes/aero-lower_meshes/lifter_base.dae" scale="1 1 1" />
         </geometry>
       </collision>
@@ -34,5 +33,28 @@
         <origin xyz="-0.012819 -0.002679 0.007207" rpy="0 -0 0"/>
         <inertia ixx="0.0658136" ixy="-0.000159462" ixz="0.010103" iyy="0.0504268" iyz="0.000173435" izz="0.0889772"/>
-      </inertial> -->
+      </inertial>
+    </link>
+    <gazebo reference="${base_link}">
+      <mu1>0.9</mu1>
+      <mu2>0.9</mu2>
+    </gazebo>
+    <link name="leg_base_link">
+      <visual>
+        <origin xyz="0 0 0" rpy="0 -0 0"/>
+        <geometry>
+          <mesh filename="package://aero_description/meshes/aero-lower_meshes/lifter_top_connector.dae" scale="1 1 1" />
+        </geometry>
+      </visual>
+      <collision>
+        <origin xyz="0 0 0" rpy="0 -0 0"/>
+        <geometry>
+          <mesh filename="package://aero_description/meshes/aero-lower_meshes/lifter_top_connector.dae" scale="1 1 1" />
+        </geometry>
+      </collision>
+      <inertial>
+        <mass value="7.64604" />
+        <origin xyz="-0.012819 -0.002679 0.007207" rpy="0 -0 0"/>
+        <inertia ixx="0.0658136" ixy="-0.000159462" ixz="0.010103" iyy="0.0504268" iyz="0.000173435" izz="0.0889772"/>
+      </inertial>
     </link>
     <gazebo reference="leg_base_link">
@@ -88,5 +110,27 @@
       <mu2>0.9</mu2>
     </gazebo>
-    <link name="lifter_top_link"/>
+    <link name="lifter_top_link">
+      <visual>
+        <origin xyz="0 0 0" rpy="0 -0 0"/>
+        <geometry>
+          <mesh filename="package://aero_description/meshes/aero-lower_meshes/lifter_top.dae" scale="1 1 1" />
+        </geometry>
+      </visual>
+      <collision>
+        <origin xyz="0 0 0" rpy="0 -0 0"/>
+        <geometry>
+          <mesh filename="package://aero_description/meshes/aero-lower_meshes/lifter_top.dae" scale="1 1 1" />
+        </geometry>
+      </collision>
+      <inertial>
+        <mass value="7.64604" />
+        <origin xyz="-0.012819 -0.002679 0.007207" rpy="0 -0 0"/>
+        <inertia ixx="0.0658136" ixy="-0.000159462" ixz="0.010103" iyy="0.0504268" iyz="0.000173435" izz="0.0889772"/>
+      </inertial>
+    </link>
+    <gazebo reference="lifter_top_link">
+      <mu1>0.9</mu1>
+      <mu2>0.9</mu2>
+    </gazebo>
     <joint name="lifter_top_connector" type="fixed">
       <parent link="leg_base_link"/>

File: aero_description/typeF/urdf/aero-wheels/wheels.urdf.xacro (robot description, xacro)
@@ -16,5 +16,5 @@
   <xacro:include filename="$(find aero_description)/urdf/common.xacro" />
   <xacro:macro name="wheels" params="base_link">
-    <link name="${base_link}" />
+    <link name="${base_link}"/>
     <link name="wheels_body_link">
       <visual>
@@ -36,5 +36,23 @@
       </inertial>
     </link>
-    <link name="wheels_top_link" />
+    <link name="wheels_top_link">
+      <visual>
+        <origin xyz="0.0 0.0 0.0" rpy="0 -0 0"/>
+        <geometry>
+          <mesh filename="package://aero_description/meshes/aero-lower_meshes/wheels_top.dae" scale="1 1 1" />
+        </geometry>
+      </visual>
+      <collision>
+        <origin xyz="0.0 0.0 0.0" rpy="0 -0 0"/>
+        <geometry>
+          <mesh filename="package://aero_description/meshes/aero-lower_meshes/wheels_top.dae" scale="1 1 1" />
+        </geometry>
+      </collision>
+      <inertial>
+        <mass value="10" />
+        <origin xyz="0 0 0" rpy="0 -0 0"/>
+        <inertia ixx="0.528" ixy="0" ixz="0" iyy="2.02" iyz="0" izz="2.35"/>
+      </inertial>
+    </link>
     <joint name="wheels_base_to_body_connector" type="fixed">
       <parent  link="${base_link}"/>

Commit message: fix joint name

File: aero_description/typeF/urdf/aero-wheels/lifter.urdf.xacro (robot description, xacro)
@@ -182,10 +182,10 @@
       <dynamics damping="0.2" friction="0" />
     </joint>
-    <transmission type="pr2_mechanism_model/SimpleTransmission" name="hip_joint_trans" >
-      <actuator name="hip_joint_motor" />
-      <joint name="hip_joint" />
+    <transmission type="pr2_mechanism_model/SimpleTransmission" name="ankle_joint_trans" >
+      <actuator name="ankle_joint_motor" />
+      <joint name="ankle_joint" />
       <mechanicalReduction>1</mechanicalReduction>
     </transmission>
-    <gazebo reference="hip_joint">
+    <gazebo reference="ankle_joint">
       <implicitSpringDamper>0.4</implicitSpringDamper>
     </gazebo>

File: aero_description/typeF/urdf/aero-wheels/wheels.urdf.xacro (robot description, xacro)
@@ -16,6 +16,5 @@
   <xacro:include filename="$(find aero_description)/urdf/common.xacro" />
   <xacro:macro name="wheels" params="base_link">
-    <link name="${base_link}"/>
-    <link name="wheels_body_link">
+    <link name="${base_link}">
       <visual>
         <origin xyz="0.0 0.0 0.0" rpy="0 -0 0"/>
@@ -32,8 +31,12 @@
       <inertial>
         <mass value="10" />
-        <origin xyz="0 0 0" rpy="0 -0 0"/>
+        <origin xyz="0 0 0" rpy="0 -0 0.09"/>
         <inertia ixx="0.528" ixy="0" ixz="0" iyy="2.02" iyz="0" izz="2.35"/>
       </inertial>
     </link>
+    <gazebo reference="${base_link}">
+      <mu1>0.9</mu1>
+      <mu2>0.9</mu2>
+    </gazebo>
     <link name="wheels_top_link">
       <visual>
@@ -55,9 +58,8 @@
       </inertial>
     </link>
-    <joint name="wheels_base_to_body_connector" type="fixed">
-      <parent  link="${base_link}"/>
-      <child link="wheels_body_link"/>
-      <origin xyz="0.0 0.0 0.0" rpy="0 0 0 "/>
-    </joint>
+    <gazebo reference="wheels_top_link">
+      <mu1>0.9</mu1>
+      <mu2>0.9</mu2>
+    </gazebo>
     <joint name="wheels_body_to_top_connector" type="fixed">
       <parent  link="wheels_body_link"/>
