Commit message: virtual lifter for moveit ik

File: aero_description/typeF/urdf/aero-wheels/aero-wheels.urdf.xacro (robot description, xacro)
@@ -16,6 +16,7 @@
   <xacro:include filename="$(find aero_description)/urdf/aero-wheels/lifter.urdf.xacro" />
   <xacro:include filename="$(find aero_description)/urdf/aero-wheels/wheels.urdf.xacro" />
+  <xacro:include filename="$(find aero_description)/urdf/aero-wheels/virtual_lifter.urdf.xacro" />
   <xacro:include filename="$(find aero_description)/urdf/common.xacro" />
-  <xacro:macro name="aero-wheels" params="base_link">
+  <xacro:macro name="aero-wheels" params="base_link virtual_lifter:=false x_max:=0.0 x_min:=0.0 z_max:=0.0 z_min:=0.0">
     <xacro:wheels base_link="${base_link}"/>
     <joint name="wheel_lifter_connector" type="fixed">
@@ -24,5 +25,10 @@
       <origin xyz="0.0 0.0 0.0" rpy="0 0 0 "/>
    </joint>
+   <xacro:unless value="${virtual_lifter}">
     <xacro:lifter base_link="lifter_base_link"/>
+   </xacro:unless>
+   <xacro:if value="${virtual_lifter}">
+    <xacro:virtual_lifter base_link="lifter_base_link" x_max="${x_max}" x_min="${x_min}" z_max="${z_max}" z_min="${z_min}"/>
+   </xacro:if>
   </xacro:macro>
 </robot>

File: aero_description/typeF/urdf/aero-wheels/lifter.urdf.xacro (robot description, xacro)
@@ -42,4 +42,5 @@
     <link name="leg_thigh_link">
       <visual>
+        <!--origin xyz="0.0 0.0 0.29009" rpy="0 -0 0"/-->
         <origin xyz="0.0 0.0 0.29009" rpy="0 -0 0"/>
         <geometry>
@@ -65,5 +66,6 @@
     <link name="leg_foreleg_link">
       <visual>
-        <origin xyz="0.0 0.0 0.29009" rpy="0 -0 0"/>
+        <!--origin xyz="0.0 0.0 0.29009" rpy="0 -0 0"/-->
+        <origin xyz="0.0 0.0 0.235" rpy="0 -0 0"/>
         <geometry>
           <mesh filename="package://aero_description/meshes/aero-lower_meshes/wheel_lower_mesh.dae" scale="1 1 1" />
@@ -90,10 +92,12 @@
       <parent link="leg_base_link"/>
       <child  link="lifter_top_link"/>
-      <origin xyz="-0.01591 0.0 0.05" rpy="0 -0 0 "/>
+      <!--origin xyz="-0.01591 0.0 0.05" rpy="0 -0 0 "/-->
+      <origin xyz="-0.01591 0.0 0.10509" rpy="0 -0 0 "/>
     </joint>
     <joint name="hip_joint" type="revolute">
       <parent link="leg_thigh_link"/>
       <child  link="leg_base_link"/>
-      <origin xyz="0 0 0.29009" rpy="0 -0 0 "/>
+      <!--origin xyz="0 0 0.29009" rpy="0 -0 0 "/-->
+      <origin xyz="0 0 0.235" rpy="0 -0 0 "/>
       <axis   xyz="0 -1 0"/>
       <limit lower="0" upper="1.5707" effort="100" velocity="0.5" />
@@ -111,5 +115,6 @@
       <parent link="leg_foreleg_link"/>
       <child  link="leg_thigh_link"/>
-      <origin xyz="0.0 0.0 0.29009" rpy="0 -0 0 "/>
+      <!--origin xyz="0 0 0.29009" rpy="0 -0 0 "/-->
+      <origin xyz="0 0 0.235" rpy="0 -0 0 "/>
       <axis   xyz="0 1 0"/>
       <limit lower="0" upper="3.14159" effort="100" velocity="0.5" />
@@ -127,5 +132,6 @@
       <parent link="${base_link}"/>
       <child  link="leg_foreleg_link"/>
-      <origin xyz="0.0 0.0 0.07" rpy="0 -0 0 "/>
+      <!--origin xyz="0.0 0.0 0.07" rpy="0 -0 0 "/-->
+      <origin xyz="0.0 0.0 0.12509" rpy="0 -0 0 "/>
       <axis   xyz="0 -1 0"/>
       <limit lower="0" upper="1.5707" effort="100" velocity="0.5" />

Commit message: Change New wheel model

File: aero_description/typeF/urdf/aero-wheels/aero-wheels.urdf.xacro (robot description, xacro)
@@ -23,5 +23,5 @@
       <parent  link="wheels_top_link"/>
       <child link="lifter_base_link"/>
-      <origin xyz="0.0 0.0 0.0" rpy="0 0 0 "/>
+      <origin xyz="0.0 0.0 0.005" rpy="0 0 0 "/>
    </joint>
    <xacro:unless value="${virtual_lifter}">

File: aero_description/typeF/urdf/aero-wheels/lifter.urdf.xacro (robot description, xacro)
@@ -39,15 +39,84 @@
       <mu2>0.9</mu2>
     </gazebo>
+    <link name="leg_foreleg_link">
+      <visual>
+        <origin xyz="0.0 0.0 0" rpy="3.1415 -0 0"/>
+        <geometry>
+          <mesh filename="package://aero_description/meshes/aero-lower_meshes/lifter_bone.dae" scale="1 1 1" />
+        </geometry>
+      </visual>
+      <collision>
+        <origin xyz="0.0 0.0 0.0" rpy="0 -0 0"/>
+        <geometry>
+          <mesh filename="package://aero_description/meshes/aero-lower_meshes/lifter_bone.dae" scale="1 1 1" />
+        </geometry>
+      </collision>
+      <inertial>
+        <mass value="2.06679" />
+        <origin xyz="0.081713 0.000812 -0.146934" rpy="0 -0 0"/>
+        <inertia ixx="0.0408818" ixy="-9.39301e-06" ixz="-0.000750165" iyy="0.0403969" iyz="-0.000120419" izz="0.00260982"/>
+      </inertial>
+    </link>
+    <gazebo reference="leg_foreleg_link">
+      <mu1>0.9</mu1>
+      <mu2>0.9</mu2>
+    </gazebo>
+    <link name="leg_knee_link">
+      <visual>
+        <origin xyz="0.0 0.0 0" rpy="3.1415 -0 0"/>
+        <geometry>
+          <mesh filename="package://aero_description/meshes/aero-lower_meshes/lifter_knee.dae" scale="1 1 1" />
+        </geometry>
+      </visual>
+      <collision>
+        <origin xyz="0.0 0.0 0.0" rpy="0 -0 0"/>
+        <geometry>
+          <mesh filename="package://aero_description/meshes/aero-lower_meshes/lifter_knee.dae" scale="1 1 1" />
+        </geometry>
+      </collision>
+      <inertial>
+        <mass value="2.06679" />
+        <origin xyz="0.081713 0.000812 -0.146934" rpy="0 -0 0"/>
+        <inertia ixx="0.0408818" ixy="-9.39301e-06" ixz="-0.000750165" iyy="0.0403969" iyz="-0.000120419" izz="0.00260982"/>
+      </inertial>
+    </link>
+    <gazebo reference="leg_knee_link">
+      <mu1>0.9</mu1>
+      <mu2>0.9</mu2>
+    </gazebo>
+    <link name="leg_thigh_link">
+      <visual>
+        <origin xyz="0 0 0.25" rpy="0 0 0"/>
+        <geometry>
+          <mesh filename="package://aero_description/meshes/aero-lower_meshes/lifter_bone.dae" scale="1 1 1" />
+        </geometry>
+      </visual>
+      <collision>
+        <origin xyz="0.0 0.0 0.0" rpy="0 -0 0"/>
+        <geometry>
+          <mesh filename="package://aero_description/meshes/aero-lower_meshes/lifter_bone.dae" scale="1 1 1" />
+        </geometry>
+      </collision>
+      <inertial>
+        <mass value="2.62321" />
+        <origin xyz="0.0587169 0 -0.135292" rpy="0 -0 0"/>
+        <inertia ixx="0.0161595" ixy="-9.27234e-05" ixz="0.00262839" iyy="0.0166415" iyz="-0.00017447" izz="0.00477281"/>
+      </inertial>
+    </link>
+    <gazebo reference="leg_thigh_link">
+      <mu1>0.9</mu1>
+      <mu2>0.9</mu2>
+    </gazebo>
     <link name="leg_base_link">
       <visual>
-        <origin xyz="0 0 0" rpy="0 -0 0"/>
-        <geometry>
-          <mesh filename="package://aero_description/meshes/aero-lower_meshes/lifter_top_connector.dae" scale="1 1 1" />
-        </geometry>
-      </visual>
-      <collision>
-        <origin xyz="0 0 0" rpy="0 -0 0"/>
-        <geometry>
-          <mesh filename="package://aero_description/meshes/aero-lower_meshes/lifter_top_connector.dae" scale="1 1 1" />
+        <origin xyz="0 0 0.05" rpy="3.1415920 0 0"/>
+        <geometry>
+          <mesh filename="package://aero_description/meshes/aero-lower_meshes/lifter_base.dae" scale="1 1 1" />
+        </geometry>
+      </visual>
+      <collision>
+        <origin xyz="0 0 0" rpy="0 -0 0"/>
+        <geometry>
+          <mesh filename="package://aero_description/meshes/aero-lower_meshes/lifter_base.dae" scale="1 1 1" />
         </geometry>
       </collision>
@@ -62,52 +131,4 @@
       <mu2>0.9</mu2>
     </gazebo>
-    <link name="leg_thigh_link">
-      <visual>
-        <!--origin xyz="0.0 0.0 0.29009" rpy="0 -0 0"/-->
-        <origin xyz="0.0 0.0 0.29009" rpy="0 -0 0"/>
-        <geometry>
-          <mesh filename="package://aero_description/meshes/aero-lower_meshes/wheel_upper_mesh.dae" scale="1 1 1" />
-        </geometry>
-      </visual>
-      <collision>
-        <origin xyz="0.0 0.0 0.0" rpy="0 -0 0"/>
-        <geometry>
-          <mesh filename="package://aero_description/meshes/aero-lower_meshes/wheel_upper_mesh.dae" scale="1 1 1" />
-        </geometry>
-      </collision>
-      <inertial>
-        <mass value="2.62321" />
-        <origin xyz="0.0587169 0 -0.135292" rpy="0 -0 0"/>
-        <inertia ixx="0.0161595" ixy="-9.27234e-05" ixz="0.00262839" iyy="0.0166415" iyz="-0.00017447" izz="0.00477281"/>
-      </inertial>
-    </link>
-    <gazebo reference="leg_thigh_link">
-      <mu1>0.9</mu1>
-      <mu2>0.9</mu2>
-    </gazebo>
-    <link name="leg_foreleg_link">
-      <visual>
-        <!--origin xyz="0.0 0.0 0.29009" rpy="0 -0 0"/-->
-        <origin xyz="0.0 0.0 0.235" rpy="0 -0 0"/>
-        <geometry>
-          <mesh filename="package://aero_description/meshes/aero-lower_meshes/wheel_lower_mesh.dae" scale="1 1 1" />
-        </geometry>
-      </visual>
-      <collision>
-        <origin xyz="0.0 0.0 0.0" rpy="0 -0 0"/>
-        <geometry>
-          <mesh filename="package://aero_description/meshes/aero-lower_meshes/wheel_lower_mesh.dae" scale="1 1 1" />
-        </geometry>
-      </collision>
-      <inertial>
-        <mass value="2.06679" />
-        <origin xyz="0.081713 0.000812 -0.146934" rpy="0 -0 0"/>
-        <inertia ixx="0.0408818" ixy="-9.39301e-06" ixz="-0.000750165" iyy="0.0403969" iyz="-0.000120419" izz="0.00260982"/>
-      </inertial>
-    </link>
-    <gazebo reference="leg_foreleg_link">
-      <mu1>0.9</mu1>
-      <mu2>0.9</mu2>
-    </gazebo>
     <link name="lifter_top_link">
       <visual>
@@ -136,12 +157,10 @@
       <parent link="leg_base_link"/>
       <child  link="lifter_top_link"/>
-      <!--origin xyz="-0.01591 0.0 0.05" rpy="0 -0 0 "/-->
-      <origin xyz="-0.01591 0.0 0.10509" rpy="0 -0 0 "/>
+      <origin xyz="0 0 0.055" rpy="0 0 0"/>
     </joint>
     <joint name="hip_joint" type="revolute">
       <parent link="leg_thigh_link"/>
-      <child  link="leg_base_link"/>
-      <!--origin xyz="0 0 0.29009" rpy="0 -0 0 "/-->
-      <origin xyz="0 0 0.235" rpy="0 -0 0 "/>
+      <child link="leg_base_link"/>
+      <origin xyz="0 0 0.25" rpy="0 0 0"/>
       <axis   xyz="0 -1 0"/>
       <limit lower="0" upper="1.5707" effort="100" velocity="0.5" />
@@ -156,9 +175,9 @@
       <implicitSpringDamper>0.4</implicitSpringDamper>
     </gazebo>
+<!--
     <joint name="knee_joint" type="revolute">
       <parent link="leg_foreleg_link"/>
-      <child  link="leg_thigh_link"/>
-      <!--origin xyz="0 0 0.29009" rpy="0 -0 0 "/-->
-      <origin xyz="0 0 0.235" rpy="0 -0 0 "/>
+      <child  link="leg_knee_link"/>
+      <origin xyz="0 0 0.25" rpy="0 0 0"/>
       <axis   xyz="0 1 0"/>
       <limit lower="0" upper="3.14159" effort="100" velocity="0.5" />
@@ -173,9 +192,9 @@
       <implicitSpringDamper>0.4</implicitSpringDamper>
     </gazebo>
+-->
     <joint name="ankle_joint" type="revolute">
       <parent link="${base_link}"/>
       <child  link="leg_foreleg_link"/>
-      <!--origin xyz="0.0 0.0 0.07" rpy="0 -0 0 "/-->
-      <origin xyz="0.0 0.0 0.12509" rpy="0 -0 0 "/>
+      <origin xyz="0 0 0.05" rpy="0 0 0"/>
       <axis   xyz="0 -1 0"/>
       <limit lower="0" upper="1.5707" effort="100" velocity="0.5" />
@@ -190,4 +209,51 @@
       <implicitSpringDamper>0.4</implicitSpringDamper>
     </gazebo>
+<!--- mimic joints -->
+<!-- requried -->
+    <joint name="knee_joint_foreleg_dummy" type="continuous">
+      <parent link="leg_foreleg_link"/>
+      <child  link="leg_knee_link"/>
+      <origin xyz="0 0 0.25" rpy="0 0 0"/>
+      <axis   xyz="0 -1 0"/>
+      <mimic joint="ankle_joint" multiplier="-1" offset="0" />
+    </joint>
+    <joint name="knee_joint_thigh_dummy" type="continuous">
+      <parent link="leg_knee_link"/>
+      <child  link="leg_thigh_link"/>
+      <origin xyz="0 0 0.12" rpy="0 0 0"/>
+      <axis xyz="0 -1 0"/>
+      <mimic joint="hip_joint" multiplier="-1" offset="0" />
+    </joint>
+<!-- redundant -->
+    <link name="leg_foreleg_link_dummy">
+      <visual>
+        <geometry>
+          <mesh filename="package://aero_description/meshes/aero-lower_meshes/lifter_bone_dummy.dae" scale="1 1 1" />
+        </geometry>
+        <origin xyz="0 0 0.25" rpy="0 0 0"/>
+      </visual>
+    </link>
+    <link name="leg_thigh_link_dummy">
+      <visual>
+        <geometry>
+          <mesh filename="package://aero_description/meshes/aero-lower_meshes/lifter_bone_dummy.dae" scale="1 1 1" />
+        </geometry>
+        <origin xyz="0 0 0.25" rpy="0 0 0"/>
+      </visual>
+    </link>
+    <joint name="ankle_joint_dummy" type="continuous">
+      <parent link="${base_link}"/>
+      <child link="leg_foreleg_link_dummy"/>
+      <origin xyz="0.03182 0 0.08182" rpy="0 0 0"/>
+      <axis xyz="0 -1 0"/>
+      <mimic joint="ankle_joint" multiplier="1" offset="0" />
+    </joint>
+    <joint name="hip_joint_dummy" type="continuous">
+      <parent link="leg_knee_link"/>
+      <child link="leg_thigh_link_dummy"/>
+      <origin xyz="0.03182 0 0.08818" rpy="0 0 0"/>
+      <axis xyz="0 1 0"/>
+      <mimic joint="hip_joint" multiplier="1" offset="0" />
+    </joint>
   </xacro:macro>
 </robot>

File: aero_description/typeF/urdf/aero-wheels/wheels.urdf.xacro (robot description, xacro)
@@ -62,8 +62,148 @@
       <mu2>0.9</mu2>
     </gazebo>
+    <link name="wheels_front_left_mecanum">
+      <visual>
+        <origin xyz="0.0 0.0 0.0" rpy="-1.57079632679 0 0"/>
+        <geometry>
+          <mesh filename="package://aero_description/meshes/aero-lower_meshes/wheels_mecanum.dae" scale="1 1 1" />
+        </geometry>
+      </visual>
+      <collision>
+        <origin xyz="0.0 0.0 0.0" rpy="0 -0 0"/>
+        <geometry>
+          <mesh filename="package://aero_description/meshes/aero-lower_meshes/wheels_mecanum.dae" scale="1 1 1" />
+        </geometry>
+      </collision>
+      <inertial>
+        <mass value="10" />
+        <origin xyz="0 0 0" rpy="0 -0 0"/>
+        <inertia ixx="0.528" ixy="0" ixz="0" iyy="2.02" iyz="0" izz="2.35"/>
+      </inertial>
+    </link>
+    <gazebo reference="wheels_front_left_mecanum">
+      <mu1>0.9</mu1>
+      <mu2>0.9</mu2>
+    </gazebo>
+    <link name="wheels_front_right_mecanum">
+      <visual>
+        <origin xyz="0.0 0.0 0.0" rpy="-1.57079632679 0 0"/>
+        <geometry>
+          <mesh filename="package://aero_description/meshes/aero-lower_meshes/wheels_mecanum.dae" scale="1 1 1" />
+        </geometry>
+      </visual>
+      <collision>
+        <origin xyz="0.0 0.0 0.0" rpy="0 -0 0"/>
+        <geometry>
+          <mesh filename="package://aero_description/meshes/aero-lower_meshes/wheels_mecanum.dae" scale="1 1 1" />
+        </geometry>
+      </collision>
+      <inertial>
+        <mass value="10" />
+        <origin xyz="0 0 0" rpy="0 -0 0"/>
+        <inertia ixx="0.528" ixy="0" ixz="0" iyy="2.02" iyz="0" izz="2.35"/>
+      </inertial>
+    </link>
+    <gazebo reference="wheels_front_left_mecanum">
+      <mu1>0.9</mu1>
+      <mu2>0.9</mu2>
+    </gazebo>
+    <link name="wheels_rear_left_mecanum">
+      <visual>
+        <origin xyz="0.0 0.0 0.0" rpy="-1.57079632679 0 0"/>
+        <geometry>
+          <mesh filename="package://aero_description/meshes/aero-lower_meshes/wheels_mecanum.dae" scale="1 1 1" />
+        </geometry>
+      </visual>
+      <collision>
+        <origin xyz="0.0 0.0 0.0" rpy="0 -0 0"/>
+        <geometry>
+          <mesh filename="package://aero_description/meshes/aero-lower_meshes/wheels_mecanum.dae" scale="1 1 1" />
+        </geometry>
+      </collision>
+      <inertial>
+        <mass value="10" />
+        <origin xyz="0 0 0" rpy="0 -0 0"/>
+        <inertia ixx="0.528" ixy="0" ixz="0" iyy="2.02" iyz="0" izz="2.35"/>
+      </inertial>
+    </link>
+    <gazebo reference="wheels_rear_left_mecanum">
+      <mu1>0.9</mu1>
+      <mu2>0.9</mu2>
+    </gazebo>
+    <link name="wheels_rear_right_mecanum">
+      <visual>
+        <origin xyz="0.0 0.0 0.0" rpy="-1.57079632679 0 0"/>
+        <geometry>
+          <mesh filename="package://aero_description/meshes/aero-lower_meshes/wheels_mecanum.dae" scale="1 1 1" />
+        </geometry>
+      </visual>
+      <collision>
+        <origin xyz="0.0 0.0 0.0" rpy="0 -0 0"/>
+        <geometry>
+          <mesh filename="package://aero_description/meshes/aero-lower_meshes/wheels_mecanum.dae" scale="1 1 1" />
+        </geometry>
+      </collision>
+      <inertial>
+        <mass value="10" />
+        <origin xyz="0 0 0" rpy="0 -0 0"/>
+        <inertia ixx="0.528" ixy="0" ixz="0" iyy="2.02" iyz="0" izz="2.35"/>
+      </inertial>
+    </link>
+    <gazebo reference="wheels_rear_right_mecanum">
+      <mu1>0.9</mu1>
+      <mu2>0.9</mu2>
+    </gazebo>
+    <link name="wheels_base_laser_link">
+      <visual>
+        <origin xyz="0.0 0.0 0.0" rpy="0 0 0"/>
+        <geometry>
+          <mesh filename="package://aero_description/meshes/aero-lower_meshes/wheels_urg.dae" scale="1 1 1" />
+        </geometry>
+      </visual>
+      <collision>
+        <origin xyz="0.0 0.0 0.0" rpy="0 -0 0"/>
+        <geometry>
+          <mesh filename="package://aero_description/meshes/aero-lower_meshes/wheels_urg.dae" scale="1 1 1" />
+        </geometry>
+      </collision>
+      <inertial>
+        <mass value="10" />
+        <origin xyz="0 0 0" rpy="0 -0 0"/>
+        <inertia ixx="0.528" ixy="0" ixz="0" iyy="2.02" iyz="0" izz="2.35"/>
+      </inertial>
+    </link>
+    <gazebo reference="wheels_base_laser_link">
+      <mu1>0.9</mu1>
+      <mu2>0.9</mu2>
+    </gazebo>
     <joint name="wheels_body_to_top_connector" type="fixed">
       <parent  link="${base_link}"/>
       <child link="wheels_top_link"/>
-      <origin xyz="0.0 0.0 0.17" rpy="0 0 0 "/>
+      <origin xyz="0.0 0.0 0.115" rpy="0 0 0 "/>
+    </joint>
+    <joint name="wheels_body_to_front_left_mecanum_connector" type="fixed">
+      <parent  link="${base_link}"/>
+      <child link="wheels_front_left_mecanum"/>
+      <origin xyz="0.225 0.19456 0" rpy="0 0 0"/>
+    </joint>
+    <joint name="wheels_body_to_front_right_mecanum_connector" type="fixed">
+      <parent  link="${base_link}"/>
+      <child link="wheels_front_right_mecanum"/>
+      <origin xyz="0.225 -0.19456 0" rpy="0 0 0"/>
+    </joint>
+    <joint name="wheels_body_to_rear_left_mecanum_connector" type="fixed">
+      <parent  link="${base_link}"/>
+      <child link="wheels_rear_left_mecanum"/>
+      <origin xyz="-0.225 0.19456 0" rpy="0 0 0"/>
+    </joint>
+    <joint name="wheels_body_to_rear_right_mecanum_connector" type="fixed">
+      <parent  link="${base_link}"/>
+      <child link="wheels_rear_right_mecanum"/>
+      <origin xyz="-0.225 -0.19456 0" rpy="0 0 0"/>
+    </joint>
+    <joint name="wheels_body_to_base_laser_connector" type="fixed">
+      <parent  link="${base_link}"/>
+      <child link="wheels_base_laser_link"/>
+      <origin xyz="0.220697 0 0.1594" rpy="0 0 0"/>
     </joint>
   </xacro:macro>
