Commit message: mod virtual urdf parameter

File: aero_description/typeF/urdf/aero-wheels/virtual_lifter.urdf.xacro (robot description, xacro)
@@ -47,5 +47,5 @@
       <child  link="lifter_top_link"/>
       <!--origin xyz="-0.01591 0.0 0.05" rpy="0 -0 0 "/-->
-      <origin xyz="-0.01591 0.0 0.055" rpy="0 -0 0 "/>
+      <origin xyz="0.0 0.0 0.055" rpy="0 -0 0 "/>
     </joint>
     <joint name="virtual_lifter_z_joint" type="prismatic">
@@ -70,5 +70,5 @@
       <child  link="virtual_lifter_x_link"/>
       <!--origin xyz="0.0 0.0 0.07" rpy="0 -0 0 "/-->
-      <origin xyz="0.0 0.0 0.12" rpy="0 -0 0 "/>
+      <origin xyz="0.0 0.0 0.17" rpy="0 -0 0 "/>
       <axis   xyz="0 -1 0"/>
     </joint>
