Commit message: lifter length fixed from 0.235 to 0.25

File: aero_description/typeF/robots/aero_moveit_ik_op.urdf.xacro (robot description, xacro)
@@ -18,4 +18,4 @@
     <origin xyz="0.0 0.0 0.0" rpy="0 0 0 "/>
   </joint>
-  <xacro:aero-wheels base_link="base_link" virtual_lifter="true" x_max="0.16" x_min="-0.16" z_max="-0.075" z_min="-0.235"/>
+  <xacro:aero-wheels base_link="base_link" virtual_lifter="true" x_max="0.17" x_min="-0.17" z_max="-0.08" z_min="-0.25"/>
 </robot>

File: aero_description/typeF/urdf/aero-wheels/virtual_lifter.urdf.xacro (robot description, xacro)
@@ -47,5 +47,5 @@
       <child  link="lifter_top_link"/>
       <!--origin xyz="-0.01591 0.0 0.05" rpy="0 -0 0 "/-->
-      <origin xyz="-0.01591 0.0 0.10509" rpy="0 -0 0 "/>
+      <origin xyz="-0.01591 0.0 0.055" rpy="0 -0 0 "/>
     </joint>
     <joint name="virtual_lifter_z_joint" type="prismatic">
@@ -61,5 +61,5 @@
       <child  link="virtual_lifter_z_link"/>
       <!--origin xyz="0.0 0.0 0.58018" rpy="0 -0 0 "/-->
-      <origin xyz="0.0 0.0 0.47" rpy="0 -0 0 "/>
+      <origin xyz="0.0 0.0 0.5" rpy="0 -0 0 "/>
       <axis   xyz="1 0 0"/>
       <limit lower="${x_min}" upper="${x_max}" effort="100" velocity="0.1" />
@@ -70,5 +70,5 @@
       <child  link="virtual_lifter_x_link"/>
       <!--origin xyz="0.0 0.0 0.07" rpy="0 -0 0 "/-->
-      <origin xyz="0.0 0.0 0.12509" rpy="0 -0 0 "/>
+      <origin xyz="0.0 0.0 0.12" rpy="0 -0 0 "/>
       <axis   xyz="0 -1 0"/>
     </joint>
