Commit message: remove mesh

File: aero_description/typeF/robots/aero_moveit_ik.urdf.xacro (robot description, xacro)
@@ -12,5 +12,5 @@
   <xacro:include filename="$(find aero_description)/urdf/aero-wheels/aero-wheels.urdf.xacro" />
   <!-- Now we can start using the macros included above to define the actual aero -->
-  <xacro:aero_upper base_link="waist_link"/>
+  <xacro:aero_upper base_link="waist_link" disable_mesh="true"/>
   <joint name="upper_lower_connector" type="fixed">
     <parent link="lifter_top_link"/>

File: aero_description/typeF/robots/aero_moveit_ik_ho.urdf.xacro (robot description, xacro)
@@ -12,5 +12,5 @@
   <xacro:include filename="$(find aero_description)/urdf/aero-wheels/aero-wheels.urdf.xacro" />
   <!-- Now we can start using the macros included above to define the actual aero -->
-  <xacro:aero_upper base_link="waist_link"/>
+  <xacro:aero_upper base_link="waist_link" disable_mesh="true"/>
   <joint name="upper_lower_connector" type="fixed">
     <parent link="lifter_top_link"/>

File: aero_description/typeF/robots/aero_moveit_ik_op.urdf.xacro (robot description, xacro)
@@ -12,5 +12,5 @@
   <xacro:include filename="$(find aero_description)/urdf/aero-wheels/aero-wheels.urdf.xacro" />
   <!-- Now we can start using the macros included above to define the actual aero -->
-  <xacro:aero_upper base_link="waist_link"/>
+  <xacro:aero_upper base_link="waist_link" disable_mesh="true"/>
   <joint name="upper_lower_connector" type="fixed">
     <parent link="lifter_top_link"/>

File: aero_description/typeF/urdf/aero_upper/aero_upper.urdf.xacro (robot description, xacro)
@@ -9,18 +9,18 @@
   <xacro:include filename="$(find aero_description)/urdf/common.xacro" />
   <!-- ============================   aero_upper   ============================ -->
-  <xacro:macro name="aero_upper" params="base_link">
+  <xacro:macro name="aero_upper" params="base_link disable_mesh:=false">
   <link name="${base_link}">
-    <visual>
+    <xacro:unless value="${disable_mesh}"> <visual>
       <origin xyz="0 0 0" rpy="0 -0 0"/>
       <geometry>
         <mesh filename="package://aero_description/meshes/aero_upper_meshes/WAIST_LINK0_mesh.dae" scale="1 1 1" />
       </geometry>
-    </visual>
-    <collision>
+    </visual> </xacro:unless>
+    <xacro:unless value="${disable_mesh}"> <collision>
       <origin xyz="0 0 0" rpy="0 -0 0"/>
       <geometry>
         <mesh filename="package://aero_description/meshes/aero_upper_meshes/WAIST_LINK0_mesh.dae" scale="1 1 1" />
       </geometry>
-    </collision>
+    </collision> </xacro:unless>
     <inertial>
       <mass value="0" />
@@ -34,16 +34,16 @@
   </gazebo>
   <link name="hip_sphere_link">
-    <visual>
+    <xacro:unless value="${disable_mesh}"> <visual>
       <origin xyz="0 0 0" rpy="0 -0 0"/>
       <geometry>
         <mesh filename="package://aero_description/meshes/aero_upper_meshes/WAIST_LINK1_mesh.dae" scale="1 1 1" />
       </geometry>
-    </visual>
-    <collision>
+    </visual> </xacro:unless>
+    <xacro:unless value="${disable_mesh}"> <collision>
       <origin xyz="0 0 0" rpy="0 -0 0"/>
       <geometry>
         <mesh filename="package://aero_description/meshes/aero_upper_meshes/WAIST_LINK1_mesh.dae" scale="1 1 1" />
       </geometry>
-    </collision>
+    </collision> </xacro:unless>
     <inertial>
       <mass value="1.257" />
@@ -68,16 +68,16 @@
   </gazebo>
   <link name="body_link">
-    <visual>
+    <xacro:unless value="${disable_mesh}"> <visual>
       <origin xyz="0 0 0" rpy="0 -0 0"/>
       <geometry>
         <mesh filename="package://aero_description/meshes/aero_upper_meshes/WAIST_LINK3_mesh.dae" scale="1 1 1" />
       </geometry>
-    </visual>
-    <collision>
+    </visual> </xacro:unless>
+    <xacro:unless value="${disable_mesh}"> <collision>
       <origin xyz="0 0 0" rpy="0 -0 0"/>
       <geometry>
         <mesh filename="package://aero_description/meshes/aero_upper_meshes/WAIST_LINK3_mesh.dae" scale="1 1 1" />
       </geometry>
-    </collision>
+    </collision> </xacro:unless>
     <inertial>
       <mass value="10.551" />
@@ -91,16 +91,16 @@
   </gazebo>
   <link name="l_shoulder_link">
-    <visual>
+    <xacro:unless value="${disable_mesh}"> <visual>
       <origin xyz="0 0 0" rpy="-0.174532925 -0 0"/>
       <geometry>
         <mesh filename="package://aero_description/meshes/aero_upper_meshes/LARM_LINK1_mesh.dae" scale="1 1 1" />
       </geometry>
-    </visual>
-    <collision>
+    </visual> </xacro:unless>
+    <xacro:unless value="${disable_mesh}"> <collision>
       <origin xyz="0 0 0" rpy="-0.174532925 -0 0"/>
       <geometry>
         <mesh filename="package://aero_description/meshes/aero_upper_meshes/LARM_LINK1_mesh.dae" scale="1 1 1" />
       </geometry>
-    </collision>
+    </collision> </xacro:unless>
     <inertial>
       <mass value="0.242" />
@@ -114,16 +114,16 @@
   </gazebo>
   <link name="l_shoulder_center">
-    <visual>
+    <xacro:unless value="${disable_mesh}"> <visual>
       <origin xyz="0 0 0" rpy="0 -0 0"/>
       <geometry>
         <mesh filename="package://aero_description/meshes/aero_upper_meshes/LARM_LINK2_mesh.dae" scale="1 1 1" />
       </geometry>
-    </visual>
-    <collision>
+    </visual> </xacro:unless>
+    <xacro:unless value="${disable_mesh}"> <collision>
       <origin xyz="0 0 0" rpy="0 -0 0"/>
       <geometry>
         <mesh filename="package://aero_description/meshes/aero_upper_meshes/LARM_LINK2_mesh.dae" scale="1 1 1" />
       </geometry>
-    </collision>
+    </collision> </xacro:unless>
     <inertial>
       <mass value="0.744" />
@@ -137,16 +137,16 @@
   </gazebo>
   <link name="l_upperarm_link">
-    <visual>
+    <xacro:unless value="${disable_mesh}"> <visual>
       <origin xyz="0 0 0" rpy="0 -0 0"/>
       <geometry>
         <mesh filename="package://aero_description/meshes/aero_upper_meshes/LARM_LINK3_mesh.dae" scale="1 1 1" />
       </geometry>
-    </visual>
-    <collision>
+    </visual> </xacro:unless>
+    <xacro:unless value="${disable_mesh}"> <collision>
       <origin xyz="0 0 0" rpy="0 -0 0"/>
       <geometry>
         <mesh filename="package://aero_description/meshes/aero_upper_meshes/LARM_LINK3_mesh.dae" scale="1 1 1" />
       </geometry>
-    </collision>
+    </collision> </xacro:unless>
     <inertial>
       <mass value="0.574" />
@@ -160,16 +160,16 @@
   </gazebo>
   <link name="l_elbow_link">
-    <visual>
+    <xacro:unless value="${disable_mesh}"> <visual>
       <origin xyz="-0.035 0 -0.035" rpy="0 -0 0"/>
       <geometry>
         <mesh filename="package://aero_description/meshes/aero_upper_meshes/LARM_LINK4_mesh.dae" scale="1 1 1" />
       </geometry>
-    </visual>
-    <collision>
+    </visual> </xacro:unless>
+    <xacro:unless value="${disable_mesh}"> <collision>
       <origin xyz="-0.035 0 -0.035" rpy="0 -0 0"/>
       <geometry>
         <mesh filename="package://aero_description/meshes/aero_upper_meshes/LARM_LINK4_mesh.dae" scale="1 1 1" />
       </geometry>
-    </collision>
+    </collision> </xacro:unless>
     <inertial>
       <mass value="0.711" />
@@ -183,16 +183,16 @@
   </gazebo>
   <link name="l_forearm_link">
-    <visual>
+    <xacro:unless value="${disable_mesh}"> <visual>
       <origin xyz="0 0 0" rpy="0 -0 0"/>
       <geometry>
         <mesh filename="package://aero_description/meshes/aero_upper_meshes/LARM_LINK5_mesh.dae" scale="1 1 1" />
       </geometry>
-    </visual>
-    <collision>
+    </visual> </xacro:unless>
+    <xacro:unless value="${disable_mesh}"> <collision>
       <origin xyz="0 0 0" rpy="0 -0 0"/>
       <geometry>
         <mesh filename="package://aero_description/meshes/aero_upper_meshes/LARM_LINK5_mesh.dae" scale="1 1 1" />
       </geometry>
-    </collision>
+    </collision> </xacro:unless>
     <inertial>
       <mass value="0.132" />
@@ -217,16 +217,16 @@
   </gazebo>
   <link name="l_hand_link">
-    <visual>
+    <xacro:unless value="${disable_mesh}"> <visual>
       <origin xyz="0 0 0" rpy="0 -0 0"/>
       <geometry>
         <mesh filename="package://aero_description/meshes/aero_upper_meshes/LARM_LINK7_mesh.dae" scale="1 1 1" />
       </geometry>
-    </visual>
-    <collision>
+    </visual> </xacro:unless>
+    <xacro:unless value="${disable_mesh}"> <collision>
       <origin xyz="0 0 0" rpy="0 -0 0"/>
       <geometry>
         <mesh filename="package://aero_description/meshes/aero_upper_meshes/LARM_LINK7_mesh.dae" scale="1 1 1" />
       </geometry>
-    </collision>
+    </collision> </xacro:unless>
     <inertial>
       <mass value="0.183" />
@@ -240,16 +240,16 @@
   </gazebo>
   <link name="l_thumb_link">
-    <visual>
+    <xacro:unless value="${disable_mesh}"> <visual>
       <origin xyz="0 -0.013 0.115" rpy="0 -0 0 "/>
       <geometry>
         <mesh filename="package://aero_description/meshes/aero_upper_meshes/LARM_INDEX_LINK1_mesh.dae" scale="1 1 1" />
       </geometry>
-    </visual>
-    <collision>
+    </visual> </xacro:unless>
+    <xacro:unless value="${disable_mesh}"> <collision>
       <origin xyz="0 -0.013 0.115" rpy="0 -0 0 "/>
       <geometry>
         <mesh filename="package://aero_description/meshes/aero_upper_meshes/LARM_INDEX_LINK1_mesh.dae" scale="1 1 1" />
       </geometry>
-    </collision>
+    </collision> </xacro:unless>
     <inertial>
       <mass value="0" />
@@ -263,16 +263,16 @@
   </gazebo>
   <link name="l_indexbase_link">
-    <visual>
+    <xacro:unless value="${disable_mesh}"> <visual>
       <origin xyz="0 0.015754 0.149615" rpy="0 -0 0"/>
       <geometry>
         <mesh filename="package://aero_description/meshes/aero_upper_meshes/LARM_INDEX_LINK2_mesh.dae" scale="1 1 1" />
       </geometry>
-    </visual>
-    <collision>
+    </visual> </xacro:unless>
+    <xacro:unless value="${disable_mesh}"> <collision>
       <origin xyz="0 0.015754 0.149615" rpy="0 -0 0"/>
       <geometry>
         <mesh filename="package://aero_description/meshes/aero_upper_meshes/LARM_INDEX_LINK2_mesh.dae" scale="1 1 1" />
       </geometry>
-    </collision>
+    </collision> </xacro:unless>
     <inertial>
       <mass value="0" />
@@ -286,16 +286,16 @@
   </gazebo>
   <link name="l_indexmid_link">
-    <visual>
+    <xacro:unless value="${disable_mesh}"> <visual>
       <origin xyz="0 0.03747 0.162972" rpy="0 -0 0"/>
       <geometry>
         <mesh filename="package://aero_description/meshes/aero_upper_meshes/LARM_INDEX_LINK3_mesh.dae" scale="1 1 1" />
       </geometry>
-    </visual>
-    <collision>
+    </visual> </xacro:unless>
+    <xacro:unless value="${disable_mesh}"> <collision>
       <origin xyz="0 0.03747 0.162972" rpy="0 -0 0"/>
       <geometry>
         <mesh filename="package://aero_description/meshes/aero_upper_meshes/LARM_INDEX_LINK3_mesh.dae" scale="1 1 1" />
       </geometry>
-    </collision>
+    </collision> </xacro:unless>
     <inertial>
       <mass value="0" />
@@ -309,16 +309,16 @@
   </gazebo>
   <link name="l_indexend_link">
-    <visual>
+    <xacro:unless value="${disable_mesh}"> <visual>
       <origin xyz="0 0.022355 0.079645" rpy="0 -0 0 "/>
       <geometry>
         <mesh filename="package://aero_description/meshes/aero_upper_meshes/LARM_THUMB_LINK_mesh.dae" scale="1 1 1" />
       </geometry>
-    </visual>
-    <collision>
+    </visual> </xacro:unless>
+    <xacro:unless value="${disable_mesh}"> <collision>
       <origin xyz="0 0.022355 0.079645" rpy="0 -0 0 "/>
       <geometry>
         <mesh filename="package://aero_description/meshes/aero_upper_meshes/LARM_THUMB_LINK_mesh.dae" scale="1 1 1" />
       </geometry>
-    </collision>
+    </collision> </xacro:unless>
     <inertial>
       <mass value="0" />
@@ -332,16 +332,16 @@
   </gazebo>
   <link name="neck_link">
-    <visual>
+    <xacro:unless value="${disable_mesh}"> <visual>
       <origin xyz="0 0 0" rpy="0 -0 0"/>
       <geometry>
         <mesh filename="package://aero_description/meshes/aero_upper_meshes/NECK_LINK1_mesh.dae" scale="1 1 1" />
       </geometry>
-    </visual>
-    <collision>
+    </visual> </xacro:unless>
+    <xacro:unless value="${disable_mesh}"> <collision>
       <origin xyz="0 0 0" rpy="0 -0 0"/>
       <geometry>
         <mesh filename="package://aero_description/meshes/aero_upper_meshes/NECK_LINK1_mesh.dae" scale="1 1 1" />
       </geometry>
-    </collision>
+    </collision> </xacro:unless>
     <inertial>
       <mass value="0.341" />
@@ -355,16 +355,16 @@
   </gazebo>
   <link name="head_base_link">
-    <visual>
+    <xacro:unless value="${disable_mesh}"> <visual>
       <origin xyz="0 0 0" rpy="0 -0 0"/>
       <geometry>
         <mesh filename="package://aero_description/meshes/aero_upper_meshes/NECK_LINK2_mesh.dae" scale="1 1 1" />
       </geometry>
-    </visual>
-    <collision>
+    </visual> </xacro:unless>
+    <xacro:unless value="${disable_mesh}"> <collision>
       <origin xyz="0 0 0" rpy="0 -0 0"/>
       <geometry>
         <mesh filename="package://aero_description/meshes/aero_upper_meshes/NECK_LINK2_mesh.dae" scale="1 1 1" />
       </geometry>
-    </collision>
+    </collision> </xacro:unless>
     <inertial>
       <mass value="0" />
@@ -378,16 +378,16 @@
   </gazebo>
   <link name="head_link">
-    <visual>
+    <xacro:unless value="${disable_mesh}"> <visual>
       <origin xyz="0 0 0" rpy="0 -0 0"/>
       <geometry>
         <mesh filename="package://aero_description/meshes/aero_upper_meshes/NECK_LINK3_mesh.dae" scale="1 1 1" />
       </geometry>
-    </visual>
-    <collision>
+    </visual> </xacro:unless>
+    <xacro:unless value="${disable_mesh}"> <collision>
       <origin xyz="0 0 0" rpy="0 -0 0"/>
       <geometry>
         <mesh filename="package://aero_description/meshes/aero_upper_meshes/NECK_LINK3_mesh.dae" scale="1 1 1" />
       </geometry>
-    </collision>
+    </collision> </xacro:unless>
     <inertial>
       <mass value="0.974" />
@@ -401,16 +401,16 @@
   </gazebo>
   <link name="r_shoulder_link">
-    <visual>
+    <xacro:unless value="${disable_mesh}"> <visual>
       <origin xyz="0 0 0" rpy="0.174532925 -0 0"/>
       <geometry>
         <mesh filename="package://aero_description/meshes/aero_upper_meshes/RARM_LINK1_mesh.dae" scale="1 1 1" />
       </geometry>
-    </visual>
-    <collision>
+    </visual> </xacro:unless>
+    <xacro:unless value="${disable_mesh}"> <collision>
       <origin xyz="0 0 0" rpy="0 -0 0"/>
       <geometry>
         <mesh filename="package://aero_description/meshes/aero_upper_meshes/RARM_LINK1_mesh.dae" scale="1 1 1" />
       </geometry>
-    </collision>
+    </collision> </xacro:unless>
     <inertial>
       <mass value="0.242" />
@@ -424,16 +424,16 @@
   </gazebo>
   <link name="r_shoulder_center">
-    <visual>
+    <xacro:unless value="${disable_mesh}"> <visual>
       <origin xyz="0 0 0" rpy="0 -0 0"/>
       <geometry>
         <mesh filename="package://aero_description/meshes/aero_upper_meshes/RARM_LINK2_mesh.dae" scale="1 1 1" />
       </geometry>
-    </visual>
-    <collision>
+    </visual> </xacro:unless>
+    <xacro:unless value="${disable_mesh}"> <collision>
       <origin xyz="0 0 0" rpy="0 -0 0"/>
       <geometry>
         <mesh filename="package://aero_description/meshes/aero_upper_meshes/RARM_LINK2_mesh.dae" scale="1 1 1" />
       </geometry>
-    </collision>
+    </collision> </xacro:unless>
     <inertial>
       <mass value="0.744" />
@@ -447,16 +447,16 @@
   </gazebo>
   <link name="r_upperarm_link">
-    <visual>
+    <xacro:unless value="${disable_mesh}"> <visual>
       <origin xyz="0 0 0" rpy="0 -0 0"/>
       <geometry>
         <mesh filename="package://aero_description/meshes/aero_upper_meshes/RARM_LINK3_mesh.dae" scale="1 1 1" />
       </geometry>
-    </visual>
-    <collision>
+    </visual> </xacro:unless>
+    <xacro:unless value="${disable_mesh}"> <collision>
       <origin xyz="0 0 0" rpy="0 -0 0"/>
       <geometry>
         <mesh filename="package://aero_description/meshes/aero_upper_meshes/RARM_LINK3_mesh.dae" scale="1 1 1" />
       </geometry>
-    </collision>
+    </collision> </xacro:unless>
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