Commit message: remove mesh to avoid long loading time

File: aero_description/typeF/robots/aero_moveit_ik.urdf.xacro (robot description, xacro)
@@ -18,4 +18,4 @@
     <origin xyz="0.0 0.0 0.0" rpy="0 0 0 "/>
   </joint>
-  <xacro:aero-wheels base_link="base_link" virtual_lifter="true" x_max="-0.2" x_min="0.2" z_max="0.0" z_min="-0.4"/>
+  <xacro:aero-wheels base_link="base_link" virtual_lifter="true" x_max="-0.2" x_min="0.2" z_max="0.0" z_min="-0.4" disable_mesh="true"/>
 </robot>

File: aero_description/typeF/robots/aero_moveit_ik_ho.urdf.xacro (robot description, xacro)
@@ -18,4 +18,4 @@
     <origin xyz="0.0 0.0 0.0" rpy="0 0 0 "/>
   </joint>
-  <xacro:aero-wheels base_link="base_link" virtual_lifter="true" x_max="0.0" x_min="-0.0" z_max="0.0" z_min="-0.4"/>
+  <xacro:aero-wheels base_link="base_link" virtual_lifter="true" x_max="0.0" x_min="-0.0" z_max="0.0" z_min="-0.4" disable_mesh="true"/>
 </robot>

File: aero_description/typeF/robots/aero_moveit_ik_op.urdf.xacro (robot description, xacro)
@@ -18,4 +18,4 @@
     <origin xyz="0.0 0.0 0.0" rpy="0 0 0 "/>
   </joint>
-  <xacro:aero-wheels base_link="base_link" virtual_lifter="true" x_max="0.17" x_min="-0.17" z_max="-0.08" z_min="-0.25"/>
+  <xacro:aero-wheels base_link="base_link" virtual_lifter="true" x_max="0.17" x_min="-0.17" z_max="-0.08" z_min="-0.25" disable_mesh="true"/>
 </robot>

File: aero_description/typeF/urdf/aero-wheels/aero-wheels.urdf.xacro (robot description, xacro)
@@ -18,6 +18,6 @@
   <xacro:include filename="$(find aero_description)/urdf/aero-wheels/virtual_lifter.urdf.xacro" />
   <xacro:include filename="$(find aero_description)/urdf/common.xacro" />
-  <xacro:macro name="aero-wheels" params="base_link virtual_lifter:=false x_max:=0.0 x_min:=0.0 z_max:=0.0 z_min:=0.0">
-    <xacro:wheels base_link="${base_link}"/>
+  <xacro:macro name="aero-wheels" params="base_link virtual_lifter:=false x_max:=0.0 x_min:=0.0 z_max:=0.0 z_min:=0.0 disable_mesh:=false">
+    <xacro:wheels base_link="${base_link}" disable_mesh="${disable_mesh}"/>
     <joint name="wheel_lifter_connector" type="fixed">
       <parent  link="wheels_top_link"/>

File: aero_description/typeF/urdf/aero-wheels/wheels.urdf.xacro (robot description, xacro)
@@ -15,18 +15,18 @@
        xmlns:xacro="http://ros.org/wiki/xacro">
   <xacro:include filename="$(find aero_description)/urdf/common.xacro" />
-  <xacro:macro name="wheels" params="base_link">
+  <xacro:macro name="wheels" params="base_link disable_mesh:=false">
     <link name="${base_link}">
-      <visual>
+      <xacro:unless value="${disable_mesh}"> <visual>
         <origin xyz="0.0 0.0 0.0" rpy="0 -0 0"/>
         <geometry>
           <mesh filename="package://aero_description/meshes/aero-lower_meshes/wheels_base.dae" scale="1 1 1" />
-        </geometry>
-      </visual>
-      <collision>
+          </geometry>
+      </visual> </xacro:unless>
+      <xacro:unless value="${disable_mesh}"> <collision>
         <origin xyz="0.0 0.0 0.0" rpy="0 -0 0"/>
         <geometry>
           <mesh filename="package://aero_description/meshes/aero-lower_meshes/wheels_base.dae" scale="1 1 1" />
         </geometry>
-      </collision>
+      </collision> </xacro:unless>
       <inertial>
         <mass value="10" />
@@ -40,16 +40,16 @@
     </gazebo>
     <link name="wheels_top_link">
-      <visual>
+      <xacro:unless value="${disable_mesh}"> <visual>
         <origin xyz="0.0 0.0 0.0" rpy="0 -0 0"/>
         <geometry>
           <mesh filename="package://aero_description/meshes/aero-lower_meshes/wheels_top.dae" scale="1 1 1" />
         </geometry>
-      </visual>
-      <collision>
+      </visual> </xacro:unless>
+      <xacro:unless value="${disable_mesh}"> <collision>
         <origin xyz="0.0 0.0 0.0" rpy="0 -0 0"/>
         <geometry>
           <mesh filename="package://aero_description/meshes/aero-lower_meshes/wheels_top.dae" scale="1 1 1" />
         </geometry>
-      </collision>
+      </collision> </xacro:unless>
       <inertial>
         <mass value="10" />
@@ -63,16 +63,16 @@
     </gazebo>
     <link name="wheels_front_left_mecanum">
-      <visual>
-        <origin xyz="0.0 0.0 0.0" rpy="-1.57079632679 0 0"/>
-        <geometry>
-          <mesh filename="package://aero_description/meshes/aero-lower_meshes/wheels_mecanum.dae" scale="1 1 1" />
-        </geometry>
-      </visual>
-      <collision>
-        <origin xyz="0.0 0.0 0.0" rpy="0 -0 0"/>
-        <geometry>
-          <mesh filename="package://aero_description/meshes/aero-lower_meshes/wheels_mecanum.dae" scale="1 1 1" />
-        </geometry>
-      </collision>
+      <xacro:unless value="${disable_mesh}"> <visual>
+        <origin xyz="0.0 0.0 0.0" rpy="-1.57079632679 0 0"/>
+        <geometry>
+          <mesh filename="package://aero_description/meshes/aero-lower_meshes/wheels_mecanum.dae" scale="1 1 1" />
+        </geometry>
+      </visual> </xacro:unless>
+      <xacro:unless value="${disable_mesh}"> <collision>
+        <origin xyz="0.0 0.0 0.0" rpy="0 -0 0"/>
+        <geometry>
+          <mesh filename="package://aero_description/meshes/aero-lower_meshes/wheels_mecanum.dae" scale="1 1 1" />
+        </geometry>
+      </collision> </xacro:unless>
       <inertial>
         <mass value="10" />
@@ -86,16 +86,16 @@
     </gazebo>
     <link name="wheels_front_right_mecanum">
-      <visual>
-        <origin xyz="0.0 0.0 0.0" rpy="-1.57079632679 0 0"/>
-        <geometry>
-          <mesh filename="package://aero_description/meshes/aero-lower_meshes/wheels_mecanum.dae" scale="1 1 1" />
-        </geometry>
-      </visual>
-      <collision>
-        <origin xyz="0.0 0.0 0.0" rpy="0 -0 0"/>
-        <geometry>
-          <mesh filename="package://aero_description/meshes/aero-lower_meshes/wheels_mecanum.dae" scale="1 1 1" />
-        </geometry>
-      </collision>
+      <xacro:unless value="${disable_mesh}"> <visual>
+        <origin xyz="0.0 0.0 0.0" rpy="-1.57079632679 0 0"/>
+        <geometry>
+          <mesh filename="package://aero_description/meshes/aero-lower_meshes/wheels_mecanum.dae" scale="1 1 1" />
+        </geometry>
+      </visual> </xacro:unless>
+      <xacro:unless value="${disable_mesh}"> <collision>
+        <origin xyz="0.0 0.0 0.0" rpy="0 -0 0"/>
+        <geometry>
+          <mesh filename="package://aero_description/meshes/aero-lower_meshes/wheels_mecanum.dae" scale="1 1 1" />
+        </geometry>
+      </collision> </xacro:unless>
       <inertial>
         <mass value="10" />
@@ -109,16 +109,16 @@
     </gazebo>
     <link name="wheels_rear_left_mecanum">
-      <visual>
-        <origin xyz="0.0 0.0 0.0" rpy="-1.57079632679 0 0"/>
-        <geometry>
-          <mesh filename="package://aero_description/meshes/aero-lower_meshes/wheels_mecanum.dae" scale="1 1 1" />
-        </geometry>
-      </visual>
-      <collision>
-        <origin xyz="0.0 0.0 0.0" rpy="0 -0 0"/>
-        <geometry>
-          <mesh filename="package://aero_description/meshes/aero-lower_meshes/wheels_mecanum.dae" scale="1 1 1" />
-        </geometry>
-      </collision>
+      <xacro:unless value="${disable_mesh}"> <visual>
+        <origin xyz="0.0 0.0 0.0" rpy="-1.57079632679 0 0"/>
+        <geometry>
+          <mesh filename="package://aero_description/meshes/aero-lower_meshes/wheels_mecanum.dae" scale="1 1 1" />
+        </geometry>
+      </visual> </xacro:unless>
+      <xacro:unless value="${disable_mesh}"> <collision>
+        <origin xyz="0.0 0.0 0.0" rpy="0 -0 0"/>
+        <geometry>
+          <mesh filename="package://aero_description/meshes/aero-lower_meshes/wheels_mecanum.dae" scale="1 1 1" />
+        </geometry>
+      </collision> </xacro:unless>
       <inertial>
         <mass value="10" />
@@ -132,16 +132,16 @@
     </gazebo>
     <link name="wheels_rear_right_mecanum">
-      <visual>
-        <origin xyz="0.0 0.0 0.0" rpy="-1.57079632679 0 0"/>
-        <geometry>
-          <mesh filename="package://aero_description/meshes/aero-lower_meshes/wheels_mecanum.dae" scale="1 1 1" />
-        </geometry>
-      </visual>
-      <collision>
-        <origin xyz="0.0 0.0 0.0" rpy="0 -0 0"/>
-        <geometry>
-          <mesh filename="package://aero_description/meshes/aero-lower_meshes/wheels_mecanum.dae" scale="1 1 1" />
-        </geometry>
-      </collision>
+      <xacro:unless value="${disable_mesh}"> <visual>
+        <origin xyz="0.0 0.0 0.0" rpy="-1.57079632679 0 0"/>
+        <geometry>
+          <mesh filename="package://aero_description/meshes/aero-lower_meshes/wheels_mecanum.dae" scale="1 1 1" />
+        </geometry>
+      </visual> </xacro:unless>
+      <xacro:unless value="${disable_mesh}"> <collision>
+        <origin xyz="0.0 0.0 0.0" rpy="0 -0 0"/>
+        <geometry>
+          <mesh filename="package://aero_description/meshes/aero-lower_meshes/wheels_mecanum.dae" scale="1 1 1" />
+        </geometry>
+      </collision> </xacro:unless>
       <inertial>
         <mass value="10" />
@@ -155,16 +155,16 @@
     </gazebo>
     <link name="wheels_base_laser_link">
-      <visual>
+      <xacro:unless value="${disable_mesh}"> <visual>
         <origin xyz="0.0 0.0 0.0" rpy="0 0 0"/>
         <geometry>
           <mesh filename="package://aero_description/meshes/aero-lower_meshes/wheels_urg.dae" scale="1 1 1" />
         </geometry>
-      </visual>
-      <collision>
+      </visual> </xacro:unless>
+      <xacro:unless value="${disable_mesh}"> <collision>
         <origin xyz="0.0 0.0 0.0" rpy="0 -0 0"/>
         <geometry>
           <mesh filename="package://aero_description/meshes/aero-lower_meshes/wheels_urg.dae" scale="1 1 1" />
         </geometry>
-      </collision>
+      </collision> </xacro:unless>
       <inertial>
         <mass value="10" />

Commit message: fix disable mesh

File: aero_description/typeF/robots/aero_moveit_ik.urdf.xacro (robot description, xacro)
@@ -13,5 +13,5 @@
   <xacro:include filename="$(find aero_description)/urdf/aero-wheels.urdf.xacro" />
  <!-- Now we can start using the macros included above to define the actual robot -->
- <xacro:aero-upper/>
+ <xacro:aero-upper disable_mesh="true"/>
   <xacro:aero-wheels base_link="base_link" virtual_lifter="true" x_max="-0.2" x_min="0.2" z_max="0.0" z_min="-0.4" disable_mesh="true"/>
 </robot>

File: aero_description/typeF/robots/aero_moveit_ik_ho.urdf.xacro (robot description, xacro)
@@ -13,5 +13,5 @@
   <xacro:include filename="$(find aero_description)/urdf/aero-wheels.urdf.xacro" />
   <!-- Now we can start using the macros included above to define the actual aero -->
-  <xacro:aero-upper/>
+  <xacro:aero-upper disable_mesh="true"/>
   <xacro:aero-wheels base_link="base_link" virtual_lifter="true" x_max="0.0" x_min="-0.0" z_max="0.0" z_min="-0.4" disable_mesh="true"/>
 </robot>

File: aero_description/typeF/robots/aero_moveit_ik_op.urdf.xacro (robot description, xacro)
@@ -13,5 +13,5 @@
   <xacro:include filename="$(find aero_description)/urdf/aero-wheels.urdf.xacro" />
  <!-- Now we can start using the macros included above to define the actual robot -->
- <xacro:aero-upper/>
+ <xacro:aero-upper disable_mesh="true"/>
  <xacro:aero-wheels base_link="base_link" virtual_lifter="true" x_max="0.17" x_min="-0.17" z_max="-0.08" z_min="-0.25" disable_mesh="true"/>
 </robot>

File: aero_description/typeF/urdf/aero-upper.urdf.xacro (robot description, xacro)
@@ -17,8 +17,8 @@
   <xacro:include filename="$(find aero_description)/urdf/typeF_upperbody/aero_upper_typef.urdf.xacro" />
   <xacro:include filename="$(find aero_description)/urdf/trx_s/trx_s.urdf.xacro" />
-  <xacro:macro name="aero-upper">
-  <xacro:aero_upper base_link="waist_link" r_hand_link="r_hand_link" l_hand_link="l_hand_link"/>
-  <xacro:trx_s prefix="r" reflect="1"/>
-  <xacro:trx_s prefix="l" reflect="-1"/>
+  <xacro:macro name="aero-upper" params="disable_mesh:=false">
+  <xacro:aero_upper base_link="waist_link" r_hand_link="r_hand_link" l_hand_link="l_hand_link" disable_mesh="${disable_mesh}"/>
+  <xacro:trx_s prefix="r" reflect="1" disable_mesh="${disable_mesh}"/>
+  <xacro:trx_s prefix="l" reflect="-1" disable_mesh="${disable_mesh}"/>
   <joint name="upper_lower_connector" type="fixed">
     <parent link="lifter_top_link"/>
