Commit message: divide urdf and mesh to parts directories

File: aero_description/typeF/robots/aero.urdf.xacro (robot description, xacro)
@@ -6,19 +6,12 @@
        name="AeroUpperRobot" >
   <!-- The following included files set up definitions of parts of the robot body -->
+  <!-- common variables -->
   <xacro:include filename="$(find aero_description)/urdf/common.xacro" />
-  <!-- aero_upper body -->
-  <xacro:include filename="$(find aero_description)/urdf/aero_upper/aero_upper.urdf.xacro" />
-  <!-- aero-lower_body -->
-  <xacro:include filename="$(find aero_description)/urdf/aero-wheels/aero-wheels.urdf.xacro" />
-  <!-- Now we can start using the macros included above to define the actual aero -->
-  <xacro:aero_upper base_link="waist_link"/>
-  <joint name="upper_lower_connector" type="fixed">
-    <parent link="lifter_top_link"/>
-    <child link="waist_link"/>
-    <origin xyz="0.0 0.0 0.0" rpy="0 0 0 "/>
-  </joint>
-  <xacro:aero-wheels base_link="base_link"/>
-    <plugin name="gazebo_ros_control" filename="libgazebo_ros_control.so"/>
-  <gazebo>
-  </gazebo>
+  <!-- wraps upperbody and hand-->
+  <xacro:include filename="$(find aero_description)/urdf/aero-upper.urdf.xacro" />
+  <!-- wraps lifter and wheels-->
+  <xacro:include filename="$(find aero_description)/urdf/aero-wheels.urdf.xacro" />
+ <!-- Now we can start using the macros included above to define the actual robot -->
+ <xacro:aero-upper/>
+ <xacro:aero-wheels base_link="base_link"/>
 </robot>

File: aero_description/typeF/robots/aero_moveit_ik.urdf.xacro (robot description, xacro)
@@ -6,16 +6,12 @@
        name="AeroUpperRobot" >
   <!-- The following included files set up definitions of parts of the robot body -->
+  <!-- common variables -->
   <xacro:include filename="$(find aero_description)/urdf/common.xacro" />
-  <!-- aero_upper body -->
-  <xacro:include filename="$(find aero_description)/urdf/aero_upper/aero_upper.urdf.xacro" />
-  <!-- aero-lower_body -->
-  <xacro:include filename="$(find aero_description)/urdf/aero-wheels/aero-wheels.urdf.xacro" />
-  <!-- Now we can start using the macros included above to define the actual aero -->
-  <xacro:aero_upper base_link="waist_link" disable_mesh="true"/>
-  <joint name="upper_lower_connector" type="fixed">
-    <parent link="lifter_top_link"/>
-    <child link="waist_link"/>
-    <origin xyz="0.0 0.0 0.0" rpy="0 0 0 "/>
-  </joint>
+  <!-- wraps upperbody and hand-->
+  <xacro:include filename="$(find aero_description)/urdf/aero-upper.urdf.xacro" />
+  <!-- wraps lifter and wheels-->
+  <xacro:include filename="$(find aero_description)/urdf/aero-wheels.urdf.xacro" />
+ <!-- Now we can start using the macros included above to define the actual robot -->
+ <xacro:aero-upper/>
   <xacro:aero-wheels base_link="base_link" virtual_lifter="true" x_max="-0.2" x_min="0.2" z_max="0.0" z_min="-0.4" disable_mesh="true"/>
 </robot>

File: aero_description/typeF/robots/aero_moveit_ik_ho.urdf.xacro (robot description, xacro)
@@ -6,16 +6,12 @@
        name="AeroUpperRobot" >
   <!-- The following included files set up definitions of parts of the robot body -->
+  <!-- common variables -->
   <xacro:include filename="$(find aero_description)/urdf/common.xacro" />
-  <!-- aero_upper body -->
-  <xacro:include filename="$(find aero_description)/urdf/aero_upper/aero_upper.urdf.xacro" />
-  <!-- aero-lower_body -->
-  <xacro:include filename="$(find aero_description)/urdf/aero-wheels/aero-wheels.urdf.xacro" />
+  <!-- wraps upperbody and hand-->
+  <xacro:include filename="$(find aero_description)/urdf/aero-upper.urdf.xacro" />
+  <!-- wraps lifter and wheels-->
+  <xacro:include filename="$(find aero_description)/urdf/aero-wheels.urdf.xacro" />
   <!-- Now we can start using the macros included above to define the actual aero -->
-  <xacro:aero_upper base_link="waist_link" disable_mesh="true"/>
-  <joint name="upper_lower_connector" type="fixed">
-    <parent link="lifter_top_link"/>
-    <child link="waist_link"/>
-    <origin xyz="0.0 0.0 0.0" rpy="0 0 0 "/>
-  </joint>
+  <xacro:aero-upper/>
   <xacro:aero-wheels base_link="base_link" virtual_lifter="true" x_max="0.0" x_min="-0.0" z_max="0.0" z_min="-0.4" disable_mesh="true"/>
 </robot>

File: aero_description/typeF/robots/aero_moveit_ik_op.urdf.xacro (robot description, xacro)
@@ -6,16 +6,12 @@
        name="AeroUpperRobot" >
   <!-- The following included files set up definitions of parts of the robot body -->
+  <!-- common variables -->
   <xacro:include filename="$(find aero_description)/urdf/common.xacro" />
-  <!-- aero_upper body -->
-  <xacro:include filename="$(find aero_description)/urdf/aero_upper/aero_upper.urdf.xacro" />
-  <!-- aero-lower_body -->
-  <xacro:include filename="$(find aero_description)/urdf/aero-wheels/aero-wheels.urdf.xacro" />
-  <!-- Now we can start using the macros included above to define the actual aero -->
-  <xacro:aero_upper base_link="waist_link" disable_mesh="true"/>
-  <joint name="upper_lower_connector" type="fixed">
-    <parent link="lifter_top_link"/>
-    <child link="waist_link"/>
-    <origin xyz="0.0 0.0 0.0" rpy="0 0 0 "/>
-  </joint>
-  <xacro:aero-wheels base_link="base_link" virtual_lifter="true" x_max="0.17" x_min="-0.17" z_max="-0.08" z_min="-0.25" disable_mesh="true"/>
+  <!-- wraps upperbody and hand-->
+  <xacro:include filename="$(find aero_description)/urdf/aero-upper.urdf.xacro" />
+  <!-- wraps lifter and wheels-->
+  <xacro:include filename="$(find aero_description)/urdf/aero-wheels.urdf.xacro" />
+ <!-- Now we can start using the macros included above to define the actual robot -->
+ <xacro:aero-upper/>
+ <xacro:aero-wheels base_link="base_link" virtual_lifter="true" x_max="0.17" x_min="-0.17" z_max="-0.08" z_min="-0.25" disable_mesh="true"/>
 </robot>

Commit message: [aero_shop] fix urdf for using in gazebo for typeF, there is no effect to real robot

File: aero_description/typeF/robots/aero.urdf.xacro (robot description, xacro)
@@ -15,3 +15,5 @@
  <xacro:aero-upper/>
  <xacro:aero-wheels base_link="base_link"/>
+ <xacro:gazebo_trajectory_controller />
+ <xacro:gazebo_base_controller base_frame="base_link" />
 </robot>

File: aero_shop/trx_s/urdf/trx_s.urdf.xacro (robot description, xacro)
@@ -19,10 +19,18 @@
       </geometry>
     </visual> </xacro:unless>
-    <xacro:unless value="${disable_mesh}"> <collision>
-      <origin xyz="0 0 0" rpy="0 -0 ${(1.0 - reflect) * M_PI / 2.0}"/>
+    <xacro:unless value="${disable_mesh}">
+    <collision>
+      <origin rpy="${reflect * 0.7} 0 0" xyz="0 0 -0.093"/>
       <geometry>
-        <mesh filename="package://aero_description/meshes/trx_s/RARM_LINK7_mesh.dae" scale="1 1 1" />
+        <box size="0.036 0.070 0.030" />
       </geometry>
-    </collision> </xacro:unless>
+    </collision>
+    <collision>
+      <origin rpy="${reflect * -0.10} 0 0" xyz="0 ${reflect * -0.007} -0.055"/>
+      <geometry>
+        <box size="0.036 0.050 0.070" />
+      </geometry>
+    </collision>
+    </xacro:unless>
     <inertial>
       <mass value="0.183" />
@@ -40,16 +48,16 @@
     </visual> </xacro:unless>
     <xacro:unless value="${disable_mesh}"> <collision>
-      <origin xyz="0 ${0.013 * reflect} 0.115" rpy="0 -0 ${(1.0 - reflect) * M_PI / 2.0}"/>
+      <origin xyz="0 ${reflect * 0.013494 } -0.021422" rpy="${reflect * -0.85} 0 0"/>
       <geometry>
-        <mesh filename="package://aero_description/meshes/trx_s/RARM_INDEX_LINK1_mesh.dae" scale="1 1 1" />
+        <box size="0.041 0.061 0.016" />  <!-- 0.85 -->
       </geometry>
     </collision> </xacro:unless>
     <inertial>
-      <mass value="0" />
-      <origin xyz="0 0 0" rpy="0 -0 0"/>
-      <inertia ixx="0" ixy="0" ixz="0" iyy="0" iyz="0" izz="0"/>
+      <mass value="0.1" />
+      <origin xyz="0 ${reflect * 0.014} -0.021" rpy="0 0 0"/>
+      <inertia ixx="0.001" iyy="0.0001" izz="0.0001" ixy="0" ixz="0" iyz="0" />
     </inertial>
   </link>
-  <xacro:gazebo_link_reference link_name="${prefix}_indexthumb_link" />
+  <xacro:gazebo_link_reference link_name="${prefix}_indexbase_link" />
   <link name="${prefix}_indexmid_link">
     <xacro:unless value="${disable_mesh}"> <visual>
@@ -60,13 +68,13 @@
     </visual> </xacro:unless>
     <xacro:unless value="${disable_mesh}"> <collision>
-      <origin xyz="0 ${-0.015754 * reflect} 0.149615" rpy="0 -0 ${(1.0 - reflect) * M_PI / 2.0}"/>
+      <origin xyz="0 ${reflect * 0.014} -0.008" rpy="${reflect * -0.3} 0 0"/> <!-- 0.3 -->
       <geometry>
-        <mesh filename="package://aero_description/meshes/trx_s/RARM_INDEX_LINK2_mesh.dae" scale="1 1 1" />
+        <box size="0.034 0.030 0.016" />
       </geometry>
     </collision> </xacro:unless>
     <inertial>
-      <mass value="0" />
-      <origin xyz="0 0 0" rpy="0 -0 0"/>
-      <inertia ixx="0" ixy="0" ixz="0" iyy="0" iyz="0" izz="0"/>
+      <mass value="0.1" />
+      <origin xyz="0 ${reflect * 0.014} -0.008" rpy="0 0 0"/>
+      <inertia ixx="0.001" iyy="0.0001" izz="0.0001" ixy="0" ixz="0" iyz="0" />
     </inertial>
   </link>
@@ -80,13 +88,13 @@
     </visual> </xacro:unless>
     <xacro:unless value="${disable_mesh}"> <collision>
-      <origin xyz="0 ${-0.03747 * reflect} 0.162972" rpy="0 -0 ${(1.0 - reflect) * M_PI / 2.0}"/>
+      <origin xyz="0 ${reflect * 0.013} 0.004" rpy="0 0 0"/> <!-- 0.0 -->
       <geometry>
-        <mesh filename="package://aero_description/meshes/trx_s/RARM_INDEX_LINK3_mesh.dae" scale="1 1 1" />
+        <box size="0.040 0.028 0.016" />
       </geometry>
     </collision> </xacro:unless>
     <inertial>
-      <mass value="0" />
-      <origin xyz="0 0 0" rpy="0 -0 0"/>
-      <inertia ixx="0" ixy="0" ixz="0" iyy="0" iyz="0" izz="0"/>
+      <mass value="0.1" />
+      <origin xyz="0 ${reflect * 0.02} 0" rpy="0 0 0"/>
+      <inertia ixx="0.0001" iyy="0.0001" izz="0.0001" ixy="0" ixz="0" iyz="0" />
     </inertial>
   </link>
@@ -99,14 +107,22 @@
       </geometry>
     </visual> </xacro:unless>
-    <xacro:unless value="${disable_mesh}"> <collision>
-      <origin xyz="0 ${-0.022355 * reflect} 0.079645" rpy="0 -0 ${(1.0 - reflect) * M_PI / 2.0}"/>
+    <xacro:unless value="${disable_mesh}">
+    <collision>
+      <origin rpy="0.63 0 0" xyz="0.0 ${reflect * 0.019645} -0.010355"/>
       <geometry>
-        <mesh filename="package://aero_description/meshes/trx_s/RARM_THUMB_LINK_mesh.dae" scale="1 1 1" />
+        <box size="0.012 0.008 0.050"/>
       </geometry>
-    </collision> </xacro:unless>
+    </collision>
+    <collision>
+      <origin rpy="0.1 0 0" xyz="0.0 ${reflect * 0.035645} -0.050355"/>
+      <geometry>
+        <box size="0.012 0.008 0.050"/>
+      </geometry>
+    </collision>
+    </xacro:unless>
     <inertial>
-      <mass value="0" />
-      <origin xyz="0 0 0" rpy="0 -0 0"/>
-      <inertia ixx="0" ixy="0" ixz="0" iyy="0" iyz="0" izz="0"/>
+      <mass value="0.1" />
+      <origin xyz="0 ${reflect * 0.05} -0.06" rpy="0 0 0"/>
+      <inertia ixx="0.001" iyy="0.0001" izz="0.0001" ixy="0" ixz="0" iyz="0" />
     </inertial>
   </link>
@@ -120,5 +136,5 @@
     <dynamics damping="0.2" friction="0" />
   </joint>
-  <xacro:gazebo_transmission joint_name="${prefix}_indexbase_joint" />
+  <xacro:gazebo_joint_reference joint_name="${prefix}_indexbase_joint" />
   <joint name="${prefix}_indexmid_joint" type="revolute">
     <parent link="${prefix}_indexbase_link"/>
@@ -129,5 +145,5 @@
     <dynamics damping="0.2" friction="0" />
   </joint>
-  <xacro:gazebo_transmission joint_name="${prefix}_indexmid_joint" />
+  <xacro:gazebo_joint_reference joint_name="${prefix}_indexmid_joint" />
   <joint name="${prefix}_indexend_joint" type="revolute">
     <parent link="${prefix}_indexmid_link"/>
@@ -138,5 +154,5 @@
     <dynamics damping="0.2" friction="0" />
   </joint>
-  <xacro:gazebo_transmission joint_name="${prefix}_indexend_joint" />
+  <xacro:gazebo_joint_reference joint_name="${prefix}_indexend_joint" />
   <joint name="${prefix}_thumb_joint" type="revolute">
     <parent link="${prefix}_hand_link"/>

File: aero_shop/typeC_lifter/urdf/lifter.urdf.xacro (robot description, xacro)
@@ -15,4 +15,5 @@
        xmlns:xacro="http://ros.org/wiki/xacro">
   <xacro:include filename="$(find aero_description)/urdf/common.xacro" />
+  <xacro:include filename="$(find aero_description)/common_urdf/gazebo.xacro" />
   <xacro:macro name="lifter" params="base_link">
     <link name="${base_link}">
@@ -35,8 +36,5 @@
       </inertial>
     </link>
-    <gazebo reference="${base_link}">
-      <mu1>0.9</mu1>
-      <mu2>0.9</mu2>
-    </gazebo>
+    <xacro:gazebo_link_reference link_name="${base_link}" />
     <link name="leg_shank_link">
       <visual>
@@ -47,5 +45,5 @@
       </visual>
       <collision>
-        <origin xyz="0.0 0.0 0.0" rpy="0 -0 0"/>
+        <origin xyz="0.0 0.0 0" rpy="3.1415 -0 0"/>
         <geometry>
           <mesh filename="package://aero_description/meshes/typeC_lifter/lifter_bone.dae" scale="1 1 1" />
@@ -58,8 +56,5 @@
       </inertial>
     </link>
-    <gazebo reference="leg_shank_link">
-      <mu1>0.9</mu1>
-      <mu2>0.9</mu2>
-    </gazebo>
+    <xacro:gazebo_link_reference link_name="leg_shank_link" />
     <link name="leg_knee_link">
       <visual>
@@ -70,5 +65,5 @@
       </visual>
       <collision>
-        <origin xyz="0.0 0.0 0.0" rpy="0 -0 0"/>
+        <origin xyz="0.0 0.0 0" rpy="3.1415 -0 0"/>
         <geometry>
           <mesh filename="package://aero_description/meshes/typeC_lifter/lifter_knee.dae" scale="1 1 1" />
@@ -81,8 +76,5 @@
       </inertial>
     </link>
-    <gazebo reference="leg_knee_link">
-      <mu1>0.9</mu1>
-      <mu2>0.9</mu2>
-    </gazebo>
+    <xacro:gazebo_link_reference link_name="leg_knee_link" />
     <link name="leg_thigh_link">
       <visual>
@@ -93,5 +85,5 @@
       </visual>
       <collision>
-        <origin xyz="0.0 0.0 0.0" rpy="0 -0 0"/>
+        <origin xyz="0 0 0.25" rpy="0 0 0"/>
         <geometry>
           <mesh filename="package://aero_description/meshes/typeC_lifter/lifter_bone.dae" scale="1 1 1" />
@@ -104,8 +96,5 @@
       </inertial>
     </link>
-    <gazebo reference="leg_thigh_link">
-      <mu1>0.9</mu1>
-      <mu2>0.9</mu2>
-    </gazebo>
+    <xacro:gazebo_link_reference link_name="leg_thigh_link" />
     <link name="leg_base_link">
       <visual>
@@ -116,5 +105,5 @@
       </visual>
       <collision>
-        <origin xyz="0 0 0" rpy="0 -0 0"/>
+        <origin xyz="0 0 0.05" rpy="3.1415920 0 0"/>
         <geometry>
           <mesh filename="package://aero_description/meshes/typeC_lifter/lifter_base.dae" scale="1 1 1" />
@@ -127,8 +116,5 @@
       </inertial>
     </link>
-    <gazebo reference="leg_base_link">
-      <mu1>0.9</mu1>
-      <mu2>0.9</mu2>
-    </gazebo>
+    <xacro:gazebo_link_reference link_name="leg_base_link" />
     <link name="lifter_top_link">
       <visual>
@@ -150,8 +136,5 @@
       </inertial>
     </link>
-    <gazebo reference="lifter_top_link">
-      <mu1>0.9</mu1>
-      <mu2>0.9</mu2>
-    </gazebo>
+    <xacro:gazebo_link_reference link_name="lifter_top_link" />
     <joint name="lifter_top_connector" type="fixed">
       <parent link="leg_base_link"/>
@@ -171,14 +154,7 @@
       <origin xyz="0 0 0.12" rpy="0 0 0"/>
       <axis xyz="0 -1 0"/>
-      <limit effort="100" lower="-1.5707" upper="0" velocity="0.5"/>
-    </joint>
-    <transmission type="pr2_mechanism_model/SimpleTransmission" name="knee_joint_trans" >
-      <actuator name="knee_joint_motor" />
-      <joint name="knee_joint" />
-      <mechanicalReduction>1</mechanicalReduction>
-    </transmission>
-    <gazebo reference="knee_joint">
-      <implicitSpringDamper>0.4</implicitSpringDamper>
-    </gazebo>
+      <limit effort="1000" lower="-1.5707" upper="0" velocity="0.5"/>
+    </joint>
+    <xacro:gazebo_transmission joint_name="knee_joint" />
     <joint name="ankle_joint" type="revolute">
       <parent link="${base_link}"/>
@@ -186,15 +162,8 @@
       <origin xyz="0 0 0.05" rpy="0 0 0"/>
       <axis   xyz="0 -1 0"/>
-      <limit lower="0" upper="1.5707" effort="100" velocity="0.5" />
+      <limit effort="1000" lower="0" upper="1.5707" velocity="0.5" />
       <dynamics damping="0.2" friction="0" />
     </joint>
-    <transmission type="pr2_mechanism_model/SimpleTransmission" name="ankle_joint_trans" >
-      <actuator name="ankle_joint_motor" />
-      <joint name="ankle_joint" />
-      <mechanicalReduction>1</mechanicalReduction>
-    </transmission>
-    <gazebo reference="ankle_joint">
-      <implicitSpringDamper>0.4</implicitSpringDamper>
-    </gazebo>
+    <xacro:gazebo_transmission joint_name="ankle_joint" />
 <!--- mimic joints -->
 <!-- requried -->
@@ -214,4 +183,9 @@
         <origin xyz="0 0 0.25" rpy="0 0 0"/>
       </visual>
+      <inertial> <!-- for gazebo visualization -->
+        <mass value="0.4"/>
+        <origin rpy="0 0 0" xyz="-0.04 0.0 0.14"/>
+        <inertia ixx="0.001" ixy="0" ixz="0" iyy="0.001" iyz="0" izz="0.001"/>
+      </inertial>
     </link>
     <link name="leg_thigh_link_dummy">
@@ -222,4 +196,9 @@
         <origin xyz="0 0 0.25" rpy="0 0 0"/>
       </visual>
+      <inertial> <!-- for gazebo visualization -->
+        <mass value="0.4"/>
+        <origin rpy="0 0 0" xyz="-0.04 0.0 0.14"/>
+        <inertia ixx="0.001" ixy="0" ixz="0" iyy="0.001" iyz="0" izz="0.001"/>
+      </inertial>
     </link>
     <joint name="ankle_joint_dummy" type="continuous">

File: aero_shop/typeD_wheel/urdf/wheels.urdf.xacro (robot description, xacro)
@@ -150,7 +150,7 @@
       </visual> </xacro:unless>
       <xacro:unless value="${disable_mesh}"> <collision>
-        <origin xyz="0.0 0.0 0.0" rpy="0 -0 0"/>
-        <geometry>
-          <mesh filename="package://aero_description/meshes/typeD_wheel/wheels_urg.dae" scale="1 1 1" />
+        <origin xyz="0.0 0.0 -0.0124" rpy="0 -0 0"/>
+        <geometry>
+          <box size="0.08 0.1 0.07" />
         </geometry>
       </collision> </xacro:unless>
