Commit message: update settings for gazebo

File: aero_description/typeF/robots/aero.urdf.xacro (robot description, xacro)
@@ -28,9 +28,9 @@
             command_max="200" command_min="-200"> ankle_joint_dummy</mimic>
      <mimic joint="knee_joint"  offset="0.0" multiplier="-1.0"
-            P="3000" I="0.0" D="3" i_max="0" i_min="0"
-            command_max="1000" command_min="-1000"> knee_joint_mimic</mimic>
+            P="4000" I="0.1" D="80" i_max="500" i_min="-500"
+            command_max="2000" command_min="-2000"> knee_joint_mimic</mimic>
      <mimic joint="ankle_joint"  offset="0.0" multiplier="-1.0"
-            P="3000" I="0.0" D="3" i_max="0" i_min="0"
-            command_max="1000" command_min="-1000"> ankle_joint_mimic</mimic>
+            P="4000" I="0.1" D="80" i_max="500" i_min="-500"
+            command_max="2000" command_min="-2000"> ankle_joint_mimic</mimic>
      <!-- lhand -->
      <mimic joint="l_thumb_joint"  offset="0.0" multiplier="-1.0"

File: aero_shop/typeB_lifter/urdf/lifter.urdf.xacro (robot description, xacro)
@@ -53,5 +53,6 @@
       <inertial>
         <mass value="2.06679" />
-        <origin xyz="0.081713 0.000812 -0.146934" rpy="0 -0 0"/>
+        <!--origin xyz="0.081713 0.000812 -0.146934" rpy="0 -0 0"/-->
+        <origin xyz="0.051713 0.000812 0.146934" rpy="0 -0 0"/>
         <inertia ixx="0.0408818" ixy="-9.39301e-06" ixz="-0.000750165" iyy="0.0403969" iyz="-0.000120419" izz="0.00260982"/>
       </inertial>
@@ -73,5 +74,6 @@
       <inertial>
         <mass value="2.06679" />
-        <origin xyz="0.081713 0.000812 -0.146934" rpy="0 -0 0"/>
+        <!--origin xyz="0.081713 0.000812 -0.146934" rpy="0 -0 0"/-->
+        <origin xyz="0.031713 0.000812 0.046934" rpy="0 -0 0"/>
         <inertia ixx="0.0408818" ixy="-9.39301e-06" ixz="-0.000750165" iyy="0.0403969" iyz="-0.000120419" izz="0.00260982"/>
       </inertial>
@@ -93,5 +95,6 @@
       <inertial>
         <mass value="2.62321" />
-        <origin xyz="0.0587169 0 -0.135292" rpy="0 -0 0"/>
+        <!--origin xyz="0.0587169 0 -0.135292" rpy="0 -0 0"/-->
+        <origin xyz="0.0587169 0 0.135292" rpy="0 -0 0"/>
         <inertia ixx="0.0161595" ixy="-9.27234e-05" ixz="0.00262839" iyy="0.0166415" iyz="-0.00017447" izz="0.00477281"/>
       </inertial>
@@ -131,9 +134,10 @@
         </geometry>
       </collision>
-      <inertial>
+      <!-- same value as base?? -->
+      <!--inertial>
         <mass value="7.64604" />
         <origin xyz="-0.012819 -0.002679 0.007207" rpy="0 -0 0"/>
         <inertia ixx="0.0658136" ixy="-0.000159462" ixz="0.010103" iyy="0.0504268" iyz="0.000173435" izz="0.0889772"/>
-      </inertial>
+      </inertial-->
     </link>
     <xacro:gazebo_link_reference link_name="lifter_top_link" />
@@ -155,5 +159,5 @@
       <origin xyz="0 0 0.12" rpy="0 0 0"/>
       <axis xyz="0 -1 0"/>
-      <limit effort="1000" lower="-1.5707" upper="0" velocity="0.5"/>
+      <limit effort="10000" lower="-1.5707" upper="0" velocity="0.5"/>
     </joint>
     <xacro:gazebo_transmission joint_name="knee_joint" />

File: aero_shop/typeC_lifter/urdf/lifter.urdf.xacro (robot description, xacro)
@@ -53,6 +53,8 @@
       <inertial>
         <mass value="2.06679" />
-        <origin xyz="0.081713 0.000812 -0.146934" rpy="0 -0 0"/>
-        <inertia ixx="0.0408818" ixy="-9.39301e-06" ixz="-0.000750165" iyy="0.0403969" iyz="-0.000120419" izz="0.00260982"/>
+        <!--origin xyz="0.081713 0.000812 -0.146934" rpy="0 -0 0"/-->
+        <origin xyz="0.051713 0.0 0.146934" rpy="0 -0 0"/>
+        <!--inertia ixx="0.0408818" ixy="-9.39301e-06" ixz="-0.000750165" iyy="0.0403969" iyz="-0.000120419" izz="0.00260982"/-->
+        <inertia ixx="0.06" ixy="0.0" ixz="0.0" iyy="0.1" iyz="0.0" izz="0.06"/>
       </inertial>
     </link>
@@ -73,6 +75,8 @@
       <inertial>
         <mass value="2.06679" />
-        <origin xyz="0.081713 0.000812 -0.146934" rpy="0 -0 0"/>
-        <inertia ixx="0.0408818" ixy="-9.39301e-06" ixz="-0.000750165" iyy="0.0403969" iyz="-0.000120419" izz="0.00260982"/>
+        <!--origin xyz="0.081713 0.000812 -0.146934" rpy="0 -0 0"/-->
+        <origin xyz="-0.031713 0.0 0.046934" rpy="0 -0 0"/>
+        <!--inertia ixx="0.0408818" ixy="-9.39301e-06" ixz="-0.000750165" iyy="0.0403969" iyz="-0.000120419" izz="0.00260982"/-->
+        <inertia ixx="0.06" ixy="0.0" ixz="0.0" iyy="0.1" iyz="0.0" izz="0.06"/>
       </inertial>
     </link>
@@ -93,5 +97,6 @@
       <inertial>
         <mass value="2.62321" />
-        <origin xyz="0.0587169 0 -0.135292" rpy="0 -0 0"/>
+        <!--origin xyz="0.0587169 0 -0.135292" rpy="0 -0 0"/-->
+        <origin xyz="-0.0587169 0 0.135292" rpy="0 -0 0"/>
         <inertia ixx="0.0161595" ixy="-9.27234e-05" ixz="0.00262839" iyy="0.0166415" iyz="-0.00017447" izz="0.00477281"/>
       </inertial>
@@ -132,7 +137,7 @@
       </collision>
       <inertial>
-        <mass value="7.64604" />
-        <origin xyz="-0.012819 -0.002679 0.007207" rpy="0 -0 0"/>
-        <inertia ixx="0.0658136" ixy="-0.000159462" ixz="0.010103" iyy="0.0504268" iyz="0.000173435" izz="0.0889772"/>
+        <mass value="1.0" />
+        <origin xyz="0.0 0.0 0.0" rpy="0 0 0"/>
+        <inertia ixx="0.03" ixy="0.0" ixz="0.0" iyy="0.03" iyz="0.0" izz="0.04"/>
       </inertial>
     </link>
@@ -155,5 +160,5 @@
       <origin xyz="0 0 0.12" rpy="0 0 0"/>
       <axis xyz="0 -1 0"/>
-      <limit effort="1000" lower="-1.5707" upper="0" velocity="0.5"/>
+      <limit effort="10000" lower="-1.5707" upper="0" velocity="1.5"/>
     </joint>
     <xacro:gazebo_transmission joint_name="knee_joint" />
@@ -163,5 +168,5 @@
       <origin xyz="0 0 0.05" rpy="0 0 0"/>
       <axis   xyz="0 -1 0"/>
-      <limit effort="1000" lower="0" upper="1.5707" velocity="0.5" />
+      <limit effort="4000" lower="0" upper="1.5707" velocity="1.5" />
       <dynamics damping="0.2" friction="0" />
     </joint>

File: aero_shop/typeD_wheel/urdf/wheels.urdf.xacro (robot description, xacro)
@@ -38,6 +38,6 @@
       </collision> </xacro:unless>
       <inertial>
-        <mass value="10" />
-        <origin xyz="0 0 0" rpy="0 -0 0.09"/>
+        <mass value="70" />
+        <origin xyz="0 0 0.04" rpy="0 -0 0.0"/>
         <inertia ixx="0.528" ixy="0" ixz="0" iyy="2.02" iyz="0" izz="2.35"/>
       </inertial>
@@ -53,5 +53,5 @@
       <!-- no collision geometry -->
       <inertial>
-        <mass value="10" />
+        <mass value="1" />
         <origin xyz="0 0 0" rpy="0 -0 0"/>
         <inertia ixx="0.528" ixy="0" ixz="0" iyy="2.02" iyz="0" izz="2.35"/>
@@ -74,5 +74,5 @@
       </collision> </xacro:unless>
       <inertial>
-        <mass value="10" />
+        <mass value="1" />
         <origin xyz="0 0 0" rpy="0 -0 0"/>
         <inertia ixx="0.528" ixy="0" ixz="0" iyy="2.02" iyz="0" izz="2.35"/>
@@ -95,5 +95,5 @@
       </collision> </xacro:unless>
       <inertial>
-        <mass value="10" />
+        <mass value="1" />
         <origin xyz="0 0 0" rpy="0 -0 0"/>
         <inertia ixx="0.528" ixy="0" ixz="0" iyy="2.02" iyz="0" izz="2.35"/>
@@ -116,5 +116,5 @@
       </collision> </xacro:unless>
       <inertial>
-        <mass value="10" />
+        <mass value="1" />
         <origin xyz="0 0 0" rpy="0 -0 0"/>
         <inertia ixx="0.528" ixy="0" ixz="0" iyy="2.02" iyz="0" izz="2.35"/>
@@ -137,5 +137,5 @@
       </collision> </xacro:unless>
       <inertial>
-        <mass value="10" />
+        <mass value="1" />
         <origin xyz="0 0 0" rpy="0 -0 0"/>
         <inertia ixx="0.528" ixy="0" ixz="0" iyy="2.02" iyz="0" izz="2.35"/>
@@ -157,7 +157,7 @@
       </collision> </xacro:unless>
       <inertial>
-        <mass value="10" />
-        <origin xyz="0 0 0" rpy="0 -0 0"/>
-        <inertia ixx="0.528" ixy="0" ixz="0" iyy="2.02" iyz="0" izz="2.35"/>
+        <mass value="0.2" />
+        <origin xyz="0 0 0" rpy="0 -0 0"/>
+        <inertia ixx="0.0528" ixy="0" ixz="0" iyy="0.0202" iyz="0" izz="0.0235"/>
       </inertial>
     </link>

File: aero_shop/typeF_upperbody/urdf/aero_upper_typef.urdf.xacro (robot description, xacro)
@@ -26,5 +26,5 @@
       <mass value="1.257" />
       <origin xyz="0 0 0.0" rpy="0 -0 0"/>
-      <inertia ixx="0.0034" ixy="0" ixz="0" iyy="0.0036" iyz="0" izz="0.0017"/>
+      <inertia ixx="0.034" ixy="0" ixz="0" iyy="0.034" iyz="0" izz="0.018"/>
     </inertial>
   </link>
@@ -46,5 +46,5 @@
       <mass value="1.257" />
       <origin xyz="0 0 0.042" rpy="0 -0 0"/>
-      <inertia ixx="0.0034" ixy="0" ixz="0" iyy="0.0036" iyz="0" izz="0.0017"/>
+      <inertia ixx="0.034" ixy="0" ixz="0" iyy="0.034" iyz="0" izz="0.018"/>
     </inertial>
   </link>
@@ -52,5 +52,5 @@
   <link name="hip_center">
     <inertial>
-      <mass value="0.01" />
+      <mass value="0.1" />
       <origin xyz="0 0 0" rpy="0 -0 0"/>
       <inertia ixx="0.01" ixy="0" ixz="0" iyy="0.01" iyz="0" izz="0.01"/>
@@ -137,5 +137,5 @@
       <!-- fix for gazebo -->
       <origin xyz="0.005 0 -0.0654" rpy="0 -0 0"/>
-      <inertia ixx="0.00114" ixy="0" ixz="0" iyy="0.00117" iyz="0" izz="0.003"/>
+      <inertia ixx="0.00214" ixy="0" ixz="0" iyy="0.00217" iyz="0" izz="0.003"/>
     </inertial>
   </link>
@@ -160,5 +160,5 @@
       <!-- fix for gazebo -->
       <origin xyz="-0.03 0 -0.0546" rpy="0 -0 0"/>
-      <inertia ixx="0.00178" ixy="0" ixz="0" iyy="0.00179" iyz="0" izz="0.004"/>
+      <inertia ixx="0.00178" ixy="0" ixz="0" iyy="0.00179" iyz="0" izz="0.0035"/>
     </inertial>
   </link>
@@ -180,5 +180,5 @@
       <mass value="0.132" />
       <origin xyz="0.006 0 -0.0738" rpy="0 -0 0"/>
-      <inertia ixx="0.000276" ixy="0" ixz="0" iyy="0.000286" iyz="0" izz="0.004"/>
+      <inertia ixx="0.00276" ixy="0" ixz="0" iyy="0.00286" iyz="0" izz="0.004"/>
     </inertial>
   </link>
@@ -209,5 +209,5 @@
       <origin xyz="0 0 0.0595" rpy="0 -0 0"/>
       <!--inertia ixx="1.64186e-35" ixy="0" ixz="0" iyy="1.64186e-35" iyz="0" izz="0"/-->
-      <inertia ixx="0.0001" ixy="0" ixz="0" iyy="0.0001" iyz="0" izz="0.001"/>
+      <inertia ixx="0.001" ixy="0" ixz="0" iyy="0.001" iyz="0" izz="0.002"/>
     </inertial>
   </link>
@@ -227,7 +227,7 @@
     </collision> </xacro:unless>
     <inertial>
-      <mass value="0.01" />
-      <origin xyz="0 0 0" rpy="0 -0 0"/>
-      <inertia ixx="0.0001" ixy="0" ixz="0" iyy="0.0001" iyz="0" izz="0.0001"/>
+      <mass value="0.1" />
+      <origin xyz="0 0 0" rpy="0 -0 0"/>
+      <inertia ixx="0.0005" ixy="0" ixz="0" iyy="0.0005" iyz="0" izz="0.0005"/>
     </inertial>
   </link>
@@ -248,5 +248,5 @@
     <inertial>
       <mass value="0.974" />
-      <origin xyz="0 0 0.150" rpy="0 -0 0"/>
+      <origin xyz="0.01 0 0.070" rpy="0 -0 0"/>
       <inertia ixx="0.005" ixy="0" ixz="0" iyy="0.005" iyz="0" izz="0.005"/>
     </inertial>
@@ -312,5 +312,5 @@
       <!-- fix for gazebo -->
       <origin xyz="0.005 0 -0.0654" rpy="0 -0 0"/>
-      <inertia ixx="0.00114" ixy="0" ixz="0" iyy="0.00117" iyz="0" izz="0.003"/>
+      <inertia ixx="0.00214" ixy="0" ixz="0" iyy="0.00217" iyz="0" izz="0.003"/>
     </inertial>
   </link>
@@ -335,5 +335,5 @@
       <!-- fix for gazebo -->
       <origin xyz="-0.03 0 -0.0546" rpy="0 -0 0"/>
-      <inertia ixx="0.00178" ixy="0" ixz="0" iyy="0.00179" iyz="0" izz="0.004"/>
+      <inertia ixx="0.00178" ixy="0" ixz="0" iyy="0.00179" iyz="0" izz="0.0035"/>
     </inertial>
   </link>
@@ -355,5 +355,5 @@
       <mass value="0.132" />
       <origin xyz="0.006 0 -0.0738" rpy="0 -0 0"/>
-      <inertia ixx="0.000276" ixy="0" ixz="0" iyy="0.000286" iyz="0" izz="0.004"/>
+      <inertia ixx="0.00276" ixy="0" ixz="0" iyy="0.00286" iyz="0" izz="0.004"/>
     </inertial>
   </link>
@@ -373,5 +373,5 @@
     <axis   xyz="0 0 1"/>
     <!-- from -120 to 120 degrees-->
-    <limit lower="-2.0" upper="2.0" effort="100" velocity="0.5" />
+    <limit lower="-2.0" upper="2.0" effort="500" velocity="0.5" />
     <dynamics damping="0.2" friction="0" />
   </joint>
@@ -383,5 +383,5 @@
     <axis   xyz="0 1 0"/>
     <!-- from -5 to 30 degrees-->
-    <limit lower="-0.0872" upper="0.5235" effort="100" velocity="0.3" />
+    <limit lower="-0.0872" upper="0.5235" effort="2000" velocity="0.3" />
     <dynamics damping="0.2" friction="0" />
   </joint>
@@ -393,5 +393,5 @@
     <axis   xyz="1 0 0"/>
     <!-- from -1 to 1 degrees-->
-    <limit lower="-0.017" upper="0.017" effort="100" velocity="0.3" />
+    <limit lower="-0.017" upper="0.017" effort="2000" velocity="0.3" />
     <dynamics damping="0.2" friction="0" />
   </joint>

Commit message: [aero_description] add gazebo settings to typeFBDSy

File: aero_description/typeF/robots/aero.urdf.xacro (robot description, xacro)
@@ -15,4 +15,5 @@
  <xacro:aero-upper/>
  <xacro:aero-wheels base_link="base_link"/>
+ <!-- gazebo settings -->
  <!-- camera -->
  <link name="camera_frame" />
@@ -30,11 +31,22 @@
  <xacro:gazebo_camera link_name="camera_frame"
                       frame_name="camera_optical_frame" />
+ <!-- laser -->
  <xacro:gazebo_laser_sensor link_name="wheels_base_laser_link"
                             frame_name="wheels_base_laser_link" />
+ <!-- joint control -->
  <xacro:gazebo_trajectory_controller />
+ <!-- mobile base -->
  <xacro:gazebo_base_controller base_frame="base_link" />
+ <!-- mimic joints -->
  <gazebo>
    <plugin name="mimic_updater" filename="libmimic_plugin.so">
      <!-- lifter -->
+     <mimic joint="knee_joint"  offset="0.0" multiplier="-1.0"
+            P="4000" I="0.1" D="80" i_max="500" i_min="-500"
+            command_max="2000" command_min="-2000"> knee_joint_mimic</mimic>
+     <mimic joint="ankle_joint"  offset="0.0" multiplier="-1.0"
+            P="4000" I="0.1" D="80" i_max="500" i_min="-500"
+            command_max="2000" command_min="-2000"> ankle_joint_mimic</mimic>
+     <!-- lifter(dummy) -->
      <mimic joint="knee_joint"  offset="0.0" multiplier="-1.0"
             P="1000" I="0.0" D="1" i_max="0" i_min="0"
@@ -43,10 +55,4 @@
             P="1000" I="0.0" D="1" i_max="0" i_min="0"
             command_max="200" command_min="-200"> ankle_joint_dummy</mimic>
-     <mimic joint="knee_joint"  offset="0.0" multiplier="-1.0"
-            P="4000" I="0.1" D="80" i_max="500" i_min="-500"
-            command_max="2000" command_min="-2000"> knee_joint_mimic</mimic>
-     <mimic joint="ankle_joint"  offset="0.0" multiplier="-1.0"
-            P="4000" I="0.1" D="80" i_max="500" i_min="-500"
-            command_max="2000" command_min="-2000"> ankle_joint_mimic</mimic>
      <!-- lhand -->
      <mimic joint="l_thumb_joint"  offset="0.0" multiplier="-1.0"

File: aero_description/typeFBDSy/robots/aero.urdf.xacro (robot description, xacro)
@@ -15,5 +15,53 @@
  <xacro:aero-upper/>
  <xacro:aero-wheels base_link="base_link"/>
+ <!-- gazebo settings -->
+ <!-- camera -->
+ <link name="camera_frame" />
+ <link name="camera_optical_frame" />
+ <joint name="camera_setting" type="fixed" >
+   <parent link="head_link" />
+   <child  link="camera_frame" />
+   <origin xyz="0 0.035 0.09" rpy="0 0.15 0" />
+ </joint>
+ <joint name="camera_optical" type="fixed" >
+   <parent link="camera_frame" />
+   <child  link="camera_optical_frame" />
+   <origin xyz="0 0 0" rpy="-1.570796326795 0 -1.570796326795" />
+ </joint>
+ <xacro:gazebo_camera link_name="camera_frame"
+                      frame_name="camera_optical_frame" />
+ <!-- laser -->
+ <xacro:gazebo_laser_sensor link_name="wheels_base_laser_link"
+                            frame_name="wheels_base_laser_link" />
+ <!-- joint control -->
  <xacro:gazebo_trajectory_controller />
+ <!-- mobile base -->
  <xacro:gazebo_base_controller base_frame="base_link" />
+ <!-- mimic joints -->
+ <gazebo>
+   <plugin name="mimic_updater" filename="libmimic_plugin.so">
+     <!-- lifter -->
+     <mimic joint="knee_joint"  offset="0.0" multiplier="-1.0"
+            P="4000" I="0.1" D="80" i_max="500" i_min="-500"
+            command_max="2000" command_min="-2000"> knee_joint_mimic</mimic>
+     <mimic joint="ankle_joint"  offset="0.0" multiplier="-1.0"
+            P="4000" I="0.1" D="80" i_max="500" i_min="-500"
+            command_max="2000" command_min="-2000"> ankle_joint_mimic</mimic>
+     <!-- lifter(dummy) -->
+     <mimic joint="knee_joint"  offset="0.0" multiplier="-1.0"
+            P="1000" I="0.0" D="1" i_max="0" i_min="0"
+            command_max="200" command_min="-200"> knee_joint_dummy</mimic>
+     <mimic joint="ankle_joint"  offset="0.0" multiplier="1.0"
+            P="1000" I="0.0" D="1" i_max="0" i_min="0"
+            command_max="200" command_min="-200"> ankle_joint_dummy</mimic>
+     <!-- lhand -->
+     <mimic joint="l_indexbase_joint"  offset="-0.2" multiplier="-0.3"
+            P="30" I="0.0" D="0.03" i_max="0" i_min="0"
+            command_max="50" command_min="-50"> l_indexend_joint </mimic>
+     <!-- rhand -->
+     <mimic joint="r_indexbase_joint"  offset="0.2" multiplier="-0.3"
+            P="30" I="0.0" D="0.03" i_max="0" i_min="0"
+            command_max="50" command_min="-50"> r_indexend_joint </mimic>
+   </plugin>
+ </gazebo>
 </robot>
