Commit message: [aero_description] fix mimic description for indigo

File: aero_description/typeF/robots/aero.urdf.xacro (robot description, xacro)
@@ -44,35 +44,155 @@
      <mimic joint="knee_joint"  offset="0.0" multiplier="-1.0"
             P="4000" I="0.1" D="80" i_max="500" i_min="-500"
-            command_max="2000" command_min="-2000"> knee_joint_mimic</mimic>
+            command_max="2000" command_min="-2000">
+       knee_joint_mimic
+       <joint> knee_joint </joint>
+       <offset> 0.0 </offset>
+       <multiplier> -1.0 </multiplier>
+       <P> 4000 </P>
+       <I> 0.1 </I>
+       <D> 80 </D>
+       <i_max>  500 </i_max>
+       <i_min> -500 </i_min>
+       <command_max>  2000 </command_max>
+       <command_min> -2000 </command_min>
+     </mimic>
      <mimic joint="ankle_joint"  offset="0.0" multiplier="-1.0"
             P="4000" I="0.1" D="80" i_max="500" i_min="-500"
-            command_max="2000" command_min="-2000"> ankle_joint_mimic</mimic>
+            command_max="2000" command_min="-2000">
+       ankle_joint_mimic
+       <joint> ankle_joint </joint>
+       <offset> 0.0 </offset>
+       <multiplier> -1.0 </multiplier>
+       <P> 4000 </P>
+       <I> 0.1 </I>
+       <D> 80 </D>
+       <i_max>  500 </i_max>
+       <i_min> -500 </i_min>
+       <command_max>  2000 </command_max>
+       <command_min> -2000 </command_min>
+     </mimic>
      <!-- lifter(dummy) -->
      <mimic joint="knee_joint"  offset="0.0" multiplier="-1.0"
             P="1000" I="0.0" D="1" i_max="0" i_min="0"
-            command_max="200" command_min="-200"> knee_joint_dummy</mimic>
+            command_max="200" command_min="-200">
+       knee_joint_dummy
+       <joint> knee_joint </joint>
+       <offset> 0.0 </offset>
+       <multiplier> -1.0 </multiplier>
+       <P> 1000 </P>
+       <I> 0.0 </I>
+       <D> 1 </D>
+       <i_max>  0 </i_max>
+       <i_min> -0 </i_min>
+       <command_max>  200 </command_max>
+       <command_min> -200 </command_min>
+     </mimic>
      <mimic joint="ankle_joint"  offset="0.0" multiplier="1.0"
             P="1000" I="0.0" D="1" i_max="0" i_min="0"
-            command_max="200" command_min="-200"> ankle_joint_dummy</mimic>
+            command_max="200" command_min="-200">
+       ankle_joint_dummy
+       <joint> ankle_joint </joint>
+       <offset> 0.0 </offset>
+       <multiplier> 1.0 </multiplier>
+       <P> 1000 </P>
+       <I> 0.0 </I>
+       <D> 1 </D>
+       <i_max>  0 </i_max>
+       <i_min> -0 </i_min>
+       <command_max>  200 </command_max>
+       <command_min> -200 </command_min>
+     </mimic>
      <!-- lhand -->
      <mimic joint="l_thumb_joint"  offset="0.0" multiplier="-1.0"
             P="30" I="0.0" D="0.03" i_max="0" i_min="0"
-            command_max="50" command_min="-50"> l_indexbase_joint </mimic>
+            command_max="50" command_min="-50">
+       l_indexbase_joint
+       <joint> l_thumb_joint </joint>
+       <offset> 0.0 </offset>
+       <multiplier> -1.0 </multiplier>
+       <P> 30 </P>
+       <I> 0.0 </I>
+       <D> 0.03 </D>
+       <i_max>  0 </i_max>
+       <i_min> -0 </i_min>
+       <command_max>  50 </command_max>
+       <command_min> -50 </command_min>
+     </mimic>
      <mimic joint="l_thumb_joint"  offset="-0.2" multiplier="-0.3"
             P="30" I="0.0" D="0.03" i_max="0" i_min="0"
-            command_max="50" command_min="-50"> l_indexmid_joint </mimic>
+            command_max="50" command_min="-50">
+       l_indexmid_joint
+       <joint> l_thumb_joint </joint>
+       <offset> -0.2 </offset>
+       <multiplier> -0.3 </multiplier>
+       <P> 30 </P>
+       <I> 0.0 </I>
+       <D> 0.03 </D>
+       <i_max>  0 </i_max>
+       <i_min> -0 </i_min>
+       <command_max>  50 </command_max>
+       <command_min> -50 </command_min>
+     </mimic>
      <mimic joint="l_thumb_joint"  offset="-0.2" multiplier="-0.3"
             P="30" I="0.0" D="0.03" i_max="0" i_min="0"
-            command_max="50" command_min="-50"> l_indexend_joint </mimic>
+            command_max="50" command_min="-50">
+       l_indexend_joint
+       <joint> l_thumb_joint </joint>
+       <offset> -0.2 </offset>
+       <multiplier> -0.3 </multiplier>
+       <P> 30 </P>
+       <I> 0.0 </I>
+       <D> 0.03 </D>
+       <i_max>  0 </i_max>
+       <i_min> -0 </i_min>
+       <command_max>  50 </command_max>
+       <command_min> -50 </command_min>
+     </mimic>
      <!-- rhand -->
      <mimic joint="r_thumb_joint"  offset="0.0" multiplier="-1.0"
             P="30" I="0.0" D="0.03" i_max="0" i_min="0"
-            command_max="50" command_min="-50"> r_indexbase_joint </mimic>
+            command_max="50" command_min="-50">
+       r_indexbase_joint
+       <joint> r_thumb_joint </joint>
+       <offset> 0.0 </offset>
+       <multiplier> -1.0 </multiplier>
+       <P> 30 </P>
+       <I> 0.0 </I>
+       <D> 0.03 </D>
+       <i_max>  0 </i_max>
+       <i_min> -0 </i_min>
+       <command_max>  50 </command_max>
+       <command_min> -50 </command_min>
+     </mimic>
      <mimic joint="r_thumb_joint"  offset="0.2" multiplier="-0.3"
             P="30" I="0.0" D="0.03" i_max="0" i_min="0"
-            command_max="50" command_min="-50"> r_indexmid_joint </mimic>
+            command_max="50" command_min="-50">
+       r_indexmid_joint
+       <joint> r_thumb_joint </joint>
+       <offset> 0.2 </offset>
+       <multiplier> -0.3 </multiplier>
+       <P> 30 </P>
+       <I> 0.0 </I>
+       <D> 0.03 </D>
+       <i_max>  0 </i_max>
+       <i_min> -0 </i_min>
+       <command_max>  50 </command_max>
+       <command_min> -50 </command_min>
+     </mimic>
      <mimic joint="r_thumb_joint"  offset="0.2" multiplier="-0.3"
             P="30" I="0.0" D="0.03" i_max="0" i_min="0"
-            command_max="50" command_min="-50"> r_indexend_joint </mimic>
+            command_max="50" command_min="-50">
+       r_indexend_joint
+       <joint> r_thumb_joint </joint>
+       <offset> 0.2 </offset>
+       <multiplier> -0.3 </multiplier>
+       <P> 30 </P>
+       <I> 0.0 </I>
+       <D> 0.03 </D>
+       <i_max>  0 </i_max>
+       <i_min> -0 </i_min>
+       <command_max>  50 </command_max>
+       <command_min> -50 </command_min>
+     </mimic>
    </plugin>
  </gazebo>

File: aero_description/typeFBDSy/robots/aero.urdf.xacro (robot description, xacro)
@@ -44,23 +44,95 @@
      <mimic joint="knee_joint"  offset="0.0" multiplier="-1.0"
             P="4000" I="0.1" D="80" i_max="500" i_min="-500"
-            command_max="2000" command_min="-2000"> knee_joint_mimic</mimic>
+            command_max="2000" command_min="-2000">
+       knee_joint_mimic
+       <joint> knee_joint </joint>
+       <offset> 0.0 </offset>
+       <multiplier> -1.0 </multiplier>
+       <P> 4000 </P>
+       <I> 0.1 </I>
+       <D> 80 </D>
+       <i_max>  500 </i_max>
+       <i_min> -500 </i_min>
+       <command_max>  2000 </command_max>
+       <command_min> -2000 </command_min>
+     </mimic>
      <mimic joint="ankle_joint"  offset="0.0" multiplier="-1.0"
             P="4000" I="0.1" D="80" i_max="500" i_min="-500"
-            command_max="2000" command_min="-2000"> ankle_joint_mimic</mimic>
+            command_max="2000" command_min="-2000">
+       ankle_joint_mimic
+       <joint> ankle_joint </joint>
+       <offset> 0.0 </offset>
+       <multiplier> -1.0 </multiplier>
+       <P> 4000 </P>
+       <I> 0.1 </I>
+       <D> 80 </D>
+       <i_max>  500 </i_max>
+       <i_min> -500 </i_min>
+       <command_max>  2000 </command_max>
+       <command_min> -2000 </command_min>
+     </mimic>
      <!-- lifter(dummy) -->
      <mimic joint="knee_joint"  offset="0.0" multiplier="-1.0"
             P="1000" I="0.0" D="1" i_max="0" i_min="0"
-            command_max="200" command_min="-200"> knee_joint_dummy</mimic>
+            command_max="200" command_min="-200">
+       knee_joint_dummy
+       <joint> knee_joint </joint>
+       <offset> 0.0 </offset>
+       <multiplier> -1.0 </multiplier>
+       <P> 1000 </P>
+       <I> 0.0 </I>
+       <D> 1 </D>
+       <i_max>  0 </i_max>
+       <i_min> -0 </i_min>
+       <command_max>  200 </command_max>
+       <command_min> -200 </command_min>
+     </mimic>
      <mimic joint="ankle_joint"  offset="0.0" multiplier="1.0"
             P="1000" I="0.0" D="1" i_max="0" i_min="0"
-            command_max="200" command_min="-200"> ankle_joint_dummy</mimic>
+            command_max="200" command_min="-200">
+       ankle_joint_dummy
+       <joint> ankle_joint </joint>
+       <offset> 0.0 </offset>
+       <multiplier> 1.0 </multiplier>
+       <P> 1000 </P>
+       <I> 0.0 </I>
+       <D> 1 </D>
+       <i_max>  0 </i_max>
+       <i_min> -0 </i_min>
+       <command_max>  200 </command_max>
+       <command_min> -200 </command_min>
+     </mimic>
      <!-- lhand -->
      <mimic joint="l_indexbase_joint"  offset="-0.2" multiplier="-0.3"
             P="30" I="0.0" D="0.03" i_max="0" i_min="0"
-            command_max="50" command_min="-50"> l_indexend_joint </mimic>
+            command_max="50" command_min="-50">
+       l_indexend_joint
+       <joint> l_indexbase_joint </joint>
+       <offset> -0.2 </offset>
+       <multiplier> -0.3 </multiplier>
+       <P> 30 </P>
+       <I> 0.0 </I>
+       <D> 0.03 </D>
+       <i_max>  0 </i_max>
+       <i_min> -0 </i_min>
+       <command_max>  50 </command_max>
+       <command_min> -50 </command_min>
+     </mimic>
      <!-- rhand -->
      <mimic joint="r_indexbase_joint"  offset="0.2" multiplier="-0.3"
             P="30" I="0.0" D="0.03" i_max="0" i_min="0"
-            command_max="50" command_min="-50"> r_indexend_joint </mimic>
+            command_max="50" command_min="-50">
+       r_indexend_joint
+       <joint> r_indexbase_joint </joint>
+       <offset> 0.2 </offset>
+       <multiplier> -0.3 </multiplier>
+       <P> 30 </P>
+       <I> 0.0 </I>
+       <D> 0.03 </D>
+       <i_max>  0 </i_max>
+       <i_min> -0 </i_min>
+       <command_max>  50 </command_max>
+       <command_min> -50 </command_min>
+     </mimic>
    </plugin>
  </gazebo>

File: aero_description/typeFCESy/robots/aero.urdf.xacro (robot description, xacro)
@@ -44,23 +44,95 @@
      <mimic joint="knee_joint"  offset="0.0" multiplier="-1.0"
             P="4000" I="0.1" D="80" i_max="500" i_min="-500"
-            command_max="2000" command_min="-2000"> knee_joint_mimic</mimic>
+            command_max="2000" command_min="-2000">
+       knee_joint_mimic
+       <joint> knee_joint </joint>
+       <offset> 0.0 </offset>
+       <multiplier> -1.0 </multiplier>
+       <P> 4000 </P>
+       <I> 0.1 </I>
+       <D> 80 </D>
+       <i_max>  500 </i_max>
+       <i_min> -500 </i_min>
+       <command_max>  2000 </command_max>
+       <command_min> -2000 </command_min>
+     </mimic>
      <mimic joint="ankle_joint"  offset="0.0" multiplier="-1.0"
             P="4000" I="0.1" D="80" i_max="500" i_min="-500"
-            command_max="2000" command_min="-2000"> ankle_joint_mimic</mimic>
+            command_max="2000" command_min="-2000">
+       ankle_joint_mimic
+       <joint> ankle_joint </joint>
+       <offset> 0.0 </offset>
+       <multiplier> -1.0 </multiplier>
+       <P> 4000 </P>
+       <I> 0.1 </I>
+       <D> 80 </D>
+       <i_max>  500 </i_max>
+       <i_min> -500 </i_min>
+       <command_max>  2000 </command_max>
+       <command_min> -2000 </command_min>
+     </mimic>
      <!-- lifter(dummy) -->
      <mimic joint="knee_joint"  offset="0.0" multiplier="-1.0"
             P="1000" I="0.0" D="1" i_max="0" i_min="0"
-            command_max="200" command_min="-200"> knee_joint_dummy</mimic>
+            command_max="200" command_min="-200">
+       knee_joint_dummy
+       <joint> knee_joint </joint>
+       <offset> 0.0 </offset>
+       <multiplier> -1.0 </multiplier>
+       <P> 1000 </P>
+       <I> 0.0 </I>
+       <D> 1 </D>
+       <i_max>  0 </i_max>
+       <i_min> -0 </i_min>
+       <command_max>  200 </command_max>
+       <command_min> -200 </command_min>
+     </mimic>
      <mimic joint="ankle_joint"  offset="0.0" multiplier="1.0"
             P="1000" I="0.0" D="1" i_max="0" i_min="0"
-            command_max="200" command_min="-200"> ankle_joint_dummy</mimic>
+            command_max="200" command_min="-200">
+       ankle_joint_dummy
+       <joint> ankle_joint </joint>
+       <offset> 0.0 </offset>
+       <multiplier> 1.0 </multiplier>
+       <P> 1000 </P>
+       <I> 0.0 </I>
+       <D> 1 </D>
+       <i_max>  0 </i_max>
+       <i_min> -0 </i_min>
+       <command_max>  200 </command_max>
+       <command_min> -200 </command_min>
+     </mimic>
      <!-- lhand -->
      <mimic joint="l_indexbase_joint"  offset="-0.2" multiplier="-0.3"
             P="30" I="0.0" D="0.03" i_max="0" i_min="0"
-            command_max="50" command_min="-50"> l_indexend_joint </mimic>
+            command_max="50" command_min="-50">
+       l_indexend_joint
+       <joint> l_indexbase_joint </joint>
+       <offset> -0.2 </offset>
+       <multiplier> -0.3 </multiplier>
+       <P> 30 </P>
+       <I> 0.0 </I>
+       <D> 0.03 </D>
+       <i_max>  0 </i_max>
+       <i_min> -0 </i_min>
+       <command_max>  50 </command_max>
+       <command_min> -50 </command_min>
+     </mimic>
      <!-- rhand -->
      <mimic joint="r_indexbase_joint"  offset="0.2" multiplier="-0.3"
             P="30" I="0.0" D="0.03" i_max="0" i_min="0"
-            command_max="50" command_min="-50"> r_indexend_joint </mimic>
+            command_max="50" command_min="-50">
+       r_indexend_joint
+       <joint> r_indexbase_joint </joint>
+       <offset> 0.2 </offset>
+       <multiplier> -0.3 </multiplier>
+       <P> 30 </P>
+       <I> 0.0 </I>
+       <D> 0.03 </D>
+       <i_max>  0 </i_max>
+       <i_min> -0 </i_min>
+       <command_max>  50 </command_max>
+       <command_min> -50 </command_min>
+     </mimic>
    </plugin>
  </gazebo>
