Commit message: base_link is base_link

File: aero_description/typeF/urdf/aero_upper/aero_upper.urdf.xacro (robot description, xacro)
@@ -641,4 +641,14 @@
     <mu2>0.9</mu2>
   </gazebo>
+  <!-- for ik eef link-->
+<link name="r_eef_grasp_link"/>
+<link name="r_eef_pick_link"/>
+<link name="r_thumb_tip_link"/>
+<link name="r_index_tip_link"/>
+<link name="l_eef_grasp_link"/>
+<link name="l_eef_pick_link"/>
+<link name="l_thumb_tip_link"/>
+<link name="l_index_tip_link"/>
+  <!-- for ik eef link-->
   <joint name="waist_y_joint" type="revolute">
     <parent link="${base_link}"/>
@@ -1064,4 +1074,46 @@
     <cfmDamping>0.4</cfmDamping>
   </gazebo>
+  <!-- for ik eef connector-->
+<joint name="r_eef_grasp_joint" type="fixed">
+  <parent  link="r_hand_link"/>
+  <child link="r_eef_grasp_link"/>
+  <origin xyz="0.0 0.04 -0.14" rpy="0 1.5708 0 "/>
+</joint>
+<joint name="r_eef_pick_joint" type="fixed">
+  <parent  link="r_hand_link"/>
+  <child link="r_eef_pick_link"/>
+  <origin xyz="0.0 0.07 -0.16" rpy="0 1.5708 0 "/>
+</joint>
+<joint name="r_thumb_tip_joint" type="fixed">
+  <parent  link="r_indexend_link"/>
+  <child link="r_thumb_tip_link"/>
+  <origin xyz="0.0 0.035 -0.085" rpy="0 0 0 "/>
+</joint>
+<joint name="r_index_tip_joint" type="fixed">
+  <parent  link="r_indexmid_link"/>
+  <child link="r_index_tip_link"/>
+  <origin xyz="0.0 0.02 0.0" rpy="0 0 0 "/>
+</joint>
+<joint name="l_eef_grasp_joint" type="fixed">
+  <parent  link="l_hand_link"/>
+  <child link="l_eef_grasp_link"/>
+  <origin xyz="0.0 -0.04 -0.14" rpy="0 1.5708 0 "/>
+</joint>
+<joint name="l_eef_pick_joint" type="fixed">
+  <parent  link="l_hand_link"/>
+  <child link="l_eef_pick_link"/>
+  <origin xyz="0.0 -0.07 -0.16" rpy="0 1.5708 0 "/>
+</joint>
+<joint name="l_thumb_tip_joint" type="fixed">
+  <parent  link="l_indexend_link"/>
+  <child link="l_thumb_tip_link"/>
+  <origin xyz="0.0 -0.035 -0.085" rpy="0 0 0 "/>
+</joint>
+<joint name="l_index_tip_joint" type="fixed">
+  <parent  link="l_indexmid_link"/>
+  <child link="l_index_tip_link"/>
+  <origin xyz="0.0 -0.02 -0.0" rpy="0 0 0 "/>
+</joint>
+  <!-- for ik eef connector-->
   </xacro:macro>
 </robot>

Commit message: limit joint limit in xacro model

File: aero_description/typeF/urdf/aero_upper/aero_upper.urdf.xacro (robot description, xacro)
@@ -672,5 +672,5 @@
     <origin xyz="0 0 0.1355" rpy="0 -0 0 "/>
     <axis   xyz="0 1 0"/>
-    <limit lower="0" upper="1.5707" effort="100" velocity="0.5" />
+    <limit lower="0" upper="0.4014" effort="100" velocity="0.5" />
     <dynamics damping="0.2" friction="0" />
   </joint>
@@ -688,5 +688,5 @@
     <origin xyz="0 0 0" rpy="0 -0 0 "/>
     <axis   xyz="1 0 0"/>
-    <limit lower="-0.122173" upper="0.122173" effort="100" velocity="0.5" />
+    <limit lower="-0.017" upper="0.017" effort="100" velocity="0.5" />
     <dynamics damping="0.2" friction="0" />
   </joint>
@@ -768,5 +768,5 @@
     <origin xyz="-0.035 0 -0.070" rpy="0 -0 0 "/>
     <axis   xyz="0 0 1"/>
-    <limit lower="-3.14159" upper="3.14159" effort="100" velocity="0.5" />
+    <limit lower="-1.5708" upper="1.5708" effort="100" velocity="0.5" />
     <dynamics damping="0.2" friction="0" />
   </joint>
@@ -784,5 +784,5 @@
     <origin xyz="0 0 -0.1955" rpy="0 -0 0 "/>
     <axis   xyz="0 1 0"/>
-    <limit lower="-0.349066" upper="0.349066" effort="100" velocity="0.5" />
+    <limit lower="-0.017" upper="0.017" effort="100" velocity="0.5" />
     <dynamics damping="0.2" friction="0" />
   </joint>
@@ -881,5 +881,5 @@
     <origin xyz="0 0 0.1045" rpy="0 -0 0 "/>
     <axis   xyz="0 1 0"/>
-    <limit lower="0" upper="1.04667" effort="100" velocity="0.5" />
+    <limit lower="0" upper="0.610864" effort="100" velocity="0.5" />
     <dynamics damping="0.2" friction="0" />
   </joint>
@@ -977,5 +977,5 @@
     <origin xyz="-0.035 0 -0.070" rpy="0 -0 0 "/>
     <axis   xyz="0 0 1"/>
-    <limit lower="-3.14159" upper="3.14159" effort="100" velocity="0.5" />
+    <limit lower="-1.5708" upper="1.5708" effort="100" velocity="0.5" />
     <dynamics damping="0.2" friction="0" />
   </joint>
@@ -993,5 +993,5 @@
     <origin xyz="0 0 -0.1955" rpy="0 -0 0 "/>
     <axis   xyz="0 1 0"/>
-    <limit lower="-0.349066" upper="0.349066" effort="100" velocity="0.5" />
+    <limit lower="-0.017" upper="0.017" effort="100" velocity="0.5" />
     <dynamics damping="0.2" friction="0" />
   </joint>

Commit message: limit neck yaw to 180 degrees

File: aero_description/typeF/urdf/aero_upper/aero_upper.urdf.xacro (robot description, xacro)
@@ -865,5 +865,5 @@
     <origin xyz="0 0 0.3535" rpy="0 -0 0 "/>
     <axis   xyz="0 0 1"/>
-    <limit lower="-3.14159" upper="3.14159" effort="100" velocity="0.5" />
+    <limit lower="-1.5707" upper="1.5707" effort="100" velocity="0.5" />
     <dynamics damping="0.2" friction="0" />
   </joint>

Commit message: joint angle limits in urdf

File: aero_description/typeF/urdf/aero_upper/aero_upper.urdf.xacro (robot description, xacro)
@@ -8,4 +8,5 @@
   <!--xacro:include filename="$(find aero_description)/urdf/aero_upper/aero_upper.transmission.xacro" /-->
   <xacro:include filename="$(find aero_description)/urdf/common.xacro" />
+  <xacro:property name="wrist_sensor_offset" value="0.0"/>
   <!-- ============================   aero_upper   ============================ -->
   <xacro:macro name="aero_upper" params="base_link disable_mesh:=false">
@@ -218,5 +219,5 @@
   <link name="l_hand_link">
     <xacro:unless value="${disable_mesh}"> <visual>
-      <origin xyz="0 0 0" rpy="0 -0 0"/>
+      <origin xyz="0 0 ${-1.0 * wrist_sensor_offset}" rpy="0 -0 0"/>
       <geometry>
         <mesh filename="package://aero_description/meshes/aero_upper_meshes/LARM_LINK7_mesh.dae" scale="1 1 1" />
@@ -224,5 +225,5 @@
     </visual> </xacro:unless>
     <xacro:unless value="${disable_mesh}"> <collision>
-      <origin xyz="0 0 0" rpy="0 -0 0"/>
+      <origin xyz="0 0 ${-1.0 * wrist_sensor_offset}" rpy="0 -0 0"/>
       <geometry>
         <mesh filename="package://aero_description/meshes/aero_upper_meshes/LARM_LINK7_mesh.dae" scale="1 1 1" />
@@ -231,5 +232,5 @@
     <inertial>
       <mass value="0.183" />
-      <origin xyz="0 0 -0.0875" rpy="0 -0 0"/>
+      <origin xyz="0 0 ${-0.0875 - wrist_sensor_offset}" rpy="0 -0 0"/>
       <inertia ixx="0.000601" ixy="0" ixz="0" iyy="0.00055" iyz="0" izz="0.000102"/>
     </inertial>
@@ -528,5 +529,5 @@
   <link name="r_hand_link">
     <xacro:unless value="${disable_mesh}"> <visual>
-      <origin xyz="0 0 0" rpy="0 -0 0"/>
+      <origin xyz="0 0 ${-1.0 * wrist_sensor_offset}" rpy="0 -0 0"/>
       <geometry>
         <mesh filename="package://aero_description/meshes/aero_upper_meshes/RARM_LINK7_mesh.dae" scale="1 1 1" />
@@ -534,5 +535,5 @@
     </visual> </xacro:unless>
     <xacro:unless value="${disable_mesh}"> <collision>
-      <origin xyz="0 0 0" rpy="0 -0 0"/>
+      <origin xyz="0 0 ${-1.0 * wrist_sensor_offset}" rpy="0 -0 0"/>
       <geometry>
         <mesh filename="package://aero_description/meshes/aero_upper_meshes/RARM_LINK7_mesh.dae" scale="1 1 1" />
@@ -541,5 +542,5 @@
     <inertial>
       <mass value="0.183" />
-      <origin xyz="0 0 -0.0875" rpy="0 -0 0"/>
+      <origin xyz="0 0 ${-0.0875 - wrist_sensor_offset}" rpy="0 -0 0"/>
       <inertia ixx="0.000601" ixy="0" ixz="0" iyy="0.00055" iyz="0" izz="0.000102"/>
     </inertial>
@@ -656,5 +657,5 @@
     <origin xyz="0 0 0.010" rpy="0 -0 0 "/>
     <axis   xyz="0 0 1"/>
-    <limit lower="-3.14159" upper="3.14159" effort="100" velocity="0.5" />
+    <limit lower="-1.5707" upper="1.5707" effort="100" velocity="0.5" />
     <dynamics damping="0.2" friction="0" />
   </joint>
@@ -704,5 +705,5 @@
     <origin xyz="-0.01815 0.1342 0.3049" rpy="0 -0 0 "/>
     <axis   xyz="0 0.984808 -0.173648"/>
-    <limit lower="-1.5707" upper="0" effort="100" velocity="0.5" />
+    <limit lower="-1.50" upper="0" effort="100" velocity="0.5" />
     <dynamics damping="0.2" friction="0" />
   </joint>
@@ -736,5 +737,5 @@
     <origin xyz="0 -0.010 -0.127" rpy="0 -0 0 "/>
     <axis   xyz="0 0 1"/>
-    <limit lower="-3.14159" upper="3.14159" effort="100" velocity="0.5" />
+    <limit lower="-1.5707" upper="0.785398" effort="100" velocity="0.5" />
     <dynamics damping="0.2" friction="0" />
   </joint>
@@ -768,5 +769,5 @@
     <origin xyz="-0.035 0 -0.070" rpy="0 -0 0 "/>
     <axis   xyz="0 0 1"/>
-    <limit lower="-1.5708" upper="1.5708" effort="100" velocity="0.5" />
+    <limit lower="-1.5707" upper="1.5707" effort="100" velocity="0.5" />
     <dynamics damping="0.2" friction="0" />
   </joint>
@@ -784,5 +785,5 @@
     <origin xyz="0 0 -0.1955" rpy="0 -0 0 "/>
     <axis   xyz="0 1 0"/>
-    <limit lower="-0.017" upper="0.017" effort="100" velocity="0.5" />
+    <limit lower="-0.15" upper="0.15" effort="100" velocity="0.5" />
     <dynamics damping="0.2" friction="0" />
   </joint>
@@ -814,5 +815,5 @@
     <parent link="l_hand_link"/>
     <child  link="l_thumb_link"/>
-    <origin xyz="0 0.013 -0.115" rpy="0 -0 0 "/>
+    <origin xyz="0 0.013 ${-0.115 - wrist_sensor_offset}" rpy="0 -0 0 "/>
     <axis   xyz="1 0 0"/>
     <limit lower="-3.14159" upper="3.14159" effort="100" velocity="0.5" />
@@ -847,5 +848,5 @@
     <parent link="l_hand_link"/>
     <child  link="l_indexend_link"/>
-    <origin xyz="0 -0.022355 -0.079645" rpy="0 -0 0 "/>
+    <origin xyz="0 -0.022355 ${-0.079645 - wrist_sensor_offset}" rpy="0 -0 0 "/>
     <axis   xyz="1 0 0"/>
     <limit lower="-3.14159" upper="3.14159" effort="100" velocity="0.5" />
@@ -865,5 +866,5 @@
     <origin xyz="0 0 0.3535" rpy="0 -0 0 "/>
     <axis   xyz="0 0 1"/>
-    <limit lower="-3.14159" upper="3.14159" effort="100" velocity="0.5" />
+    <limit lower="-1.5707" upper="1.5707" effort="100" velocity="0.5" />
     <dynamics damping="0.2" friction="0" />
   </joint>
@@ -913,5 +914,5 @@
     <origin xyz="-0.01815 -0.1342 0.3049" rpy="0 -0 0 "/>
     <axis   xyz="0 0.984808 0.173648"/>
-    <limit lower="-1.5707" upper="0" effort="100" velocity="0.5" />
+    <limit lower="-1.50" upper="0" effort="100" velocity="0.5" />
     <dynamics damping="0.2" friction="0" />
   </joint>
@@ -945,5 +946,5 @@
     <origin xyz="0 0.010 -0.127" rpy="0 -0 0 "/>
     <axis   xyz="0 0 1"/>
-    <limit lower="-3.14159" upper="3.14159" effort="100" velocity="0.5" />
+    <limit lower="-0.785398" upper="1.5707" effort="100" velocity="0.5" />
     <dynamics damping="0.2" friction="0" />
   </joint>
@@ -977,5 +978,5 @@
     <origin xyz="-0.035 0 -0.070" rpy="0 -0 0 "/>
     <axis   xyz="0 0 1"/>
-    <limit lower="-1.5708" upper="1.5708" effort="100" velocity="0.5" />
+    <limit lower="-1.5707" upper="1.5707" effort="100" velocity="0.5" />
     <dynamics damping="0.2" friction="0" />
   </joint>
@@ -993,5 +994,5 @@
     <origin xyz="0 0 -0.1955" rpy="0 -0 0 "/>
     <axis   xyz="0 1 0"/>
-    <limit lower="-0.017" upper="0.017" effort="100" velocity="0.5" />
+    <limit lower="-0.15" upper="0.15" effort="100" velocity="0.5" />
     <dynamics damping="0.2" friction="0" />
   </joint>
@@ -1023,5 +1024,5 @@
     <parent link="r_hand_link"/>
     <child  link="r_thumb_link"/>
-    <origin xyz="0 -0.013 -0.115" rpy="0 -0 0 "/>
+    <origin xyz="0 -0.013 ${-0.115 - wrist_sensor_offset}" rpy="0 -0 0 "/>
     <axis   xyz="1 0 0"/>
     <limit lower="-3.14159" upper="3.14159" effort="100" velocity="0.5" />
@@ -1061,5 +1062,5 @@
     <parent link="r_hand_link"/>
     <child  link="r_indexend_link"/>
-    <origin xyz="0 0.022355 -0.079645" rpy="0 -0 0 "/>
+    <origin xyz="0 0.022355 ${-0.079645 - wrist_sensor_offset}" rpy="0 -0 0 "/>
     <axis   xyz="1 0 0"/>
     <limit lower="-3.14159" upper="3.14159" effort="100" velocity="0.5" />
@@ -1078,10 +1079,10 @@
   <parent  link="r_hand_link"/>
   <child link="r_eef_grasp_link"/>
-  <origin xyz="0.0 0.04 -0.14" rpy="0 1.5708 0 "/>
+  <origin xyz="0.0 0.04 ${-0.14 - wrist_sensor_offset}" rpy="0 1.5708 0 "/>
 </joint>
 <joint name="r_eef_pick_joint" type="fixed">
   <parent  link="r_hand_link"/>
   <child link="r_eef_pick_link"/>
-  <origin xyz="0.0 0.07 -0.16" rpy="0 1.5708 0 "/>
+  <origin xyz="0.0 0.07 ${-0.16 - wrist_sensor_offset}" rpy="0 1.5708 0 "/>
 </joint>
 <joint name="r_thumb_tip_joint" type="fixed">
@@ -1098,10 +1099,10 @@
   <parent  link="l_hand_link"/>
   <child link="l_eef_grasp_link"/>
-  <origin xyz="0.0 -0.04 -0.14" rpy="0 1.5708 0 "/>
+  <origin xyz="0.0 -0.04 ${-0.14 - wrist_sensor_offset}" rpy="0 1.5708 0 "/>
 </joint>
 <joint name="l_eef_pick_joint" type="fixed">
   <parent  link="l_hand_link"/>
   <child link="l_eef_pick_link"/>
-  <origin xyz="0.0 -0.07 -0.16" rpy="0 1.5708 0 "/>
+  <origin xyz="0.0 -0.07 ${-0.16 - wrist_sensor_offset}" rpy="0 1.5708 0 "/>
 </joint>
 <joint name="l_thumb_tip_joint" type="fixed">
