Commit message: modify link hand link names in urdf

File: aero_description/typeF/urdf/aero_upper/aero_upper.urdf.xacro (robot description, xacro)
@@ -240,15 +240,84 @@
     <mu2>0.9</mu2>
   </gazebo>
+  <link name="l_indexbase_link">
+    <xacro:unless value="${disable_mesh}"> <visual>
+      <origin xyz="0 -0.013 0.115" rpy="0 -0 0 "/>
+      <geometry>
+        <mesh filename="package://aero_description/meshes/aero_upper_meshes/LARM_INDEX_LINK1_mesh.dae" scale="1 1 1" />
+      </geometry>
+    </visual> </xacro:unless>
+    <xacro:unless value="${disable_mesh}"> <collision>
+      <origin xyz="0 -0.013 0.115" rpy="0 -0 0 "/>
+      <geometry>
+        <mesh filename="package://aero_description/meshes/aero_upper_meshes/LARM_INDEX_LINK1_mesh.dae" scale="1 1 1" />
+      </geometry>
+    </collision> </xacro:unless>
+    <inertial>
+      <mass value="0" />
+      <origin xyz="0 0 0" rpy="0 -0 0"/>
+      <inertia ixx="0" ixy="0" ixz="0" iyy="0" iyz="0" izz="0"/>
+    </inertial>
+  </link>
+  <gazebo reference="l_indexbase_link">
+    <mu1>0.9</mu1>
+    <mu2>0.9</mu2>
+  </gazebo>
+  <link name="l_indexmid_link">
+    <xacro:unless value="${disable_mesh}"> <visual>
+      <origin xyz="0 0.015754 0.149615" rpy="0 -0 0"/>
+      <geometry>
+        <mesh filename="package://aero_description/meshes/aero_upper_meshes/LARM_INDEX_LINK2_mesh.dae" scale="1 1 1" />
+      </geometry>
+    </visual> </xacro:unless>
+    <xacro:unless value="${disable_mesh}"> <collision>
+      <origin xyz="0 0.015754 0.149615" rpy="0 -0 0"/>
+      <geometry>
+        <mesh filename="package://aero_description/meshes/aero_upper_meshes/LARM_INDEX_LINK2_mesh.dae" scale="1 1 1" />
+      </geometry>
+    </collision> </xacro:unless>
+    <inertial>
+      <mass value="0" />
+      <origin xyz="0 0 0" rpy="0 -0 0"/>
+      <inertia ixx="0" ixy="0" ixz="0" iyy="0" iyz="0" izz="0"/>
+    </inertial>
+  </link>
+  <gazebo reference="l_indexmid_link">
+    <mu1>0.9</mu1>
+    <mu2>0.9</mu2>
+  </gazebo>
+  <link name="l_indexend_link">
+    <xacro:unless value="${disable_mesh}"> <visual>
+      <origin xyz="0 0.03747 0.162972" rpy="0 -0 0"/>
+      <geometry>
+        <mesh filename="package://aero_description/meshes/aero_upper_meshes/LARM_INDEX_LINK3_mesh.dae" scale="1 1 1" />
+      </geometry>
+    </visual> </xacro:unless>
+    <xacro:unless value="${disable_mesh}"> <collision>
+      <origin xyz="0 0.03747 0.162972" rpy="0 -0 0"/>
+      <geometry>
+        <mesh filename="package://aero_description/meshes/aero_upper_meshes/LARM_INDEX_LINK3_mesh.dae" scale="1 1 1" />
+      </geometry>
+    </collision> </xacro:unless>
+    <inertial>
+      <mass value="0" />
+      <origin xyz="0 0 0" rpy="0 -0 0"/>
+      <inertia ixx="0" ixy="0" ixz="0" iyy="0" iyz="0" izz="0"/>
+    </inertial>
+  </link>
+  <gazebo reference="l_indexend_link">
+    <mu1>0.9</mu1>
+    <mu2>0.9</mu2>
+  </gazebo>
   <link name="l_thumb_link">
     <xacro:unless value="${disable_mesh}"> <visual>
-      <origin xyz="0 -0.013 0.115" rpy="0 -0 0 "/>
-      <geometry>
-        <mesh filename="package://aero_description/meshes/aero_upper_meshes/LARM_INDEX_LINK1_mesh.dae" scale="1 1 1" />
-      </geometry>
-    </visual> </xacro:unless>
-    <xacro:unless value="${disable_mesh}"> <collision>
-      <origin xyz="0 -0.013 0.115" rpy="0 -0 0 "/>
-      <geometry>
-        <mesh filename="package://aero_description/meshes/aero_upper_meshes/LARM_INDEX_LINK1_mesh.dae" scale="1 1 1" />
+      <origin xyz="0 0.022355 0.079645" rpy="0 -0 0 "/>
+      <geometry>
+        <mesh filename="package://aero_description/meshes/aero_upper_meshes/LARM_THUMB_LINK_mesh.dae" scale="1 1 1" />
+      </geometry>
+    </visual> </xacro:unless>
+    <xacro:unless value="${disable_mesh}"> <collision>
+      <origin xyz="0 0.022355 0.079645" rpy="0 -0 0 "/>
+      <geometry>
+        <mesh filename="package://aero_description/meshes/aero_upper_meshes/LARM_THUMB_LINK_mesh.dae" scale="1 1 1" />
       </geometry>
     </collision> </xacro:unless>
@@ -260,73 +329,4 @@
   </link>
   <gazebo reference="l_thumb_link">
-    <mu1>0.9</mu1>
-    <mu2>0.9</mu2>
-  </gazebo>
-  <link name="l_indexbase_link">
-    <xacro:unless value="${disable_mesh}"> <visual>
-      <origin xyz="0 0.015754 0.149615" rpy="0 -0 0"/>
-      <geometry>
-        <mesh filename="package://aero_description/meshes/aero_upper_meshes/LARM_INDEX_LINK2_mesh.dae" scale="1 1 1" />
-      </geometry>
-    </visual> </xacro:unless>
-    <xacro:unless value="${disable_mesh}"> <collision>
-      <origin xyz="0 0.015754 0.149615" rpy="0 -0 0"/>
-      <geometry>
-        <mesh filename="package://aero_description/meshes/aero_upper_meshes/LARM_INDEX_LINK2_mesh.dae" scale="1 1 1" />
-      </geometry>
-    </collision> </xacro:unless>
-    <inertial>
-      <mass value="0" />
-      <origin xyz="0 0 0" rpy="0 -0 0"/>
-      <inertia ixx="0" ixy="0" ixz="0" iyy="0" iyz="0" izz="0"/>
-    </inertial>
-  </link>
-  <gazebo reference="l_indexbase_link">
-    <mu1>0.9</mu1>
-    <mu2>0.9</mu2>
-  </gazebo>
-  <link name="l_indexmid_link">
-    <xacro:unless value="${disable_mesh}"> <visual>
-      <origin xyz="0 0.03747 0.162972" rpy="0 -0 0"/>
-      <geometry>
-        <mesh filename="package://aero_description/meshes/aero_upper_meshes/LARM_INDEX_LINK3_mesh.dae" scale="1 1 1" />
-      </geometry>
-    </visual> </xacro:unless>
-    <xacro:unless value="${disable_mesh}"> <collision>
-      <origin xyz="0 0.03747 0.162972" rpy="0 -0 0"/>
-      <geometry>
-        <mesh filename="package://aero_description/meshes/aero_upper_meshes/LARM_INDEX_LINK3_mesh.dae" scale="1 1 1" />
-      </geometry>
-    </collision> </xacro:unless>
-    <inertial>
-      <mass value="0" />
-      <origin xyz="0 0 0" rpy="0 -0 0"/>
-      <inertia ixx="0" ixy="0" ixz="0" iyy="0" iyz="0" izz="0"/>
-    </inertial>
-  </link>
-  <gazebo reference="l_indexmid_link">
-    <mu1>0.9</mu1>
-    <mu2>0.9</mu2>
-  </gazebo>
-  <link name="l_indexend_link">
-    <xacro:unless value="${disable_mesh}"> <visual>
-      <origin xyz="0 0.022355 0.079645" rpy="0 -0 0 "/>
-      <geometry>
-        <mesh filename="package://aero_description/meshes/aero_upper_meshes/LARM_THUMB_LINK_mesh.dae" scale="1 1 1" />
-      </geometry>
-    </visual> </xacro:unless>
-    <xacro:unless value="${disable_mesh}"> <collision>
-      <origin xyz="0 0.022355 0.079645" rpy="0 -0 0 "/>
-      <geometry>
-        <mesh filename="package://aero_description/meshes/aero_upper_meshes/LARM_THUMB_LINK_mesh.dae" scale="1 1 1" />
-      </geometry>
-    </collision> </xacro:unless>
-    <inertial>
-      <mass value="0" />
-      <origin xyz="0 0 0" rpy="0 -0 0"/>
-      <inertia ixx="0" ixy="0" ixz="0" iyy="0" iyz="0" izz="0"/>
-    </inertial>
-  </link>
-  <gazebo reference="l_indexend_link">
     <mu1>0.9</mu1>
     <mu2>0.9</mu2>
@@ -550,15 +550,84 @@
     <mu2>0.9</mu2>
   </gazebo>
+  <link name="r_indexbase_link">
+    <xacro:unless value="${disable_mesh}"> <visual>
+      <origin xyz="0 0.013 0.115" rpy="0 -0 0 "/>
+      <geometry>
+        <mesh filename="package://aero_description/meshes/aero_upper_meshes/RARM_INDEX_LINK1_mesh.dae" scale="1 1 1" />
+      </geometry>
+    </visual> </xacro:unless>
+    <xacro:unless value="${disable_mesh}"> <collision>
+      <origin xyz="0 0.013 0.115" rpy="0 -0 0 "/>
+      <geometry>
+        <mesh filename="package://aero_description/meshes/aero_upper_meshes/RARM_INDEX_LINK1_mesh.dae" scale="1 1 1" />
+      </geometry>
+    </collision> </xacro:unless>
+    <inertial>
+      <mass value="0" />
+      <origin xyz="0 0 0" rpy="0 -0 0"/>
+      <inertia ixx="0" ixy="0" ixz="0" iyy="0" iyz="0" izz="0"/>
+    </inertial>
+  </link>
+  <gazebo reference="r_indexthumb_link">
+    <mu1>0.9</mu1>
+    <mu2>0.9</mu2>
+  </gazebo>
+  <link name="r_indexmid_link">
+    <xacro:unless value="${disable_mesh}"> <visual>
+      <origin xyz="0 -0.015754 0.149615" rpy="0 -0 0"/>
+      <geometry>
+        <mesh filename="package://aero_description/meshes/aero_upper_meshes/RARM_INDEX_LINK2_mesh.dae" scale="1 1 1" />
+      </geometry>
+    </visual> </xacro:unless>
+    <xacro:unless value="${disable_mesh}"> <collision>
+      <origin xyz="0 -0.015754 0.149615" rpy="0 -0 0"/>
+      <geometry>
+        <mesh filename="package://aero_description/meshes/aero_upper_meshes/RARM_INDEX_LINK2_mesh.dae" scale="1 1 1" />
+      </geometry>
+    </collision> </xacro:unless>
+    <inertial>
+      <mass value="0" />
+      <origin xyz="0 0 0" rpy="0 -0 0"/>
+      <inertia ixx="0" ixy="0" ixz="0" iyy="0" iyz="0" izz="0"/>
+    </inertial>
+  </link>
+  <gazebo reference="r_indexmid_link">
+    <mu1>0.9</mu1>
+    <mu2>0.9</mu2>
+  </gazebo>
+  <link name="r_indexend_link">
+    <xacro:unless value="${disable_mesh}"> <visual>
+      <origin xyz="0 -0.03747 0.162972" rpy="0 -0 0"/>
+      <geometry>
+        <mesh filename="package://aero_description/meshes/aero_upper_meshes/RARM_INDEX_LINK3_mesh.dae" scale="1 1 1" />
+      </geometry>
+    </visual> </xacro:unless>
+    <xacro:unless value="${disable_mesh}"> <collision>
+      <origin xyz="0 -0.03747 0.162972" rpy="0 -0 0"/>
+      <geometry>
+        <mesh filename="package://aero_description/meshes/aero_upper_meshes/RARM_INDEX_LINK3_mesh.dae" scale="1 1 1" />
+      </geometry>
+    </collision> </xacro:unless>
+    <inertial>
+      <mass value="0" />
+      <origin xyz="0 0 0" rpy="0 -0 0"/>
+      <inertia ixx="0" ixy="0" ixz="0" iyy="0" iyz="0" izz="0"/>
+    </inertial>
+  </link>
+  <gazebo reference="r_indexend_link">
+    <mu1>0.9</mu1>
+    <mu2>0.9</mu2>
+  </gazebo>
   <link name="r_thumb_link">
     <xacro:unless value="${disable_mesh}"> <visual>
-      <origin xyz="0 0.013 0.115" rpy="0 -0 0 "/>
-      <geometry>
-        <mesh filename="package://aero_description/meshes/aero_upper_meshes/RARM_INDEX_LINK1_mesh.dae" scale="1 1 1" />
-      </geometry>
-    </visual> </xacro:unless>
-    <xacro:unless value="${disable_mesh}"> <collision>
-      <origin xyz="0 0.013 0.115" rpy="0 -0 0 "/>
-      <geometry>
-        <mesh filename="package://aero_description/meshes/aero_upper_meshes/RARM_INDEX_LINK1_mesh.dae" scale="1 1 1" />
+      <origin xyz="0 -0.022355 0.079645" rpy="0 -0 0 "/>
+      <geometry>
+        <mesh filename="package://aero_description/meshes/aero_upper_meshes/RARM_THUMB_LINK_mesh.dae" scale="1 1 1" />
+      </geometry>
+    </visual> </xacro:unless>
+    <xacro:unless value="${disable_mesh}"> <collision>
+      <origin xyz="0 -0.022355 0.079645" rpy="0 -0 0 "/>
+      <geometry>
+        <mesh filename="package://aero_description/meshes/aero_upper_meshes/RARM_THUMB_LINK_mesh.dae" scale="1 1 1" />
       </geometry>
     </collision> </xacro:unless>
@@ -570,73 +639,4 @@
   </link>
   <gazebo reference="r_thumb_link">
-    <mu1>0.9</mu1>
-    <mu2>0.9</mu2>
-  </gazebo>
-  <link name="r_indexbase_link">
-    <xacro:unless value="${disable_mesh}"> <visual>
-      <origin xyz="0 -0.015754 0.149615" rpy="0 -0 0"/>
-      <geometry>
-        <mesh filename="package://aero_description/meshes/aero_upper_meshes/RARM_INDEX_LINK2_mesh.dae" scale="1 1 1" />
-      </geometry>
-    </visual> </xacro:unless>
-    <xacro:unless value="${disable_mesh}"> <collision>
-      <origin xyz="0 -0.015754 0.149615" rpy="0 -0 0"/>
-      <geometry>
-        <mesh filename="package://aero_description/meshes/aero_upper_meshes/RARM_INDEX_LINK2_mesh.dae" scale="1 1 1" />
-      </geometry>
-    </collision> </xacro:unless>
-    <inertial>
-      <mass value="0" />
-      <origin xyz="0 0 0" rpy="0 -0 0"/>
-      <inertia ixx="0" ixy="0" ixz="0" iyy="0" iyz="0" izz="0"/>
-    </inertial>
-  </link>
-  <gazebo reference="r_indexbase_link">
-    <mu1>0.9</mu1>
-    <mu2>0.9</mu2>
-  </gazebo>
-  <link name="r_indexmid_link">
-    <xacro:unless value="${disable_mesh}"> <visual>
-      <origin xyz="0 -0.03747 0.162972" rpy="0 -0 0"/>
-      <geometry>
-        <mesh filename="package://aero_description/meshes/aero_upper_meshes/RARM_INDEX_LINK3_mesh.dae" scale="1 1 1" />
-      </geometry>
-    </visual> </xacro:unless>
-    <xacro:unless value="${disable_mesh}"> <collision>
-      <origin xyz="0 -0.03747 0.162972" rpy="0 -0 0"/>
-      <geometry>
-        <mesh filename="package://aero_description/meshes/aero_upper_meshes/RARM_INDEX_LINK3_mesh.dae" scale="1 1 1" />
-      </geometry>
-    </collision> </xacro:unless>
-    <inertial>
-      <mass value="0" />
-      <origin xyz="0 0 0" rpy="0 -0 0"/>
-      <inertia ixx="0" ixy="0" ixz="0" iyy="0" iyz="0" izz="0"/>
-    </inertial>
-  </link>
-  <gazebo reference="r_indexmid_link">
-    <mu1>0.9</mu1>
-    <mu2>0.9</mu2>
-  </gazebo>
-  <link name="r_indexend_link">
-    <xacro:unless value="${disable_mesh}"> <visual>
-      <origin xyz="0 -0.022355 0.079645" rpy="0 -0 0 "/>
-      <geometry>
-        <mesh filename="package://aero_description/meshes/aero_upper_meshes/RARM_THUMB_LINK_mesh.dae" scale="1 1 1" />
-      </geometry>
-    </visual> </xacro:unless>
-    <xacro:unless value="${disable_mesh}"> <collision>
-      <origin xyz="0 -0.022355 0.079645" rpy="0 -0 0 "/>
-      <geometry>
-        <mesh filename="package://aero_description/meshes/aero_upper_meshes/RARM_THUMB_LINK_mesh.dae" scale="1 1 1" />
-      </geometry>
-    </collision> </xacro:unless>
-    <inertial>
-      <mass value="0" />
-      <origin xyz="0 0 0" rpy="0 -0 0"/>
-      <inertia ixx="0" ixy="0" ixz="0" iyy="0" iyz="0" izz="0"/>
-    </inertial>
-  </link>
-  <gazebo reference="r_indexend_link">
     <mu1>0.9</mu1>
     <mu2>0.9</mu2>
@@ -814,5 +814,5 @@
   <joint name="l_indexbase_joint" type="revolute">
     <parent link="l_hand_link"/>
-    <child  link="l_thumb_link"/>
+    <child  link="l_indexbase_link"/>
     <origin xyz="0 0.013 ${-0.115 - wrist_sensor_offset}" rpy="0 -0 0 "/>
     <axis   xyz="1 0 0"/>
@@ -824,17 +824,17 @@
   </gazebo>
   <joint name="l_indexmid_joint" type="revolute">
-    <parent link="l_thumb_link"/>
-    <child  link="l_indexbase_link"/>
-    <origin xyz="0 -0.028754 -0.034615" rpy="0 -0 0 "/>
-    <axis   xyz="1 0 0"/>
-    <limit lower="-3.14159" upper="3.14159" effort="100" velocity="0.5" />
-    <dynamics damping="0.2" friction="0" />
-  </joint>
-  <gazebo reference="l_indexmid_joint">
-    <implicitSpringDamper>0.4</implicitSpringDamper>
-  </gazebo>
-  <joint name="l_indexend_joint" type="revolute">
     <parent link="l_indexbase_link"/>
     <child  link="l_indexmid_link"/>
+    <origin xyz="0 -0.028754 -0.034615" rpy="0 -0 0 "/>
+    <axis   xyz="1 0 0"/>
+    <limit lower="-3.14159" upper="3.14159" effort="100" velocity="0.5" />
+    <dynamics damping="0.2" friction="0" />
+  </joint>
+  <gazebo reference="l_indexmid_joint">
+    <implicitSpringDamper>0.4</implicitSpringDamper>
+  </gazebo>
+  <joint name="l_indexend_joint" type="revolute">
+    <parent link="l_indexmid_link"/>
+    <child  link="l_indexend_link"/>
     <origin xyz="0 -0.021716 -0.013357" rpy="0 -0 0 "/>
     <axis   xyz="1 0 0"/>
@@ -847,5 +847,5 @@
   <joint name="l_thumb_joint" type="revolute">
     <parent link="l_hand_link"/>
-    <child  link="l_indexend_link"/>
+    <child  link="l_thumb_link"/>
     <origin xyz="0 -0.022355 ${-0.079645 - wrist_sensor_offset}" rpy="0 -0 0 "/>
     <axis   xyz="1 0 0"/>
@@ -1023,5 +1023,5 @@
   <joint name="r_indexbase_joint" type="revolute">
     <parent link="r_hand_link"/>
-    <child  link="r_thumb_link"/>
+    <child  link="r_indexbase_link"/>
     <origin xyz="0 -0.013 ${-0.115 - wrist_sensor_offset}" rpy="0 -0 0 "/>
     <axis   xyz="1 0 0"/>
@@ -1033,17 +1033,17 @@
   </gazebo>
   <joint name="r_indexmid_joint" type="revolute">
-    <parent link="r_thumb_link"/>
-    <child  link="r_indexbase_link"/>
-    <origin xyz="0 0.028754 -0.034615" rpy="0 -0 0 "/>
-    <axis   xyz="1 0 0"/>
-    <limit lower="-3.14159" upper="3.14159" effort="100" velocity="0.5" />
-    <dynamics damping="0.2" friction="0" />
-  </joint>
-  <gazebo reference="r_indexmid_joint">
-    <implicitSpringDamper>0.4</implicitSpringDamper>
-  </gazebo>
-  <joint name="r_indexend_joint" type="revolute">
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