Commit message: mod joint velocities

File: aero_shop/typeB_lifter/urdf/virtual_lifter.urdf.xacro (robot description, xacro)
@@ -37,5 +37,5 @@
       <origin xyz="0.0 0.0 -0.0" rpy="0 -0 0 "/>
       <axis   xyz="0 0 1"/>
-      <limit lower="${z_min}" upper="${z_max}" effort="100" velocity="0.15" />
+      <limit lower="${z_min}" upper="${z_max}" effort="100" velocity="0.11" />
       <dynamics damping="0.2" friction="0" />
     </joint>
@@ -46,5 +46,5 @@
       <origin xyz="0.0 0.0 0.5" rpy="0 -0 0 "/>
       <axis   xyz="1 0 0"/>
-      <limit lower="${x_min}" upper="${x_max}" effort="100" velocity="0.15" />
+      <limit lower="${x_min}" upper="${x_max}" effort="100" velocity="0.11" />
       <dynamics damping="0.2" friction="0" />
     </joint>

File: aero_shop/typeF_upperbody/urdf/aero_upper_typef.urdf.xacro (robot description, xacro)
@@ -467,5 +467,5 @@
     <axis   xyz="0 0.984808 -0.173648"/>
     <!-- from -88 to 15 degrees-->
-    <limit lower="-1.535" upper="0.261" effort="100" velocity="2.2" />
+    <limit lower="-1.535" upper="0.261" effort="100" velocity="0.5" />
     <dynamics damping="0.2" friction="0" />
   </joint>
@@ -484,5 +484,5 @@
     <axis   xyz="1 0 0"/>
     <!-- from 0 to 90 degrees-->
-    <limit lower="0" upper="1.5707" effort="100" velocity="1.5" />
+    <limit lower="0" upper="1.5707" effort="100" velocity="0.6" />
     <dynamics damping="0.2" friction="0" />
   </joint>
@@ -501,5 +501,5 @@
     <axis   xyz="0 0 1"/>
     <!-- from -180 to 45 degrees-->
-    <limit lower="-1.5707" upper="0.785398" effort="100" velocity="3.0" />
+    <limit lower="-1.5707" upper="0.785398" effort="100" velocity="0.5" />
     <dynamics damping="0.2" friction="0" />
   </joint>
@@ -518,5 +518,5 @@
     <axis   xyz="0 1 0"/>
     <!-- from -140 to 0 degrees-->
-    <limit lower="-2.44246" upper="0" effort="100" velocity="2.3" />
+    <limit lower="-2.44246" upper="0" effort="100" velocity="1.0" />
     <dynamics damping="0.2" friction="0" />
   </joint>
@@ -535,5 +535,5 @@
     <axis   xyz="0 0 1"/>
     <!-- from -180 to 180 degrees-->
-    <limit lower="-1.5707" upper="1.5707" effort="100" velocity="5.6" />
+    <limit lower="-1.5707" upper="1.5707" effort="100" velocity="1.5" />
     <dynamics damping="0.2" friction="0" />
   </joint>
@@ -552,5 +552,5 @@
     <axis   xyz="0 1 0"/>
     <!-- from -9 to 9 degrees-->
-    <limit lower="-0.15" upper="0.15" effort="100" velocity="2.2" />
+    <limit lower="-0.15" upper="0.15" effort="100" velocity="1.3" />
     <dynamics damping="0.2" friction="0" />
   </joint>
@@ -569,5 +569,5 @@
     <axis   xyz="1 0 0"/>
     <!-- from -75 to 40 degrees-->
-    <limit lower="-1.309" upper="0.698132" effort="100" velocity="2.2" />
+    <limit lower="-1.309" upper="0.698132" effort="100" velocity="1.3" />
     <dynamics damping="0.2" friction="0" />
   </joint>
@@ -634,5 +634,5 @@
     <axis   xyz="0 0.984808 0.173648"/>
     <!-- from -88 to 15 degrees-->
-    <limit lower="-1.535" upper="0.261" effort="100" velocity="2.2" />
+    <limit lower="-1.535" upper="0.261" effort="100" velocity="0.5" />
     <dynamics damping="0.2" friction="0" />
   </joint>
@@ -651,5 +651,5 @@
     <axis   xyz="1 0 0"/>
     <!-- from -90 to 0 degrees-->
-    <limit lower="-1.5707" upper="0" effort="100" velocity="1.5" />
+    <limit lower="-1.5707" upper="0" effort="100" velocity="0.6" />
     <dynamics damping="0.2" friction="0" />
   </joint>
@@ -668,5 +668,5 @@
     <axis   xyz="0 0 1"/>
     <!-- from -45 to 180 degrees-->
-    <limit lower="-0.785398" upper="1.5707" effort="100" velocity="3.0" />
+    <limit lower="-0.785398" upper="1.5707" effort="100" velocity="0.5" />
     <dynamics damping="0.2" friction="0" />
   </joint>
@@ -685,5 +685,5 @@
     <axis   xyz="0 1 0"/>
     <!-- from -140 to 0 degrees-->
-    <limit lower="-2.44246" upper="0" effort="100" velocity="2.3" />
+    <limit lower="-2.44246" upper="0" effort="100" velocity="1.0" />
     <dynamics damping="0.2" friction="0" />
   </joint>
@@ -702,5 +702,5 @@
     <axis   xyz="0 0 1"/>
     <!-- from -180 to 180 degrees-->
-    <limit lower="-1.5707" upper="1.5707" effort="100" velocity="5.6" />
+    <limit lower="-1.5707" upper="1.5707" effort="100" velocity="1.5" />
     <dynamics damping="0.2" friction="0" />
   </joint>
@@ -719,5 +719,5 @@
     <axis   xyz="0 1 0"/>
     <!-- from -9 to 9 degrees-->
-    <limit lower="-0.15" upper="0.15" effort="100" velocity="2.2" />
+    <limit lower="-0.15" upper="0.15" effort="100" velocity="1.3" />
     <dynamics damping="0.2" friction="0" />
   </joint>
@@ -736,5 +736,5 @@
     <axis   xyz="1 0 0"/>
     <!-- from -40 to 75 degrees-->
-    <limit lower="-0.698132" upper="1.309" effort="100" velocity="2.2" />
+    <limit lower="-0.698132" upper="1.309" effort="100" velocity="1.3" />
     <dynamics damping="0.2" friction="0" />
   </joint>
