Commit message: [aero_shop] fix urdf for using in gazebo, there is no effect to real robot

File: aero_shop/trx_s/urdf/trx_s.urdf.xacro (robot description, xacro)
@@ -6,4 +6,5 @@
        xmlns:xacro="http://ros.org/wiki/xacro">
   <xacro:include filename="$(find aero_description)/urdf/common.xacro" />
+  <xacro:include filename="$(find aero_description)/common_urdf/gazebo.xacro" />
   <property name="M_PI" value="3.1415926535897931" />
   <!-- ============================   trx_s   ============================ -->
@@ -30,8 +31,5 @@
     </inertial>
   </link>
-  <gazebo reference="${prefix}_hand_link">
-    <mu1>0.9</mu1>
-    <mu2>0.9</mu2>
-  </gazebo>
+  <xacro:gazebo_link_reference link_name="${prefix}_hand_link" />
   <link name="${prefix}_indexbase_link">
     <xacro:unless value="${disable_mesh}"> <visual>
@@ -53,8 +51,5 @@
     </inertial>
   </link>
-  <gazebo reference="${prefix}_indexthumb_link">
-    <mu1>0.9</mu1>
-    <mu2>0.9</mu2>
-  </gazebo>
+  <xacro:gazebo_link_reference link_name="${prefix}_indexthumb_link" />
   <link name="${prefix}_indexmid_link">
     <xacro:unless value="${disable_mesh}"> <visual>
@@ -76,8 +71,5 @@
     </inertial>
   </link>
-  <gazebo reference="${prefix}_indexmid_link">
-    <mu1>0.9</mu1>
-    <mu2>0.9</mu2>
-  </gazebo>
+  <xacro:gazebo_link_reference link_name="${prefix}_indexmid_link" />
   <link name="${prefix}_indexend_link">
     <xacro:unless value="${disable_mesh}"> <visual>
@@ -99,8 +91,5 @@
     </inertial>
   </link>
-  <gazebo reference="${prefix}_indexend_link">
-    <mu1>0.9</mu1>
-    <mu2>0.9</mu2>
-  </gazebo>
+  <xacro:gazebo_link_reference link_name="${prefix}_indexend_link" />
   <link name="${prefix}_thumb_link">
     <xacro:unless value="${disable_mesh}"> <visual>
@@ -122,8 +111,5 @@
     </inertial>
   </link>
-  <gazebo reference="${prefix}_thumb_link">
-    <mu1>0.9</mu1>
-    <mu2>0.9</mu2>
-  </gazebo>
+  <xacro:gazebo_link_reference link_name="${prefix}_thumb_link" />
   <joint name="${prefix}_indexbase_joint" type="revolute">
     <parent link="${prefix}_hand_link"/>
@@ -134,7 +120,5 @@
     <dynamics damping="0.2" friction="0" />
   </joint>
-  <gazebo reference="${prefix}_indexbase_joint">
-    <implicitSpringDamper>0.4</implicitSpringDamper>
-  </gazebo>
+  <xacro:gazebo_transmission joint_name="${prefix}_indexbase_joint" />
   <joint name="${prefix}_indexmid_joint" type="revolute">
     <parent link="${prefix}_indexbase_link"/>
@@ -145,7 +129,5 @@
     <dynamics damping="0.2" friction="0" />
   </joint>
-  <gazebo reference="${prefix}_indexmid_joint">
-    <implicitSpringDamper>0.4</implicitSpringDamper>
-  </gazebo>
+  <xacro:gazebo_transmission joint_name="${prefix}_indexmid_joint" />
   <joint name="${prefix}_indexend_joint" type="revolute">
     <parent link="${prefix}_indexmid_link"/>
@@ -156,12 +138,5 @@
     <dynamics damping="0.2" friction="0" />
   </joint>
-  <transmission type="pr2_mechanism_model/SimpleTransmission" name="${prefix}_indexend_joint_trans" >
-    <actuator name="${prefix}_indexend_joint_motor" />
-    <joint name="${prefix}_indexend_joint" />
-    <mechanicalReduction>1</mechanicalReduction>
-  </transmission>
-  <gazebo reference="${prefix}_indexend_joint">
-    <implicitSpringDamper>0.4</implicitSpringDamper>
-  </gazebo>
+  <xacro:gazebo_transmission joint_name="${prefix}_indexend_joint" />
   <joint name="${prefix}_thumb_joint" type="revolute">
     <parent link="${prefix}_hand_link"/>
@@ -172,12 +147,5 @@
     <dynamics damping="0.2" friction="0" />
   </joint>
-  <transmission type="pr2_mechanism_model/SimpleTransmission" name="${prefix}_thumb_joint_trans" >
-    <actuator name="${prefix}_thumb_joint_motor" />
-    <joint name="${prefix}_thumb_joint" />
-    <mechanicalReduction>1</mechanicalReduction>
-  </transmission>
-  <gazebo reference="${prefix}_thumb_joint">
-    <implicitSpringDamper>0.4</implicitSpringDamper>
-  </gazebo>
+  <xacro:gazebo_transmission joint_name="${prefix}_thumb_joint" />
   <!-- for ik eef link-->
   <link name="${prefix}_eef_grasp_link"/>

File: aero_shop/typeB_lifter/urdf/lifter.urdf.xacro (robot description, xacro)
@@ -15,4 +15,5 @@
        xmlns:xacro="http://ros.org/wiki/xacro">
   <xacro:include filename="$(find aero_description)/urdf/common.xacro" />
+  <xacro:include filename="$(find aero_description)/common_urdf/gazebo.xacro" />
   <xacro:macro name="lifter" params="base_link">
     <link name="${base_link}">
@@ -35,8 +36,5 @@
       </inertial>
     </link>
-    <gazebo reference="${base_link}">
-      <mu1>0.9</mu1>
-      <mu2>0.9</mu2>
-    </gazebo>
+    <xacro:gazebo_link_reference link_name="${base_link}" />
     <link name="leg_shank_link">
       <visual>
@@ -47,5 +45,5 @@
       </visual>
       <collision>
-        <origin xyz="0.0 0.0 0.0" rpy="0 -0 0"/>
+        <origin xyz="0.0 0.0 0" rpy="3.1415 -0 0"/>
         <geometry>
           <mesh filename="package://aero_description/meshes/typeB_lifter/lifter_bone.dae" scale="1 1 1" />
@@ -58,8 +56,5 @@
       </inertial>
     </link>
-    <gazebo reference="leg_shank_link">
-      <mu1>0.9</mu1>
-      <mu2>0.9</mu2>
-    </gazebo>
+    <xacro:gazebo_link_reference link_name="leg_shank_link" />
     <link name="leg_knee_link">
       <visual>
@@ -70,5 +65,5 @@
       </visual>
       <collision>
-        <origin xyz="0.0 0.0 0.0" rpy="0 -0 0"/>
+        <origin xyz="0.0 0.0 0" rpy="3.1415 -0 0"/>
         <geometry>
           <mesh filename="package://aero_description/meshes/typeB_lifter/lifter_knee.dae" scale="1 1 1" />
@@ -81,8 +76,5 @@
       </inertial>
     </link>
-    <gazebo reference="leg_knee_link">
-      <mu1>0.9</mu1>
-      <mu2>0.9</mu2>
-    </gazebo>
+    <xacro:gazebo_link_reference link_name="leg_knee_link" />
     <link name="leg_thigh_link">
       <visual>
@@ -93,5 +85,5 @@
       </visual>
       <collision>
-        <origin xyz="0.0 0.0 0.0" rpy="0 -0 0"/>
+        <origin xyz="0 0 0.25" rpy="0 0 0"/>
         <geometry>
           <mesh filename="package://aero_description/meshes/typeB_lifter/lifter_bone.dae" scale="1 1 1" />
@@ -104,8 +96,5 @@
       </inertial>
     </link>
-    <gazebo reference="leg_thigh_link">
-      <mu1>0.9</mu1>
-      <mu2>0.9</mu2>
-    </gazebo>
+    <xacro:gazebo_link_reference link_name="leg_thigh_link" />
     <link name="leg_base_link">
       <visual>
@@ -116,5 +105,5 @@
       </visual>
       <collision>
-        <origin xyz="0 0 0" rpy="0 -0 0"/>
+        <origin xyz="0 0 0.05" rpy="3.1415920 0 0"/>
         <geometry>
           <mesh filename="package://aero_description/meshes/typeB_lifter/lifter_base.dae" scale="1 1 1" />
@@ -127,8 +116,5 @@
       </inertial>
     </link>
-    <gazebo reference="leg_base_link">
-      <mu1>0.9</mu1>
-      <mu2>0.9</mu2>
-    </gazebo>
+    <xacro:gazebo_link_reference link_name="leg_base_link" />
     <link name="lifter_top_link">
       <visual>
@@ -150,8 +136,5 @@
       </inertial>
     </link>
-    <gazebo reference="lifter_top_link">
-      <mu1>0.9</mu1>
-      <mu2>0.9</mu2>
-    </gazebo>
+    <xacro:gazebo_link_reference link_name="lifter_top_link" />
     <joint name="lifter_top_connector" type="fixed">
       <parent link="leg_base_link"/>
@@ -171,14 +154,7 @@
       <origin xyz="0 0 0.12" rpy="0 0 0"/>
       <axis xyz="0 -1 0"/>
-      <limit effort="100" lower="-1.5707" upper="0" velocity="0.5"/>
-    </joint>
-    <transmission type="pr2_mechanism_model/SimpleTransmission" name="knee_joint_trans" >
-      <actuator name="knee_joint_motor" />
-      <joint name="knee_joint" />
-      <mechanicalReduction>1</mechanicalReduction>
-    </transmission>
-    <gazebo reference="knee_joint">
-      <implicitSpringDamper>0.4</implicitSpringDamper>
-    </gazebo>
+      <limit effort="1000" lower="-1.5707" upper="0" velocity="0.5"/>
+    </joint>
+    <xacro:gazebo_transmission joint_name="knee_joint" />
     <joint name="ankle_joint" type="revolute">
       <parent link="${base_link}"/>
@@ -186,15 +162,8 @@
       <origin xyz="0 0 0.05" rpy="0 0 0"/>
       <axis   xyz="0 -1 0"/>
-      <limit lower="0" upper="1.5707" effort="100" velocity="0.5" />
+      <limit effort="1000" lower="0" upper="1.5707" velocity="0.5" />
       <dynamics damping="0.2" friction="0" />
     </joint>
-    <transmission type="pr2_mechanism_model/SimpleTransmission" name="ankle_joint_trans" >
-      <actuator name="ankle_joint_motor" />
-      <joint name="ankle_joint" />
-      <mechanicalReduction>1</mechanicalReduction>
-    </transmission>
-    <gazebo reference="ankle_joint">
-      <implicitSpringDamper>0.4</implicitSpringDamper>
-    </gazebo>
+    <xacro:gazebo_transmission joint_name="ankle_joint" />
 <!--- mimic joints -->
 <!-- requried -->
@@ -214,4 +183,9 @@
         <origin xyz="0 0 0.25" rpy="0 0 0"/>
       </visual>
+      <inertial> <!-- for gazebo visualization -->
+        <mass value="0.4"/>
+        <origin rpy="0 0 0" xyz="-0.04 0.0 0.14"/>
+        <inertia ixx="0.001" ixy="0" ixz="0" iyy="0.001" iyz="0" izz="0.001"/>
+      </inertial>
     </link>
     <link name="leg_thigh_link_dummy">
@@ -222,4 +196,9 @@
         <origin xyz="0 0 0.25" rpy="0 0 0"/>
       </visual>
+      <inertial> <!-- for gazebo visualization -->
+        <mass value="0.4"/>
+        <origin rpy="0 0 0" xyz="-0.04 0.0 0.14"/>
+        <inertia ixx="0.001" ixy="0" ixz="0" iyy="0.001" iyz="0" izz="0.001"/>
+      </inertial>
     </link>
     <joint name="ankle_joint_dummy" type="continuous">

File: aero_shop/typeD_wheel/urdf/wheels.urdf.xacro (robot description, xacro)
@@ -15,4 +15,5 @@
        xmlns:xacro="http://ros.org/wiki/xacro">
   <xacro:include filename="$(find aero_description)/urdf/common.xacro" />
+  <xacro:include filename="$(find aero_description)/common_urdf/gazebo.xacro" />
   <xacro:property name="wheel_radius" value="0.075"/>
   <xacro:macro name="wheels" params="base_link disable_mesh:=false">
@@ -26,157 +27,139 @@
       </visual> </xacro:unless>
       <xacro:unless value="${disable_mesh}"> <collision>
+        <!--origin xyz="0.0 0.0 0.0" rpy="0 -0 0"/>
+        <geometry>
+          <mesh filename="package://aero_description/meshes/typeD_wheel/wheels_base.dae" scale="1 1 1" />
+        </geometry-->
+        <origin xyz="0.018 0.0 0.0375" rpy="0 -0 0"/>
+        <geometry>
+          <box size="0.72 0.52 0.149" />
+        </geometry>
+      </collision> </xacro:unless>
+      <inertial>
+        <mass value="10" />
+        <origin xyz="0 0 0" rpy="0 -0 0.09"/>
+        <inertia ixx="0.528" ixy="0" ixz="0" iyy="2.02" iyz="0" izz="2.35"/>
+      </inertial>
+    </link>
+    <xacro:gazebo_link_reference link_name="wheel_base_link" />
+    <link name="wheels_top_link">
+      <xacro:unless value="${disable_mesh}"> <visual>
         <origin xyz="0.0 0.0 0.0" rpy="0 -0 0"/>
         <geometry>
-          <mesh filename="package://aero_description/meshes/typeD_wheel/wheels_base.dae" scale="1 1 1" />
-        </geometry>
-      </collision> </xacro:unless>
-      <inertial>
-        <mass value="10" />
-        <origin xyz="0 0 0" rpy="0 -0 0.09"/>
-        <inertia ixx="0.528" ixy="0" ixz="0" iyy="2.02" iyz="0" izz="2.35"/>
-      </inertial>
-    </link>
-    <gazebo reference="wheel_base_link">
-      <mu1>0.9</mu1>
-      <mu2>0.9</mu2>
-    </gazebo>
-    <link name="wheels_top_link">
-      <xacro:unless value="${disable_mesh}"> <visual>
+          <mesh filename="package://aero_description/meshes/typeD_wheel/wheels_top.dae" scale="1 1 1" />
+        </geometry>
+      </visual> </xacro:unless>
+      <!-- no collision geometry -->
+      <inertial>
+        <mass value="10" />
+        <origin xyz="0 0 0" rpy="0 -0 0"/>
+        <inertia ixx="0.528" ixy="0" ixz="0" iyy="2.02" iyz="0" izz="2.35"/>
+      </inertial>
+    </link>
+    <xacro:gazebo_link_reference link_name="wheels_top_link" />
+    <link name="wheels_front_left_mecanum">
+      <xacro:unless value="${disable_mesh}"> <visual>
+        <origin xyz="0.0 0.0 0.0" rpy="-1.57079632679 0 0"/>
+        <geometry>
+          <mesh filename="package://aero_description/meshes/typeD_wheel/wheels_mecanum.dae" scale="1 1 1" />
+        </geometry>
+      </visual> </xacro:unless>
+      <xacro:unless value="${disable_mesh}"> <collision>
+        <origin xyz="0.0 0.0 0.0" rpy="-1.57079632679 0 0"/>
+        <geometry>
+          <!--cylinder length="0.046" radius="0.076" /-->
+          <box size="0.152 0.152 0.046" />
+        </geometry>
+      </collision> </xacro:unless>
+      <inertial>
+        <mass value="10" />
+        <origin xyz="0 0 0" rpy="0 -0 0"/>
+        <inertia ixx="0.528" ixy="0" ixz="0" iyy="2.02" iyz="0" izz="2.35"/>
+      </inertial>
+    </link>
+    <xacro:gazebo_link_reference link_name="wheels_front_left_mecanum" />
+    <link name="wheels_front_right_mecanum">
+      <xacro:unless value="${disable_mesh}"> <visual>
+        <origin xyz="0.0 0.0 0.0" rpy="-1.57079632679 0 0"/>
+        <geometry>
+          <mesh filename="package://aero_description/meshes/typeD_wheel/wheels_mecanum.dae" scale="1 1 1" />
+        </geometry>
+      </visual> </xacro:unless>
+      <xacro:unless value="${disable_mesh}"> <collision>
+        <origin xyz="0.0 0.0 0.0" rpy="-1.57079632679 0 0"/>
+        <geometry>
+          <!--cylinder length="0.046" radius="0.076" /-->
+          <box size="0.152 0.152 0.046" />
+        </geometry>
+      </collision> </xacro:unless>
+      <inertial>
+        <mass value="10" />
+        <origin xyz="0 0 0" rpy="0 -0 0"/>
+        <inertia ixx="0.528" ixy="0" ixz="0" iyy="2.02" iyz="0" izz="2.35"/>
+      </inertial>
+    </link>
+    <xacro:gazebo_link_reference link_name="wheels_front_left_mecanum" />
+    <link name="wheels_rear_left_mecanum">
+      <xacro:unless value="${disable_mesh}"> <visual>
+        <origin xyz="0.0 0.0 0.0" rpy="-1.57079632679 0 0"/>
+        <geometry>
+          <mesh filename="package://aero_description/meshes/typeD_wheel/wheels_mecanum.dae" scale="1 1 1" />
+        </geometry>
+      </visual> </xacro:unless>
+      <xacro:unless value="${disable_mesh}"> <collision>
+        <origin xyz="0.0 0.0 0.0" rpy="-1.57079632679 0 0"/>
+        <geometry>
+          <!--cylinder length="0.046" radius="0.076" /-->
+          <box size="0.152 0.152 0.046" />
+        </geometry>
+      </collision> </xacro:unless>
+      <inertial>
+        <mass value="10" />
+        <origin xyz="0 0 0" rpy="0 -0 0"/>
+        <inertia ixx="0.528" ixy="0" ixz="0" iyy="2.02" iyz="0" izz="2.35"/>
+      </inertial>
+    </link>
+    <xacro:gazebo_link_reference link_name="wheels_rear_left_mecanum" />
+    <link name="wheels_rear_right_mecanum">
+      <xacro:unless value="${disable_mesh}"> <visual>
+        <origin xyz="0.0 0.0 0.0" rpy="-1.57079632679 0 0"/>
+        <geometry>
+          <mesh filename="package://aero_description/meshes/typeD_wheel/wheels_mecanum.dae" scale="1 1 1" />
+        </geometry>
+      </visual> </xacro:unless>
+      <xacro:unless value="${disable_mesh}"> <collision>
+        <origin xyz="0.0 0.0 0.0" rpy="-1.57079632679 0 0"/>
+        <geometry>
+          <!--cylinder length="0.046" radius="0.076" /-->
+          <box size="0.152 0.152 0.046" />
+        </geometry>
+      </collision> </xacro:unless>
+      <inertial>
+        <mass value="10" />
+        <origin xyz="0 0 0" rpy="0 -0 0"/>
+        <inertia ixx="0.528" ixy="0" ixz="0" iyy="2.02" iyz="0" izz="2.35"/>
+      </inertial>
+    </link>
+    <xacro:gazebo_link_reference link_name="wheels_rear_right_mecanum" />
+    <link name="wheels_base_laser_link">
+      <xacro:unless value="${disable_mesh}"> <visual>
+        <origin xyz="0.0 0.0 0.0" rpy="0 0 0"/>
+        <geometry>
+          <mesh filename="package://aero_description/meshes/typeD_wheel/wheels_urg.dae" scale="1 1 1" />
+        </geometry>
+      </visual> </xacro:unless>
+      <xacro:unless value="${disable_mesh}"> <collision>
         <origin xyz="0.0 0.0 0.0" rpy="0 -0 0"/>
         <geometry>
-          <mesh filename="package://aero_description/meshes/typeD_wheel/wheels_top.dae" scale="1 1 1" />
-        </geometry>
-      </visual> </xacro:unless>
-      <xacro:unless value="${disable_mesh}"> <collision>
-        <origin xyz="0.0 0.0 0.0" rpy="0 -0 0"/>
-        <geometry>
-          <mesh filename="package://aero_description/meshes/typeD_wheel/wheels_top.dae" scale="1 1 1" />
-        </geometry>
-      </collision> </xacro:unless>
-      <inertial>
-        <mass value="10" />
-        <origin xyz="0 0 0" rpy="0 -0 0"/>
-        <inertia ixx="0.528" ixy="0" ixz="0" iyy="2.02" iyz="0" izz="2.35"/>
-      </inertial>
-    </link>
-    <gazebo reference="wheels_top_link">
-      <mu1>0.9</mu1>
-      <mu2>0.9</mu2>
-    </gazebo>
-    <link name="wheels_front_left_mecanum">
-      <xacro:unless value="${disable_mesh}"> <visual>
-        <origin xyz="0.0 0.0 0.0" rpy="-1.57079632679 0 0"/>
-        <geometry>
-          <mesh filename="package://aero_description/meshes/typeD_wheel/wheels_mecanum.dae" scale="1 1 1" />
-        </geometry>
-      </visual> </xacro:unless>
-      <xacro:unless value="${disable_mesh}"> <collision>
-        <origin xyz="0.0 0.0 0.0" rpy="0 -0 0"/>
-        <geometry>
-          <mesh filename="package://aero_description/meshes/typeD_wheel/wheels_mecanum.dae" scale="1 1 1" />
-        </geometry>
-      </collision> </xacro:unless>
-      <inertial>
-        <mass value="10" />
-        <origin xyz="0 0 0" rpy="0 -0 0"/>
-        <inertia ixx="0.528" ixy="0" ixz="0" iyy="2.02" iyz="0" izz="2.35"/>
-      </inertial>
-    </link>
-    <gazebo reference="wheels_front_left_mecanum">
-      <mu1>0.9</mu1>
-      <mu2>0.9</mu2>
-    </gazebo>
-    <link name="wheels_front_right_mecanum">
-      <xacro:unless value="${disable_mesh}"> <visual>
-        <origin xyz="0.0 0.0 0.0" rpy="-1.57079632679 0 0"/>
-        <geometry>
-          <mesh filename="package://aero_description/meshes/typeD_wheel/wheels_mecanum.dae" scale="1 1 1" />
-        </geometry>
-      </visual> </xacro:unless>
-      <xacro:unless value="${disable_mesh}"> <collision>
-        <origin xyz="0.0 0.0 0.0" rpy="0 -0 0"/>
-        <geometry>
-          <mesh filename="package://aero_description/meshes/typeD_wheel/wheels_mecanum.dae" scale="1 1 1" />
-        </geometry>
-      </collision> </xacro:unless>
-      <inertial>
-        <mass value="10" />
-        <origin xyz="0 0 0" rpy="0 -0 0"/>
-        <inertia ixx="0.528" ixy="0" ixz="0" iyy="2.02" iyz="0" izz="2.35"/>
-      </inertial>
-    </link>
-    <gazebo reference="wheels_front_left_mecanum">
-      <mu1>0.9</mu1>
-      <mu2>0.9</mu2>
-    </gazebo>
-    <link name="wheels_rear_left_mecanum">
-      <xacro:unless value="${disable_mesh}"> <visual>
-        <origin xyz="0.0 0.0 0.0" rpy="-1.57079632679 0 0"/>
-        <geometry>
-          <mesh filename="package://aero_description/meshes/typeD_wheel/wheels_mecanum.dae" scale="1 1 1" />
-        </geometry>
-      </visual> </xacro:unless>
-      <xacro:unless value="${disable_mesh}"> <collision>
-        <origin xyz="0.0 0.0 0.0" rpy="0 -0 0"/>
-        <geometry>
-          <mesh filename="package://aero_description/meshes/typeD_wheel/wheels_mecanum.dae" scale="1 1 1" />
-        </geometry>
-      </collision> </xacro:unless>
-      <inertial>
-        <mass value="10" />
-        <origin xyz="0 0 0" rpy="0 -0 0"/>
-        <inertia ixx="0.528" ixy="0" ixz="0" iyy="2.02" iyz="0" izz="2.35"/>
-      </inertial>
-    </link>
-    <gazebo reference="wheels_rear_left_mecanum">
-      <mu1>0.9</mu1>
-      <mu2>0.9</mu2>
-    </gazebo>
-    <link name="wheels_rear_right_mecanum">
-      <xacro:unless value="${disable_mesh}"> <visual>
-        <origin xyz="0.0 0.0 0.0" rpy="-1.57079632679 0 0"/>
-        <geometry>
-          <mesh filename="package://aero_description/meshes/typeD_wheel/wheels_mecanum.dae" scale="1 1 1" />
-        </geometry>
-      </visual> </xacro:unless>
-      <xacro:unless value="${disable_mesh}"> <collision>
-        <origin xyz="0.0 0.0 0.0" rpy="0 -0 0"/>
-        <geometry>
-          <mesh filename="package://aero_description/meshes/typeD_wheel/wheels_mecanum.dae" scale="1 1 1" />
-        </geometry>
-      </collision> </xacro:unless>
-      <inertial>
-        <mass value="10" />
-        <origin xyz="0 0 0" rpy="0 -0 0"/>
-        <inertia ixx="0.528" ixy="0" ixz="0" iyy="2.02" iyz="0" izz="2.35"/>
-      </inertial>
-    </link>
-    <gazebo reference="wheels_rear_right_mecanum">
-      <mu1>0.9</mu1>
-      <mu2>0.9</mu2>
-    </gazebo>
-    <link name="wheels_base_laser_link">
-      <xacro:unless value="${disable_mesh}"> <visual>
-        <origin xyz="0.0 0.0 0.0" rpy="0 0 0"/>
-        <geometry>
           <mesh filename="package://aero_description/meshes/typeD_wheel/wheels_urg.dae" scale="1 1 1" />
         </geometry>
-      </visual> </xacro:unless>
-      <xacro:unless value="${disable_mesh}"> <collision>
-        <origin xyz="0.0 0.0 0.0" rpy="0 -0 0"/>
-        <geometry>
-          <mesh filename="package://aero_description/meshes/typeD_wheel/wheels_urg.dae" scale="1 1 1" />
-        </geometry>
-      </collision> </xacro:unless>
-      <inertial>
-        <mass value="10" />
-        <origin xyz="0 0 0" rpy="0 -0 0"/>
-        <inertia ixx="0.528" ixy="0" ixz="0" iyy="2.02" iyz="0" izz="2.35"/>
-      </inertial>
-    </link>
-    <gazebo reference="wheels_base_laser_link">
-      <mu1>0.9</mu1>
-      <mu2>0.9</mu2>
-    </gazebo>
+      </collision> </xacro:unless>
+      <inertial>
+        <mass value="10" />
+        <origin xyz="0 0 0" rpy="0 -0 0"/>
+        <inertia ixx="0.528" ixy="0" ixz="0" iyy="2.02" iyz="0" izz="2.35"/>
+      </inertial>
+    </link>
+    <xacro:gazebo_link_reference link_name="wheels_base_laser_link" />
     <joint name="base_link_to_wheel_base_link_connector" type="fixed">
       <parent link="${base_link}"/>
