Commit message: [aero_shop] fix urdf for using in gazebo, there is no effect to real robot

File: aero_shop/typeF_upperbody/urdf/aero_upper_typef.urdf.xacro (robot description, xacro)
@@ -6,4 +6,5 @@
        xmlns:xacro="http://ros.org/wiki/xacro">
   <xacro:include filename="$(find aero_description)/urdf/common.xacro" />
+  <xacro:include filename="$(find aero_description)/common_urdf/gazebo.xacro" />
   <xacro:property name="wrist_sensor_offset" value="0.0"/>
   <!-- ============================   aero_upper   ============================ -->
@@ -28,8 +29,5 @@
     </inertial>
   </link>
-  <gazebo reference="${base_link}">
-    <mu1>0.9</mu1>
-    <mu2>0.9</mu2>
-  </gazebo>
+  <xacro:gazebo_link_reference link_name="${base_link}" />
   <link name="hip_sphere_link">
     <xacro:unless value="${disable_mesh}"> <visual>
@@ -51,8 +49,5 @@
     </inertial>
   </link>
-  <gazebo reference="hip_sphere_link">
-    <mu1>0.9</mu1>
-    <mu2>0.9</mu2>
-  </gazebo>
+  <xacro:gazebo_link_reference link_name="hip_sphere_link" />
   <link name="hip_center">
     <inertial>
@@ -62,8 +57,5 @@
     </inertial>
   </link>
-  <gazebo reference="hip_center">
-    <mu1>0.9</mu1>
-    <mu2>0.9</mu2>
-  </gazebo>
+  <xacro:gazebo_link_reference link_name="hip_center" />
   <link name="body_link">
     <xacro:unless value="${disable_mesh}"> <visual>
@@ -85,8 +77,5 @@
     </inertial>
   </link>
-  <gazebo reference="body_link">
-    <mu1>0.9</mu1>
-    <mu2>0.9</mu2>
-  </gazebo>
+  <xacro:gazebo_link_reference link_name="body_link" />
   <link name="l_shoulder_link">
     <xacro:unless value="${disable_mesh}"> <visual>
@@ -108,8 +97,5 @@
     </inertial>
   </link>
-  <gazebo reference="l_shoulder_link">
-    <mu1>0.9</mu1>
-    <mu2>0.9</mu2>
-  </gazebo>
+  <xacro:gazebo_link_reference link_name="l_shoulder_link" />
   <link name="l_shoulder_center">
     <xacro:unless value="${disable_mesh}"> <visual>
@@ -131,8 +117,5 @@
     </inertial>
   </link>
-  <gazebo reference="l_shoulder_center">
-    <mu1>0.9</mu1>
-    <mu2>0.9</mu2>
-  </gazebo>
+  <xacro:gazebo_link_reference link_name="l_shoulder_center" />
   <link name="l_upperarm_link">
     <xacro:unless value="${disable_mesh}"> <visual>
@@ -150,12 +133,12 @@
     <inertial>
       <mass value="0.574" />
+      <!--origin xyz="0.005 0 -0.0654" rpy="0 -0 0"/>
+      <inertia ixx="0.00114" ixy="0" ixz="0" iyy="0.00117" iyz="0" izz="0.000269"/-->
+      <!-- fix for gazebo -->
       <origin xyz="0.005 0 -0.0654" rpy="0 -0 0"/>
-      <inertia ixx="0.00114" ixy="0" ixz="0" iyy="0.00117" iyz="0" izz="0.000269"/>
-    </inertial>
-  </link>
-  <gazebo reference="l_upperarm_link">
-    <mu1>0.9</mu1>
-    <mu2>0.9</mu2>
-  </gazebo>
+      <inertia ixx="0.00114" ixy="0" ixz="0" iyy="0.00117" iyz="0" izz="0.003"/>
+    </inertial>
+  </link>
+  <xacro:gazebo_link_reference link_name="l_upperarm_link" />
   <link name="l_elbow_link">
     <xacro:unless value="${disable_mesh}"> <visual>
@@ -173,12 +156,12 @@
     <inertial>
       <mass value="0.711" />
-      <origin xyz="0.0047 0 -0.0546" rpy="0 -0 0"/>
-      <inertia ixx="0.00178" ixy="0" ixz="0" iyy="0.00179" iyz="0" izz="0.000273"/>
-    </inertial>
-  </link>
-  <gazebo reference="l_elbow_link">
-    <mu1>0.9</mu1>
-    <mu2>0.9</mu2>
-  </gazebo>
+      <!--origin xyz="0.0047 0 -0.0546" rpy="0 -0 0"/>
+      <inertia ixx="0.00178" ixy="0" ixz="0" iyy="0.00179" iyz="0" izz="0.000273"/-->
+      <!-- fix for gazebo -->
+      <origin xyz="-0.03 0 -0.0546" rpy="0 -0 0"/>
+      <inertia ixx="0.00178" ixy="0" ixz="0" iyy="0.00179" iyz="0" izz="0.004"/>
+    </inertial>
+  </link>
+  <xacro:gazebo_link_reference link_name="l_elbow_link" />
   <link name="l_forearm_link">
     <xacro:unless value="${disable_mesh}"> <visual>
@@ -200,8 +183,5 @@
     </inertial>
   </link>
-  <gazebo reference="l_forearm_link">
-    <mu1>0.9</mu1>
-    <mu2>0.9</mu2>
-  </gazebo>
+  <xacro:gazebo_link_reference link_name="l_forearm_link" />
   <link name="l_wrist_center">
     <inertial>
@@ -211,8 +191,5 @@
     </inertial>
   </link>
-  <gazebo reference="l_wrist_center">
-    <mu1>0.9</mu1>
-    <mu2>0.9</mu2>
-  </gazebo>
+  <xacro:gazebo_link_reference link_name="l_wrist_center" />
   <link name="neck_link">
     <xacro:unless value="${disable_mesh}"> <visual>
@@ -231,11 +208,9 @@
       <mass value="0.341" />
       <origin xyz="0 0 0.0595" rpy="0 -0 0"/>
-      <inertia ixx="1.64186e-35" ixy="0" ixz="0" iyy="1.64186e-35" iyz="0" izz="0"/>
-    </inertial>
-  </link>
-  <gazebo reference="neck_link">
-    <mu1>0.9</mu1>
-    <mu2>0.9</mu2>
-  </gazebo>
+      <!--inertia ixx="1.64186e-35" ixy="0" ixz="0" iyy="1.64186e-35" iyz="0" izz="0"/-->
+      <inertia ixx="0.0001" ixy="0" ixz="0" iyy="0.0001" iyz="0" izz="0.001"/>
+    </inertial>
+  </link>
+  <xacro:gazebo_link_reference link_name="neck_link" />
   <link name="head_base_link">
     <xacro:unless value="${disable_mesh}"> <visual>
@@ -254,11 +229,8 @@
       <mass value="0.01" />
       <origin xyz="0 0 0" rpy="0 -0 0"/>
-      <inertia ixx="0.00001" ixy="0" ixz="0" iyy="0.00001" iyz="0" izz="0.00001"/>
-    </inertial>
-  </link>
-  <gazebo reference="head_base_link">
-    <mu1>0.9</mu1>
-    <mu2>0.9</mu2>
-  </gazebo>
+      <inertia ixx="0.0001" ixy="0" ixz="0" iyy="0.0001" iyz="0" izz="0.0001"/>
+    </inertial>
+  </link>
+  <xacro:gazebo_link_reference link_name="head_base_link" />
   <link name="head_link">
     <xacro:unless value="${disable_mesh}"> <visual>
@@ -276,12 +248,9 @@
     <inertial>
       <mass value="0.974" />
-      <origin xyz="0 0 0.038" rpy="0 -0 0"/>
-      <inertia ixx="0" ixy="0" ixz="0" iyy="0" iyz="0" izz="0"/>
-    </inertial>
-  </link>
-  <gazebo reference="head_link">
-    <mu1>0.9</mu1>
-    <mu2>0.9</mu2>
-  </gazebo>
+      <origin xyz="0 0 0.150" rpy="0 -0 0"/>
+      <inertia ixx="0.005" ixy="0" ixz="0" iyy="0.005" iyz="0" izz="0.005"/>
+    </inertial>
+  </link>
+  <xacro:gazebo_link_reference link_name="head_link" />
   <link name="r_shoulder_link">
     <xacro:unless value="${disable_mesh}"> <visual>
@@ -292,5 +261,5 @@
     </visual> </xacro:unless>
     <xacro:unless value="${disable_mesh}"> <collision>
-      <origin xyz="0 0 0" rpy="0 -0 0"/>
+      <origin xyz="0 0 0" rpy="0.174532925 -0 0"/>
       <geometry>
         <mesh filename="package://aero_description/meshes/typeF_upperbody/RARM_LINK1_mesh.dae" scale="1 1 1" />
@@ -303,8 +272,5 @@
     </inertial>
   </link>
-  <gazebo reference="r_shoulder_link">
-    <mu1>0.9</mu1>
-    <mu2>0.9</mu2>
-  </gazebo>
+  <xacro:gazebo_link_reference link_name="r_shoulder_link" />
   <link name="r_shoulder_center">
     <xacro:unless value="${disable_mesh}"> <visual>
@@ -326,8 +292,5 @@
     </inertial>
   </link>
-  <gazebo reference="r_shoulder_center">
-    <mu1>0.9</mu1>
-    <mu2>0.9</mu2>
-  </gazebo>
+  <xacro:gazebo_link_reference link_name="r_shoulder_center" />
   <link name="r_upperarm_link">
     <xacro:unless value="${disable_mesh}"> <visual>
@@ -345,12 +308,12 @@
     <inertial>
       <mass value="0.574" />
+      <!--origin xyz="0.005 0 -0.0654" rpy="0 -0 0"/>
+      <inertia ixx="0.00114" ixy="0" ixz="0" iyy="0.00117" iyz="0" izz="0.000269"/-->
+      <!-- fix for gazebo -->
       <origin xyz="0.005 0 -0.0654" rpy="0 -0 0"/>
-      <inertia ixx="0.00114" ixy="0" ixz="0" iyy="0.00117" iyz="0" izz="0.000269"/>
-    </inertial>
-  </link>
-  <gazebo reference="r_upperarm_link">
-    <mu1>0.9</mu1>
-    <mu2>0.9</mu2>
-  </gazebo>
+      <inertia ixx="0.00114" ixy="0" ixz="0" iyy="0.00117" iyz="0" izz="0.003"/>
+    </inertial>
+  </link>
+  <xacro:gazebo_link_reference link_name="r_upperarm_link" />
   <link name="r_elbow_link">
     <xacro:unless value="${disable_mesh}"> <visual>
@@ -361,5 +324,5 @@
     </visual> </xacro:unless>
     <xacro:unless value="${disable_mesh}"> <collision>
-      <origin xyz="-0.035 0 -0.070" rpy="0 -0 0"/>
+      <origin xyz="-0.035 0 -0.035" rpy="0 -0 0"/>
       <geometry>
         <mesh filename="package://aero_description/meshes/typeF_upperbody/RARM_LINK4_mesh.dae" scale="1 1 1" />
@@ -368,12 +331,12 @@
     <inertial>
       <mass value="0.711" />
-      <origin xyz="0.0047 0 -0.0546" rpy="0 -0 0"/>
-      <inertia ixx="0.00178" ixy="0" ixz="0" iyy="0.00179" iyz="0" izz="0.000273"/>
-    </inertial>
-  </link>
-  <gazebo reference="r_elbow_link">
-    <mu1>0.9</mu1>
-    <mu2>0.9</mu2>
-  </gazebo>
+      <!--origin xyz="0.0047 0 -0.0546" rpy="0 -0 0"/>
+      <inertia ixx="0.00178" ixy="0" ixz="0" iyy="0.00179" iyz="0" izz="0.000273"/-->
+      <!-- fix for gazebo -->
+      <origin xyz="-0.03 0 -0.0546" rpy="0 -0 0"/>
+      <inertia ixx="0.00178" ixy="0" ixz="0" iyy="0.00179" iyz="0" izz="0.004"/>
+    </inertial>
+  </link>
+  <xacro:gazebo_link_reference link_name="r_elbow_link" />
   <link name="r_forearm_link">
     <xacro:unless value="${disable_mesh}"> <visual>
@@ -395,8 +358,5 @@
     </inertial>
   </link>
-  <gazebo reference="r_forearm_link">
-    <mu1>0.9</mu1>
-    <mu2>0.9</mu2>
-  </gazebo>
+  <xacro:gazebo_link_reference link_name="r_forearm_link" />
   <link name="r_wrist_center">
     <inertial>
@@ -406,8 +366,5 @@
     </inertial>
   </link>
-  <gazebo reference="r_wrist_center">
-    <mu1>0.9</mu1>
-    <mu2>0.9</mu2>
-  </gazebo>
+  <xacro:gazebo_link_reference link_name="r_wrist_center" />
   <joint name="waist_y_joint" type="revolute">
     <parent link="${base_link}"/>
@@ -419,12 +376,5 @@
     <dynamics damping="0.2" friction="0" />
   </joint>
-  <transmission type="pr2_mechanism_model/SimpleTransmission" name="waist_y_joint_trans" >
-    <actuator name="waist_y_joint_motor" />
-    <joint name="waist_y_joint" />
-    <mechanicalReduction>1</mechanicalReduction>
-  </transmission>
-  <gazebo reference="waist_y_joint">
-    <implicitSpringDamper>0.4</implicitSpringDamper>
-  </gazebo>
+  <xacro:gazebo_transmission joint_name="waist_y_joint" />
   <joint name="waist_p_joint" type="revolute">
     <parent link="hip_sphere_link"/>
@@ -436,12 +386,5 @@
     <dynamics damping="0.2" friction="0" />
   </joint>
-  <transmission type="pr2_mechanism_model/SimpleTransmission" name="waist_p_joint_trans" >
-    <actuator name="waist_p_joint_motor" />
-    <joint name="waist_p_joint" />
-    <mechanicalReduction>1</mechanicalReduction>
-  </transmission>
-  <gazebo reference="waist_p_joint">
-    <implicitSpringDamper>0.4</implicitSpringDamper>
-  </gazebo>
+  <xacro:gazebo_transmission joint_name="waist_p_joint" />
   <joint name="waist_r_joint" type="revolute">
     <parent link="hip_center"/>
@@ -453,12 +396,5 @@
     <dynamics damping="0.2" friction="0" />
   </joint>
-  <transmission type="pr2_mechanism_model/SimpleTransmission" name="waist_r_joint_trans" >
-    <actuator name="waist_r_joint_motor" />
-    <joint name="waist_r_joint" />
-    <mechanicalReduction>1</mechanicalReduction>
-  </transmission>
-  <gazebo reference="waist_r_joint">
-    <implicitSpringDamper>0.4</implicitSpringDamper>
-  </gazebo>
+  <xacro:gazebo_transmission joint_name="waist_r_joint" />
   <joint name="l_shoulder_p_joint" type="revolute">
     <parent link="body_link"/>
@@ -470,12 +406,5 @@
     <dynamics damping="0.2" friction="0" />
   </joint>
-  <transmission type="pr2_mechanism_model/SimpleTransmission" name="l_shoulder_p_joint_trans" >
-    <actuator name="l_shoulder_p_joint_motor" />
-    <joint name="l_shoulder_p_joint" />
-    <mechanicalReduction>1</mechanicalReduction>
-  </transmission>
-  <gazebo reference="l_shoulder_p_joint">
-    <implicitSpringDamper>0.4</implicitSpringDamper>
-  </gazebo>
+  <xacro:gazebo_transmission joint_name="l_shoulder_p_joint" />
   <joint name="l_shoulder_r_joint" type="revolute">
     <parent link="l_shoulder_link"/>
@@ -487,12 +416,5 @@
     <dynamics damping="0.2" friction="0" />
   </joint>
-  <transmission type="pr2_mechanism_model/SimpleTransmission" name="l_shoulder_r_joint_trans" >
-    <actuator name="l_shoulder_r_joint_motor" />
-    <joint name="l_shoulder_r_joint" />
-    <mechanicalReduction>1</mechanicalReduction>
-  </transmission>
-  <gazebo reference="l_shoulder_r_joint">
-    <implicitSpringDamper>0.4</implicitSpringDamper>
-  </gazebo>
+  <xacro:gazebo_transmission joint_name="l_shoulder_r_joint" />
   <joint name="l_shoulder_y_joint" type="revolute">
     <parent link="l_shoulder_center"/>
@@ -504,12 +426,5 @@
     <dynamics damping="0.2" friction="0" />
   </joint>
-  <transmission type="pr2_mechanism_model/SimpleTransmission" name="l_shoulder_y_joint_trans" >
-    <actuator name="l_shoulder_y_joint_motor" />
-    <joint name="l_shoulder_y_joint" />
-    <mechanicalReduction>1</mechanicalReduction>
-  </transmission>
-  <gazebo reference="l_shoulder_y_joint">
-    <implicitSpringDamper>0.4</implicitSpringDamper>
-  </gazebo>
+  <xacro:gazebo_transmission joint_name="l_shoulder_y_joint" />
   <joint name="l_elbow_joint" type="revolute">
     <parent link="l_upperarm_link"/>
@@ -521,12 +436,5 @@
     <dynamics damping="0.2" friction="0" />
   </joint>
-  <transmission type="pr2_mechanism_model/SimpleTransmission" name="l_elbow_joint_trans" >
-    <actuator name="l_elbow_joint_motor" />
-    <joint name="l_elbow_joint" />
-    <mechanicalReduction>1</mechanicalReduction>
-  </transmission>
-  <gazebo reference="l_elbow_joint">
-    <implicitSpringDamper>0.4</implicitSpringDamper>
-  </gazebo>
+  <xacro:gazebo_transmission joint_name="l_elbow_joint" />
   <joint name="l_wrist_y_joint" type="revolute">
     <parent link="l_elbow_link"/>
@@ -538,12 +446,5 @@
     <dynamics damping="0.2" friction="0" />
   </joint>
-  <transmission type="pr2_mechanism_model/SimpleTransmission" name="l_wrist_y_joint_trans" >
-    <actuator name="l_wrist_y_joint_motor" />
-    <joint name="l_wrist_y_joint" />
-    <mechanicalReduction>1</mechanicalReduction>
-  </transmission>
-  <gazebo reference="l_wrist_y_joint">
-    <implicitSpringDamper>0.4</implicitSpringDamper>
-  </gazebo>
+  <xacro:gazebo_transmission joint_name="l_wrist_y_joint" />
   <joint name="l_wrist_p_joint" type="revolute">
     <parent link="l_forearm_link"/>
@@ -555,12 +456,5 @@
     <dynamics damping="0.2" friction="0" />
   </joint>
-  <transmission type="pr2_mechanism_model/SimpleTransmission" name="l_wrist_p_joint_trans" >
-    <actuator name="l_wrist_p_joint_motor" />
-    <joint name="l_wrist_p_joint" />
-    <mechanicalReduction>1</mechanicalReduction>
-  </transmission>
-  <gazebo reference="l_wrist_p_joint">
-    <implicitSpringDamper>0.4</implicitSpringDamper>
-  </gazebo>
+  <xacro:gazebo_transmission joint_name="l_wrist_p_joint" />
   <joint name="l_wrist_r_joint" type="revolute">
     <parent link="l_wrist_center"/>
@@ -572,12 +466,5 @@
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
Commit message: [aero_shop] fix urdf massages

File: aero_shop/trx_s/urdf/trx_s.urdf.xacro (robot description, xacro)
@@ -8,6 +8,6 @@
   <xacro:include filename="$(find aero_description)/common_urdf/gazebo.xacro" />
   <property name="M_PI" value="3.1415926535897931" />
-  <!-- ============================   trx_s   ============================ -->
   <xacro:macro name="trx_s" params="prefix:=r reflect:=1 disable_mesh:=false">
+  <!-- ============================   Hand(trx_s)   ============================ -->
     <!-- prefix is "r" or "l" -->
     <!-- reflect=1 is rightside, reflect=-1 is leftside -->
@@ -109,5 +109,5 @@
     <xacro:unless value="${disable_mesh}">
     <collision>
-      <origin rpy="0.63 0 0" xyz="0.0 ${reflect * 0.019645} -0.010355"/>
+      <origin rpy="${reflect * 0.63} 0 0" xyz="0.0 ${reflect * 0.019645} -0.010355"/>
       <geometry>
         <box size="0.012 0.008 0.050"/>
@@ -115,5 +115,5 @@
     </collision>
     <collision>
-      <origin rpy="0.1 0 0" xyz="0.0 ${reflect * 0.035645} -0.050355"/>
+      <origin rpy="${reflect * 0.1} 0 0" xyz="0.0 ${reflect * 0.035645} -0.050355"/>
       <geometry>
         <box size="0.012 0.008 0.050"/>

File: aero_shop/typeB_lifter/urdf/lifter.urdf.xacro (robot description, xacro)
@@ -17,4 +17,5 @@
   <xacro:include filename="$(find aero_description)/common_urdf/gazebo.xacro" />
   <xacro:macro name="lifter" params="base_link">
+  <!-- ============================   aero(typeB_lifter)   ============================ -->
     <link name="${base_link}">
       <visual>

File: aero_shop/typeC_lifter/urdf/lifter.urdf.xacro (robot description, xacro)
@@ -17,4 +17,5 @@
   <xacro:include filename="$(find aero_description)/common_urdf/gazebo.xacro" />
   <xacro:macro name="lifter" params="base_link">
+  <!-- ============================   aero(typeC_lifter)   ============================ -->
     <link name="${base_link}">
       <visual>

File: aero_shop/typeD_wheel/urdf/wheels.urdf.xacro (robot description, xacro)
@@ -18,4 +18,5 @@
   <xacro:property name="wheel_radius" value="0.075"/>
   <xacro:macro name="wheels" params="base_link disable_mesh:=false">
+  <!-- ============================   aero(typeD_wheels)   ============================ -->
     <link name="${base_link}"/>
     <link name="wheel_base_link">

File: aero_shop/typeF_upperbody/urdf/aero_upper_typef.urdf.xacro (robot description, xacro)
@@ -8,6 +8,6 @@
   <xacro:include filename="$(find aero_description)/common_urdf/gazebo.xacro" />
   <xacro:property name="wrist_sensor_offset" value="0.0"/>
-  <!-- ============================   aero_upper   ============================ -->
   <xacro:macro name="aero_upper" params="base_link disable_mesh:=false r_hand_link:=r_hand_link l_hand_link:=l_hand_link">
+  <!-- ============================   aero(typeF_upper)   ============================ -->
   <link name="${base_link}">
     <xacro:unless value="${disable_mesh}"> <visual>
@@ -166,5 +166,5 @@
   <link name="l_forearm_link">
     <xacro:unless value="${disable_mesh}"> <visual>
-      <origin xyz="0 0 0" rpy="0 -0 0"/>
+      <origin xyz="0 0 0" rpy="0 0 -1.5707963267948966"/>
       <geometry>
         <mesh filename="package://aero_description/meshes/typeF_upperbody/LARM_LINK5_mesh.dae" scale="1 1 1" />
@@ -172,5 +172,5 @@
     </visual> </xacro:unless>
     <xacro:unless value="${disable_mesh}"> <collision>
-      <origin xyz="0 0 0" rpy="0 -0 0"/>
+      <origin xyz="0 0 0" rpy="0 0 -1.5707963267948966"/>
       <geometry>
         <mesh filename="package://aero_description/meshes/typeF_upperbody/LARM_LINK5_mesh.dae" scale="1 1 1" />
@@ -180,5 +180,5 @@
       <mass value="0.132" />
       <origin xyz="0.006 0 -0.0738" rpy="0 -0 0"/>
-      <inertia ixx="0.000276" ixy="0" ixz="0" iyy="0.000286" iyz="0" izz="0.0001"/>
+      <inertia ixx="0.000276" ixy="0" ixz="0" iyy="0.000286" iyz="0" izz="0.004"/>
     </inertial>
   </link>
@@ -186,7 +186,7 @@
   <link name="l_wrist_center">
     <inertial>
-      <mass value="0.01" />
-      <origin xyz="0 0 0" rpy="0 -0 0"/>
-      <inertia ixx="0.00001" ixy="0" ixz="0" iyy="0.00001" iyz="0" izz="0.00001"/>
+      <mass value="0.05" />
+      <origin xyz="0 0 0" rpy="0 -0 0"/>
+      <inertia ixx="0.0001" ixy="0" ixz="0" iyy="0.0001" iyz="0" izz="0.0001"/>
     </inertial>
   </link>
@@ -341,5 +341,5 @@
   <link name="r_forearm_link">
     <xacro:unless value="${disable_mesh}"> <visual>
-      <origin xyz="0 0 0" rpy="0 -0 0"/>
+      <origin xyz="0 0 0" rpy="0 0 1.5707963267948966"/>
       <geometry>
         <mesh filename="package://aero_description/meshes/typeF_upperbody/RARM_LINK5_mesh.dae" scale="1 1 1" />
@@ -347,5 +347,5 @@
     </visual> </xacro:unless>
     <xacro:unless value="${disable_mesh}"> <collision>
-      <origin xyz="0 0 0" rpy="0 -0 0"/>
+      <origin xyz="0 0 0" rpy="0 0 1.5707963267948966"/>
       <geometry>
         <mesh filename="package://aero_description/meshes/typeF_upperbody/RARM_LINK5_mesh.dae" scale="1 1 1" />
@@ -355,5 +355,5 @@
       <mass value="0.132" />
       <origin xyz="0.006 0 -0.0738" rpy="0 -0 0"/>
-      <inertia ixx="0.000276" ixy="0" ixz="0" iyy="0.000286" iyz="0" izz="0.0001"/>
+      <inertia ixx="0.000276" ixy="0" ixz="0" iyy="0.000286" iyz="0" izz="0.004"/>
     </inertial>
   </link>
@@ -361,7 +361,7 @@
   <link name="r_wrist_center">
     <inertial>
-      <mass value="0.01" />
-      <origin xyz="0 0 0" rpy="0 -0 0"/>
-      <inertia ixx="0.00001" ixy="0" ixz="0" iyy="0.00001" iyz="0" izz="0.00001"/>
+      <mass value="0.05" />
+      <origin xyz="0 0 0" rpy="0 -0 0"/>
+      <inertia ixx="0.0001" ixy="0" ixz="0" iyy="0.0001" iyz="0" izz="0.0001"/>
     </inertial>
   </link>
