Commit message: [aero_shop, typeE_wheel] fix inertial infomation for gazebo

File: aero_shop/typeE_wheel/urdf/wheels.urdf.xacro (robot description, xacro)
@@ -15,7 +15,9 @@
        xmlns:xacro="http://ros.org/wiki/xacro">
   <xacro:include filename="$(find aero_description)/urdf/common.xacro" />
+  <xacro:include filename="$(find aero_description)/common_urdf/gazebo.xacro" />
   <xacro:property name="wheel_radius" value="0.075"/>
   <xacro:macro name="wheels" params="base_link disable_mesh:=false">
-    <link name="${base_link}"/>
+  <!-- ============================   aero(typeE_wheels)   ============================ -->
+  <link name="${base_link}"/>
     <link name="wheel_base_link">
       <xacro:unless value="${disable_mesh}"> <visual>
@@ -26,42 +28,35 @@
       </visual> </xacro:unless>
       <xacro:unless value="${disable_mesh}"> <collision>
+        <!--origin xyz="0.0 0.0 0.0" rpy="0 -0 0"/>
+        <geometry>
+          <mesh filename="package://aero_description/meshes/typeE_wheel/wheels_base.dae" scale="1 1 1" />
+        </geometry-->
+        <origin xyz="0.018 0.0 0.0375" rpy="0 -0 0"/>
+        <geometry>
+          <box size="0.72 0.52 0.149" />
+        </geometry>
+      </collision> </xacro:unless>
+      <inertial>
+        <mass value="70" />
+        <origin xyz="0 0 0.04" rpy="0 -0 0.0"/>
+        <inertia ixx="0.528" ixy="0" ixz="0" iyy="2.02" iyz="0" izz="2.35"/>
+      </inertial>
+    </link>
+    <xacro:gazebo_link_reference link_name="wheel_base_link" />
+    <link name="wheels_top_link">
+      <xacro:unless value="${disable_mesh}"> <visual>
         <origin xyz="0.0 0.0 0.0" rpy="0 -0 0"/>
         <geometry>
-          <mesh filename="package://aero_description/meshes/typeE_wheel/wheels_base.dae" scale="1 1 1" />
-        </geometry>
-      </collision> </xacro:unless>
-      <inertial>
-        <mass value="10" />
-        <origin xyz="0 0 0" rpy="0 -0 0.09"/>
-        <inertia ixx="0.528" ixy="0" ixz="0" iyy="2.02" iyz="0" izz="2.35"/>
-      </inertial>
-    </link>
-    <gazebo reference="wheel_base_link">
-      <mu1>0.9</mu1>
-      <mu2>0.9</mu2>
-    </gazebo>
-    <link name="wheels_top_link">
-      <xacro:unless value="${disable_mesh}"> <visual>
-        <origin xyz="0.0 0.0 0.0" rpy="0 -0 0"/>
-        <geometry>
           <mesh filename="package://aero_description/meshes/typeE_wheel/wheels_top.dae" scale="1 1 1" />
         </geometry>
       </visual> </xacro:unless>
-      <xacro:unless value="${disable_mesh}"> <collision>
-        <origin xyz="0.0 0.0 0.0" rpy="0 -0 0"/>
-        <geometry>
-          <mesh filename="package://aero_description/meshes/typeE_wheel/wheels_top.dae" scale="1 1 1" />
-        </geometry>
-      </collision> </xacro:unless>
-      <inertial>
-        <mass value="10" />
-        <origin xyz="0 0 0" rpy="0 -0 0"/>
-        <inertia ixx="0.528" ixy="0" ixz="0" iyy="2.02" iyz="0" izz="2.35"/>
-      </inertial>
-    </link>
-    <gazebo reference="wheels_top_link">
-      <mu1>0.9</mu1>
-      <mu2>0.9</mu2>
-    </gazebo>
+      <!-- no collision geometry -->
+      <inertial>
+        <mass value="1" />
+        <origin xyz="0 0 0" rpy="0 -0 0"/>
+        <inertia ixx="0.528" ixy="0" ixz="0" iyy="2.02" iyz="0" izz="2.35"/>
+      </inertial>
+    </link>
+    <xacro:gazebo_link_reference link_name="wheels_top_link" />
     <link name="wheels_front_left_mecanum">
       <xacro:unless value="${disable_mesh}"> <visual>
@@ -72,19 +67,17 @@
       </visual> </xacro:unless>
       <xacro:unless value="${disable_mesh}"> <collision>
-        <origin xyz="0.0 0.0 0.0" rpy="0 -0 0"/>
-        <geometry>
-          <mesh filename="package://aero_description/meshes/typeE_wheel/wheels_mecanum.dae" scale="1 1 1" />
-        </geometry>
-      </collision> </xacro:unless>
-      <inertial>
-        <mass value="10" />
-        <origin xyz="0 0 0" rpy="0 -0 0"/>
-        <inertia ixx="0.528" ixy="0" ixz="0" iyy="2.02" iyz="0" izz="2.35"/>
-      </inertial>
-    </link>
-    <gazebo reference="wheels_front_left_mecanum">
-      <mu1>0.9</mu1>
-      <mu2>0.9</mu2>
-    </gazebo>
+        <origin xyz="0.0 0.0 0.0" rpy="-1.57079632679 0 0"/>
+        <geometry>
+          <!--cylinder length="0.046" radius="0.076" /-->
+          <box size="0.152 0.152 0.046" />
+        </geometry>
+      </collision> </xacro:unless>
+      <inertial>
+        <mass value="1" />
+        <origin xyz="0 0 0" rpy="0 -0 0"/>
+        <inertia ixx="0.528" ixy="0" ixz="0" iyy="2.02" iyz="0" izz="2.35"/>
+      </inertial>
+    </link>
+    <xacro:gazebo_link_reference link_name="wheels_front_left_mecanum" />
     <link name="wheels_front_right_mecanum">
       <xacro:unless value="${disable_mesh}"> <visual>
@@ -95,19 +88,17 @@
       </visual> </xacro:unless>
       <xacro:unless value="${disable_mesh}"> <collision>
-        <origin xyz="0.0 0.0 0.0" rpy="0 -0 0"/>
-        <geometry>
-          <mesh filename="package://aero_description/meshes/typeE_wheel/wheels_mecanum.dae" scale="1 1 1" />
-        </geometry>
-      </collision> </xacro:unless>
-      <inertial>
-        <mass value="10" />
-        <origin xyz="0 0 0" rpy="0 -0 0"/>
-        <inertia ixx="0.528" ixy="0" ixz="0" iyy="2.02" iyz="0" izz="2.35"/>
-      </inertial>
-    </link>
-    <gazebo reference="wheels_front_left_mecanum">
-      <mu1>0.9</mu1>
-      <mu2>0.9</mu2>
-    </gazebo>
+        <origin xyz="0.0 0.0 0.0" rpy="-1.57079632679 0 0"/>
+        <geometry>
+          <!--cylinder length="0.046" radius="0.076" /-->
+          <box size="0.152 0.152 0.046" />
+        </geometry>
+      </collision> </xacro:unless>
+      <inertial>
+        <mass value="1" />
+        <origin xyz="0 0 0" rpy="0 -0 0"/>
+        <inertia ixx="0.528" ixy="0" ixz="0" iyy="2.02" iyz="0" izz="2.35"/>
+      </inertial>
+    </link>
+    <xacro:gazebo_link_reference link_name="wheels_front_left_mecanum" />
     <link name="wheels_rear_left_mecanum">
       <xacro:unless value="${disable_mesh}"> <visual>
@@ -118,19 +109,17 @@
       </visual> </xacro:unless>
       <xacro:unless value="${disable_mesh}"> <collision>
-        <origin xyz="0.0 0.0 0.0" rpy="0 -0 0"/>
-        <geometry>
-          <mesh filename="package://aero_description/meshes/typeE_wheel/wheels_mecanum.dae" scale="1 1 1" />
-        </geometry>
-      </collision> </xacro:unless>
-      <inertial>
-        <mass value="10" />
-        <origin xyz="0 0 0" rpy="0 -0 0"/>
-        <inertia ixx="0.528" ixy="0" ixz="0" iyy="2.02" iyz="0" izz="2.35"/>
-      </inertial>
-    </link>
-    <gazebo reference="wheels_rear_left_mecanum">
-      <mu1>0.9</mu1>
-      <mu2>0.9</mu2>
-    </gazebo>
+        <origin xyz="0.0 0.0 0.0" rpy="-1.57079632679 0 0"/>
+        <geometry>
+          <!--cylinder length="0.046" radius="0.076" /-->
+          <box size="0.152 0.152 0.046" />
+        </geometry>
+      </collision> </xacro:unless>
+      <inertial>
+        <mass value="1" />
+        <origin xyz="0 0 0" rpy="0 -0 0"/>
+        <inertia ixx="0.528" ixy="0" ixz="0" iyy="2.02" iyz="0" izz="2.35"/>
+      </inertial>
+    </link>
+    <xacro:gazebo_link_reference link_name="wheels_rear_left_mecanum" />
     <link name="wheels_rear_right_mecanum">
       <xacro:unless value="${disable_mesh}"> <visual>
@@ -141,19 +130,17 @@
       </visual> </xacro:unless>
       <xacro:unless value="${disable_mesh}"> <collision>
-        <origin xyz="0.0 0.0 0.0" rpy="0 -0 0"/>
-        <geometry>
-          <mesh filename="package://aero_description/meshes/typeE_wheel/wheels_mecanum.dae" scale="1 1 1" />
-        </geometry>
-      </collision> </xacro:unless>
-      <inertial>
-        <mass value="10" />
-        <origin xyz="0 0 0" rpy="0 -0 0"/>
-        <inertia ixx="0.528" ixy="0" ixz="0" iyy="2.02" iyz="0" izz="2.35"/>
-      </inertial>
-    </link>
-    <gazebo reference="wheels_rear_right_mecanum">
-      <mu1>0.9</mu1>
-      <mu2>0.9</mu2>
-    </gazebo>
+        <origin xyz="0.0 0.0 0.0" rpy="-1.57079632679 0 0"/>
+        <geometry>
+          <!--cylinder length="0.046" radius="0.076" /-->
+          <box size="0.152 0.152 0.046" />
+        </geometry>
+      </collision> </xacro:unless>
+      <inertial>
+        <mass value="1" />
+        <origin xyz="0 0 0" rpy="0 -0 0"/>
+        <inertia ixx="0.528" ixy="0" ixz="0" iyy="2.02" iyz="0" izz="2.35"/>
+      </inertial>
+    </link>
+    <xacro:gazebo_link_reference link_name="wheels_rear_right_mecanum" />
     <link name="wheels_base_laser_link">
       <xacro:unless value="${disable_mesh}"> <visual>
@@ -164,19 +151,16 @@
       </visual> </xacro:unless>
       <xacro:unless value="${disable_mesh}"> <collision>
-        <origin xyz="0.0 0.0 0.0" rpy="0 -0 0"/>
-        <geometry>
-          <mesh filename="package://aero_description/meshes/typeE_wheel/wheels_urg.dae" scale="1 1 1" />
-        </geometry>
-      </collision> </xacro:unless>
-      <inertial>
-        <mass value="10" />
-        <origin xyz="0 0 0" rpy="0 -0 0"/>
-        <inertia ixx="0.528" ixy="0" ixz="0" iyy="2.02" iyz="0" izz="2.35"/>
-      </inertial>
-    </link>
-    <gazebo reference="wheels_base_laser_link">
-      <mu1>0.9</mu1>
-      <mu2>0.9</mu2>
-    </gazebo>
+        <origin xyz="0.0 0.0 -0.0124" rpy="0 -0 0"/>
+        <geometry>
+          <box size="0.08 0.1 0.07" />
+        </geometry>
+      </collision> </xacro:unless>
+      <inertial>
+        <mass value="0.2" />
+        <origin xyz="0 0 0" rpy="0 -0 0"/>
+        <inertia ixx="0.0528" ixy="0" ixz="0" iyy="0.0202" iyz="0" izz="0.0235"/>
+      </inertial>
+    </link>
+    <xacro:gazebo_link_reference link_name="wheels_base_laser_link" />
     <joint name="base_link_to_wheel_base_link_connector" type="fixed">
       <parent link="${base_link}"/>
