Commit message: inverted mesh

File: aero_shop/seed_hand/urdf/seed_hand.urdf.xacro (robot description, xacro)
@@ -93,5 +93,5 @@
   <link name="${prefix}_thumb_link">
     <xacro:unless value="${disable_mesh}"> <visual>
-      <origin xyz="0 0 0" rpy="${M_PI} 0 ${reflect * M_PI / 2.0}"/>
+      <origin xyz="0 0 0" rpy="${-M_PI} 0 ${reflect * M_PI / 2.0}"/>
       <geometry>
         <mesh filename="package://aero_description/meshes/fcsc_hand/RARM_THUMB_LINK_mesh.dae" scale="1 1 1" />
@@ -99,5 +99,5 @@
     </visual> </xacro:unless>
     <xacro:unless value="${disable_mesh}"> <collision>
-      <origin xyz="0 0 0" rpy="${M_PI} 0 ${reflect * M_PI / 2.0}"/>
+      <origin xyz="0 0 0" rpy="${-M_PI} 0 ${reflect * M_PI / 2.0}"/>
       <geometry>
         <mesh filename="package://aero_description/meshes/fcsc_hand/RARM_THUMB_LINK_mesh.dae" scale="1 1 1" />

Commit message: [aero_robot_jsk] fix urdf for using in gazebo, there is no effect to real robot

File: aero_shop/seed_hand/urdf/seed_hand.urdf.xacro (robot description, xacro)
@@ -6,4 +6,5 @@
        xmlns:xacro="http://ros.org/wiki/xacro">
   <xacro:include filename="$(find aero_description)/urdf/common.xacro" />
+  <xacro:include filename="$(find aero_description)/common_urdf/gazebo.xacro" />
   <property name="M_PI" value="3.1415926535897931" />
   <!-- ============================   fcsc_hand   ============================ -->
@@ -26,12 +27,9 @@
     <inertial>
       <mass value="0.183" />
-      <origin xyz="0 0 -0.0875" rpy="0 -0 0"/>
+      <origin xyz="0 0 -0.0875" rpy="0 -0 0"/> <!-- TODO: check -->
       <inertia ixx="0.000601" ixy="0" ixz="0" iyy="0.00055" iyz="0" izz="0.000102"/>
     </inertial>
   </link>
-  <gazebo reference="${prefix}_hand_link">
-    <mu1>0.9</mu1>
-    <mu2>0.9</mu2>
-  </gazebo>
+  <xacro:gazebo_link_reference link_name="${prefix}_hand_link" />
   <link name="${prefix}_indexbase_link">
     <xacro:unless value="${disable_mesh}"> <visual>
@@ -42,30 +40,26 @@
     </visual> </xacro:unless>
     <xacro:unless value="${disable_mesh}"> <collision>
-      <origin xyz="0 0 0" rpy="${M_PI} 0 ${reflect * M_PI / 2.0}"/>
+      <origin xyz="0 ${reflect * -0.004} -0.0123" rpy="${M_PI} 0 ${reflect * M_PI / 2.0}"/>
       <geometry>
-        <mesh filename="package://aero_description/meshes/fcsc_hand/RARM_INDEX_LINK1_mesh.dae" scale="1 1 1" />
+        <!--mesh filename="package://aero_description/meshes/fcsc_hand/RARM_INDEX_LINK1_mesh.dae" scale="1 1 1" /-->
+        <!--box size="0.028 0.0615 0.074" /-->
+        <box size="0.020 0.0615 0.054" />
       </geometry>
     </collision> </xacro:unless>
     <inertial>
-      <mass value="0" />
-      <origin xyz="0 0 0" rpy="0 -0 0"/>
-      <inertia ixx="0" ixy="0" ixz="0" iyy="0" iyz="0" izz="0"/>
+      <mass value="0.1" />
+      <origin xyz="0 0 -0.023" rpy="0 -0 0"/>
+      <inertia ixx="0.0001" iyy="0.0001" izz="0.0001" ixy="0" ixz="0" iyz="0" />
     </inertial>
   </link>
-  <gazebo reference="${prefix}_indexthumb_link">
-    <mu1>0.9</mu1>
-    <mu2>0.9</mu2>
-  </gazebo>
-  <link name="${prefix}_indexmid_link">
+  <xacro:gazebo_link_reference link_name="${prefix}_indexthumb_link" />
+  <link name="${prefix}_indexmid_link"> <!-- dummy link, backward compatibility ??? -->
     <inertial>
-      <mass value="0" />
-      <origin xyz="0 0 0" rpy="0 -0 0"/>
-      <inertia ixx="0" ixy="0" ixz="0" iyy="0" iyz="0" izz="0"/>
+      <mass value="0.1" />
+      <origin xyz="0 0 -0.023" rpy="0 -0 0"/>
+      <inertia ixx="0.0001" iyy="0.0001" izz="0.0001" ixy="0" ixz="0" iyz="0" />
     </inertial>
   </link>
-  <gazebo reference="${prefix}_indexmid_link">
-    <mu1>0.9</mu1>
-    <mu2>0.9</mu2>
-  </gazebo>
+  <xacro:gazebo_link_reference link_name="${prefix}_indexmid_link" />
   <link name="${prefix}_indexend_link">
     <xacro:unless value="${disable_mesh}"> <visual>
@@ -76,19 +70,17 @@
     </visual> </xacro:unless>
     <xacro:unless value="${disable_mesh}"> <collision>
-      <origin xyz="0 0 0" rpy="${M_PI} 0 ${reflect * M_PI / 2.0}"/>
+      <origin xyz="0 0 -0.0225" rpy="${M_PI} 0 ${reflect * M_PI / 2.0}"/>
       <geometry>
-        <mesh filename="package://aero_description/meshes/fcsc_hand/RARM_INDEX_LINK3_mesh.dae" scale="1 1 1" />
+        <!--mesh filename="package://aero_description/meshes/fcsc_hand/RARM_INDEX_LINK3_mesh.dae" scale="1 1 1" /-->
+        <box size="0.020 0.0596 0.065" />
       </geometry>
     </collision> </xacro:unless>
     <inertial>
-      <mass value="0" />
-      <origin xyz="0 0 0" rpy="0 -0 0"/>
-      <inertia ixx="0" ixy="0" ixz="0" iyy="0" iyz="0" izz="0"/>
+      <mass value="0.07" />
+      <origin xyz="0 ${reflect * 0.014} -0.0225" rpy="0 -0 0"/>
+      <inertia ixx="0.0014" iyy="0.0001" izz="0.0001" ixy="0" ixz="0" iyz="0" />
     </inertial>
   </link>
-  <gazebo reference="${prefix}_indexend_link">
-    <mu1>0.9</mu1>
-    <mu2>0.9</mu2>
-  </gazebo>
+  <xacro:gazebo_link_reference link_name="${prefix}_indexend_link" />
   <link name="${prefix}_thumb_link">
     <xacro:unless value="${disable_mesh}"> <visual>
@@ -99,19 +91,17 @@
     </visual> </xacro:unless>
     <xacro:unless value="${disable_mesh}"> <collision>
-      <origin xyz="0 0 0" rpy="${-M_PI} 0 ${reflect * M_PI / 2.0}"/>
+      <origin xyz="0.0 ${reflect * -0.003} -0.0375" rpy="${-M_PI} 0 ${reflect * M_PI / 2.0}"/>
       <geometry>
-        <mesh filename="package://aero_description/meshes/fcsc_hand/RARM_THUMB_LINK_mesh.dae" scale="1 1 1" />
+        <!--mesh filename="package://aero_description/meshes/fcsc_hand/RARM_THUMB_LINK_mesh.dae" scale="1 1 1" /-->
+        <box size="0.032 0.054 0.105" />
       </geometry>
     </collision> </xacro:unless>
     <inertial>
-      <mass value="0" />
-      <origin xyz="0 0 0" rpy="0 -0 0"/>
-      <inertia ixx="0" ixy="0" ixz="0" iyy="0" iyz="0" izz="0"/>
+      <mass value="0.1" />
+      <origin xyz="0 0 -0.04" rpy="0 -0 0"/>
+      <inertia ixx="0.0001" iyy="0.0001" izz="0.0001" ixy="0" ixz="0" iyz="0" />
     </inertial>
   </link>
-  <gazebo reference="${prefix}_thumb_link">
-    <mu1>0.9</mu1>
-    <mu2>0.9</mu2>
-  </gazebo>
+  <xacro:gazebo_link_reference link_name="${prefix}_thumb_link" />
   <joint name="${prefix}_indexbase_joint" type="revolute">
     <parent link="${prefix}_hand_link"/>
@@ -119,37 +109,28 @@
     <origin xyz="0 ${-0.02 * reflect} -0.08" rpy="${1.0472 * reflect} -0 0"/>
     <axis   xyz="1 0 0"/>
-    <limit lower="-3.14159" upper="3.14159" effort="100" velocity="0.5" />
+    <limit lower="-3.14159" upper="3.14159" effort="25" velocity="0.5" />
     <dynamics damping="0.2" friction="0" />
   </joint>
-  <gazebo reference="${prefix}_indexbase_joint">
-    <implicitSpringDamper>0.4</implicitSpringDamper>
-  </gazebo>
-  <joint name="${prefix}_indexmid_joint" type="revolute">
-    <parent link="${prefix}_indexbase_link"/>
+  <xacro:gazebo_transmission joint_name="${prefix}_indexbase_joint" />
+  <joint name="${prefix}_indexmid_joint" type="revolute"> <!-- dummy joint, should be fixed joint -->
+    <parent link="${prefix}_hand_link"/>
     <child  link="${prefix}_indexmid_link"/>
     <origin xyz="0 0 0" rpy="0 -0 0 "/>
     <axis   xyz="1 0 0"/>
-    <limit lower="-3.14159" upper="3.14159" effort="100" velocity="0.5" />
+    <limit lower="-3.14159" upper="3.14159" effort="25" velocity="0.5" />
     <dynamics damping="0.2" friction="0" />
   </joint>
-  <gazebo reference="${prefix}_indexmid_joint">
-    <implicitSpringDamper>0.4</implicitSpringDamper>
-  </gazebo>
+  <!--xacro:gazebo_transmission joint_name="${prefix}_indexmid_joint" /-->
+  <xacro:gazebo_joint_reference joint_name="${prefix}_indexmid_joint" />
   <joint name="${prefix}_indexend_joint" type="revolute">
-    <parent link="${prefix}_indexmid_link"/>
+    <parent link="${prefix}_indexbase_link"/>
     <child  link="${prefix}_indexend_link"/>
     <origin xyz="0 ${-0.004 * reflect} -0.049840" rpy="${0.17 * reflect} -0 0 "/>
     <axis   xyz="1 0 0"/>
-    <limit lower="-3.14159" upper="3.14159" effort="100" velocity="0.5" />
+    <limit lower="-3.14159" upper="3.14159" effort="25" velocity="0.5" />
     <dynamics damping="0.2" friction="0" />
   </joint>
-  <transmission type="pr2_mechanism_model/SimpleTransmission" name="${prefix}_indexend_joint_trans" >
-    <actuator name="${prefix}_indexend_joint_motor" />
-    <joint name="${prefix}_indexend_joint" />
-    <mechanicalReduction>1</mechanicalReduction>
-  </transmission>
-  <gazebo reference="${prefix}_indexend_joint">
-    <implicitSpringDamper>0.4</implicitSpringDamper>
-  </gazebo>
+  <!--xacro:gazebo_transmission joint_name="${prefix}_indexend_joint" /-->
+  <xacro:gazebo_joint_reference joint_name="${prefix}_indexend_joint" />
   <joint name="${prefix}_thumb_joint" type="revolute">
     <parent link="${prefix}_hand_link"/>
@@ -157,15 +138,8 @@
     <origin xyz="0 ${0.020 * reflect} -0.030" rpy="${0.698 * reflect} -0 0 "/>
     <axis   xyz="1 0 0"/>
-    <limit lower="-3.14159" upper="3.14159" effort="100" velocity="0.5" />
+    <limit lower="-3.14159" upper="3.14159" effort="25" velocity="0.5" />
     <dynamics damping="0.2" friction="0" />
   </joint>
-  <transmission type="pr2_mechanism_model/SimpleTransmission" name="${prefix}_thumb_joint_trans" >
-    <actuator name="${prefix}_thumb_joint_motor" />
-    <joint name="${prefix}_thumb_joint" />
-    <mechanicalReduction>1</mechanicalReduction>
-  </transmission>
-  <gazebo reference="${prefix}_thumb_joint">
-    <implicitSpringDamper>0.4</implicitSpringDamper>
-  </gazebo>
+  <xacro:gazebo_transmission joint_name="${prefix}_thumb_joint" />
   <!-- for ik eef link-->
   <link name="${prefix}_eef_grasp_link"/>

Commit message: [aero_robot_jsk] fix minor

File: aero_shop/seed_hand/urdf/seed_hand.urdf.xacro (robot description, xacro)
@@ -8,6 +8,6 @@
   <xacro:include filename="$(find aero_description)/common_urdf/gazebo.xacro" />
   <property name="M_PI" value="3.1415926535897931" />
+  <xacro:macro name="fcsc_hand" params="prefix:=r reflect:=1 disable_mesh:=false">
   <!-- ============================   fcsc_hand   ============================ -->
-  <xacro:macro name="fcsc_hand" params="prefix:=r reflect:=1 disable_mesh:=false">
     <!-- prefix is "r" or "l" -->
     <!-- reflect=1 is rightside, reflect=-1 is leftside -->

Commit message: [aero_shop/seed_hand] fix names

File: aero_shop/seed_hand/urdf/seed_hand.urdf.xacro (robot description, xacro)
@@ -8,6 +8,6 @@
   <xacro:include filename="$(find aero_description)/common_urdf/gazebo.xacro" />
   <property name="M_PI" value="3.1415926535897931" />
-  <xacro:macro name="fcsc_hand" params="prefix:=r reflect:=1 disable_mesh:=false">
-  <!-- ============================   fcsc_hand   ============================ -->
+  <xacro:macro name="seed_hand" params="prefix:=r reflect:=1 disable_mesh:=false">
+  <!-- ============================   seed_hand   ============================ -->
     <!-- prefix is "r" or "l" -->
     <!-- reflect=1 is rightside, reflect=-1 is leftside -->
@@ -16,5 +16,5 @@
       <origin xyz="0 0 0" rpy="${M_PI} -0 ${reflect * M_PI / 2.0}"/>
       <geometry>
-        <mesh filename="package://aero_description/meshes/fcsc_hand/RARM_LINK7_mesh.dae" scale="1 1 1" />
+        <mesh filename="package://aero_description/meshes/seed_hand/RARM_LINK7_mesh.dae" scale="1 1 1" />
       </geometry>
     </visual> </xacro:unless>
@@ -22,5 +22,5 @@
       <origin xyz="0 0 0" rpy="${M_PI} -0 ${reflect * M_PI / 2.0}"/>
       <geometry>
-        <mesh filename="package://aero_description/meshes/fcsc_hand/RARM_LINK7_mesh.dae" scale="1 1 1" />
+        <mesh filename="package://aero_description/meshes/seed_hand/RARM_LINK7_mesh.dae" scale="1 1 1" />
       </geometry>
     </collision> </xacro:unless>
@@ -36,5 +36,5 @@
       <origin xyz="0 0 0" rpy="${M_PI} 0 ${reflect * M_PI / 2.0}"/>
       <geometry>
-        <mesh filename="package://aero_description/meshes/fcsc_hand/RARM_INDEX_LINK1_mesh.dae" scale="1 1 1" />
+        <mesh filename="package://aero_description/meshes/seed_hand/RARM_INDEX_LINK1_mesh.dae" scale="1 1 1" />
       </geometry>
     </visual> </xacro:unless>
@@ -42,5 +42,5 @@
       <origin xyz="0 ${reflect * -0.004} -0.0123" rpy="${M_PI} 0 ${reflect * M_PI / 2.0}"/>
       <geometry>
-        <!--mesh filename="package://aero_description/meshes/fcsc_hand/RARM_INDEX_LINK1_mesh.dae" scale="1 1 1" /-->
+        <!--mesh filename="package://aero_description/meshes/seed_hand/RARM_INDEX_LINK1_mesh.dae" scale="1 1 1" /-->
         <!--box size="0.028 0.0615 0.074" /-->
         <box size="0.020 0.0615 0.054" />
@@ -66,5 +66,5 @@
       <origin xyz="0 0 0" rpy="${M_PI} 0 ${reflect * M_PI / 2.0}"/>
       <geometry>
-        <mesh filename="package://aero_description/meshes/fcsc_hand/RARM_INDEX_LINK3_mesh.dae" scale="1 1 1" />
+        <mesh filename="package://aero_description/meshes/seed_hand/RARM_INDEX_LINK3_mesh.dae" scale="1 1 1" />
       </geometry>
     </visual> </xacro:unless>
@@ -72,5 +72,5 @@
       <origin xyz="0 0 -0.0225" rpy="${M_PI} 0 ${reflect * M_PI / 2.0}"/>
       <geometry>
-        <!--mesh filename="package://aero_description/meshes/fcsc_hand/RARM_INDEX_LINK3_mesh.dae" scale="1 1 1" /-->
+        <!--mesh filename="package://aero_description/meshes/seed_hand/RARM_INDEX_LINK3_mesh.dae" scale="1 1 1" /-->
         <box size="0.020 0.0596 0.065" />
       </geometry>
@@ -87,5 +87,5 @@
       <origin xyz="0 0 0" rpy="${-M_PI} 0 ${reflect * M_PI / 2.0}"/>
       <geometry>
-        <mesh filename="package://aero_description/meshes/fcsc_hand/RARM_THUMB_LINK_mesh.dae" scale="1 1 1" />
+        <mesh filename="package://aero_description/meshes/seed_hand/RARM_THUMB_LINK_mesh.dae" scale="1 1 1" />
       </geometry>
     </visual> </xacro:unless>
@@ -93,5 +93,5 @@
       <origin xyz="0.0 ${reflect * -0.003} -0.0375" rpy="${-M_PI} 0 ${reflect * M_PI / 2.0}"/>
       <geometry>
-        <!--mesh filename="package://aero_description/meshes/fcsc_hand/RARM_THUMB_LINK_mesh.dae" scale="1 1 1" /-->
+        <!--mesh filename="package://aero_description/meshes/seed_hand/RARM_THUMB_LINK_mesh.dae" scale="1 1 1" /-->
         <box size="0.032 0.054 0.105" />
       </geometry>
