Commit message: [aero_shop, aero_description] fix urdf, moveit_config for gazebo

File: aero_description/typeFCESy/urdf/aero-wheels.urdf.xacro (robot description, xacro)
@@ -16,7 +16,7 @@
   <xacro:include filename="$(find aero_description)/urdf/common.xacro" />
   <xacro:include filename="$(find aero_description)/urdf/typeC_lifter/lifter.urdf.xacro" />
-  <xacro:include filename="$(find aero_description)/urdf/typeD_wheel/wheels.urdf.xacro" />
+  <xacro:include filename="$(find aero_description)/urdf/typeE_wheel/wheels.urdf.xacro" />
   <xacro:macro name="aero-wheels" params="base_link" >
-    <xacro:wheels base_link="${base_link}" disable_mesh="${disable_mesh}"/>
+    <xacro:wheels base_link="${base_link}" />
     <joint name="wheel_lifter_connector" type="fixed">
       <parent  link="wheels_top_link"/>

File: aero_shop/hand_yaw/urdf/hand_yaw.urdf.xacro (robot description, xacro)
@@ -31,5 +31,5 @@
       <!-- just fixed for gazebo / aim to increase z axis inertia-->
       <origin xyz="0 0.014 -0.02" rpy="0 -0 0"/>
-      <inertia ixx="0.000601" ixy="0" ixz="0" iyy="0.00055" iyz="0" izz="0.0014" />
+      <inertia ixx="0.003" ixy="0" ixz="0" iyy="0.003" iyz="0" izz="0.005" />
     </inertial>
   </link>

File: aero_shop/seed_hand/urdf/seed_hand.urdf.xacro (robot description, xacro)
@@ -19,10 +19,18 @@
       </geometry>
     </visual> </xacro:unless>
-    <xacro:unless value="${disable_mesh}"> <collision>
-      <origin xyz="0 0 0" rpy="${M_PI} -0 ${reflect * M_PI / 2.0}"/>
+    <xacro:unless value="${disable_mesh}">
+    <collision>
+      <origin xyz="0 0 -0.025" rpy="${M_PI} -0 ${reflect * M_PI / 2.0}"/>
       <geometry>
-        <mesh filename="package://aero_description/meshes/seed_hand/RARM_LINK7_mesh.dae" scale="1 1 1" />
+        <box size="0.060 0.030 0.050" />
       </geometry>
-    </collision> </xacro:unless>
+    </collision>
+    <collision>
+      <origin xyz="0 0 -0.063" rpy="${M_PI} 0.9 ${reflect * M_PI / 2.0}"/>
+      <geometry>
+        <box size="0.020 0.030 0.075" />
+      </geometry>
+    </collision>
+    </xacro:unless>
     <inertial>
       <mass value="0.183" />

File: aero_shop/typeB_lifter/urdf/lifter.urdf.xacro (robot description, xacro)
@@ -54,6 +54,7 @@
         <mass value="2.06679" />
         <!--origin xyz="0.081713 0.000812 -0.146934" rpy="0 -0 0"/-->
-        <origin xyz="0.051713 0.000812 0.146934" rpy="0 -0 0"/>
-        <inertia ixx="0.0408818" ixy="-9.39301e-06" ixz="-0.000750165" iyy="0.0403969" iyz="-0.000120419" izz="0.00260982"/>
+        <origin xyz="0.051713 0.0 0.146934" rpy="0 -0 0"/>
+        <!--inertia ixx="0.0408818" ixy="-9.39301e-06" ixz="-0.000750165" iyy="0.0403969" iyz="-0.000120419" izz="0.00260982"/-->
+        <inertia ixx="0.06" ixy="0.0" ixz="0.0" iyy="0.1" iyz="0.0" izz="0.06"/>
       </inertial>
     </link>
@@ -75,6 +76,7 @@
         <mass value="2.06679" />
         <!--origin xyz="0.081713 0.000812 -0.146934" rpy="0 -0 0"/-->
-        <origin xyz="0.031713 0.000812 0.046934" rpy="0 -0 0"/>
-        <inertia ixx="0.0408818" ixy="-9.39301e-06" ixz="-0.000750165" iyy="0.0403969" iyz="-0.000120419" izz="0.00260982"/>
+        <origin xyz="-0.031713 0.0 0.046934" rpy="0 -0 0"/>
+        <!--inertia ixx="0.0408818" ixy="-9.39301e-06" ixz="-0.000750165" iyy="0.0403969" iyz="-0.000120419" izz="0.00260982"/-->
+        <inertia ixx="0.06" ixy="0.0" ixz="0.0" iyy="0.1" iyz="0.0" izz="0.06"/>
       </inertial>
     </link>
@@ -96,5 +98,5 @@
         <mass value="2.62321" />
         <!--origin xyz="0.0587169 0 -0.135292" rpy="0 -0 0"/-->
-        <origin xyz="0.0587169 0 0.135292" rpy="0 -0 0"/>
+        <origin xyz="-0.0587169 0 0.135292" rpy="0 -0 0"/>
         <inertia ixx="0.0161595" ixy="-9.27234e-05" ixz="0.00262839" iyy="0.0166415" iyz="-0.00017447" izz="0.00477281"/>
       </inertial>
@@ -134,10 +136,9 @@
         </geometry>
       </collision>
-      <!-- same value as base?? -->
-      <!--inertial>
-        <mass value="7.64604" />
-        <origin xyz="-0.012819 -0.002679 0.007207" rpy="0 -0 0"/>
-        <inertia ixx="0.0658136" ixy="-0.000159462" ixz="0.010103" iyy="0.0504268" iyz="0.000173435" izz="0.0889772"/>
-      </inertial-->
+      <inertial>
+        <mass value="1.0" />
+        <origin xyz="0.0 0.0 0.0" rpy="0 0 0"/>
+        <inertia ixx="0.03" ixy="0.0" ixz="0.0" iyy="0.03" iyz="0.0" izz="0.04"/>
+      </inertial>
     </link>
     <xacro:gazebo_link_reference link_name="lifter_top_link" />
@@ -159,5 +160,5 @@
       <origin xyz="0 0 0.12" rpy="0 0 0"/>
       <axis xyz="0 -1 0"/>
-      <limit effort="10000" lower="-1.5707" upper="0" velocity="0.5"/>
+      <limit effort="10000" lower="-1.5707" upper="0" velocity="1.5"/>
     </joint>
     <xacro:gazebo_transmission joint_name="knee_joint" />
@@ -167,5 +168,5 @@
       <origin xyz="0 0 0.05" rpy="0 0 0"/>
       <axis   xyz="0 -1 0"/>
-      <limit effort="1000" lower="0" upper="1.5707" velocity="0.5" />
+      <limit effort="10000" lower="0" upper="1.5707" velocity="1.5" />
       <dynamics damping="0.2" friction="0" />
     </joint>
