Commit message: [aero_shop] add gazebo sensor setting to typeF

File: aero_description/common_urdf/gazebo.xacro (robot description, xacro)
@@ -45,8 +45,8 @@
     </gazebo>
   </xacro:macro>
-  <xacro:macro name="sensors" >
+  <xacro:macro name="gazebo_laser_sensor" params="link_name frame_name topic_name:=lider_scan" >
     <!-- hokuyo -->
-    <!--gazebo reference="hokuyo_link">
-      <sensor type="gpu_ray" name="head_hokuyo_sensor">
+    <gazebo reference="${frame_name}">
+      <sensor type="ray" name="head_hokuyo_sensor">
         <pose>0 0 0 0 0 0</pose>
         <visualize>false</visualize>
@@ -55,8 +55,8 @@
           <scan>
             <horizontal>
-              <samples>720</samples>
+              <samples>1000</samples>
               <resolution>1</resolution>
-              <min_angle>-1.570796</min_angle>
-              <max_angle>1.570796</max_angle>
+              <min_angle>-2.35619449</min_angle>
+              <max_angle>2.35619449</max_angle>
             </horizontal>
           </scan>
@@ -68,18 +68,22 @@
           <noise>
             <type>gaussian</type>
+                 <!--
                  Noise parameters based on published spec for Hokuyo laser
                  achieving "+-30mm" accuracy at range < 10m.  A mean of 0.0m and
                  stddev of 0.01m will put 99.7% of samples within 0.03m of the true
                  reading.
+                 -->
             <mean>0.0</mean>
             <stddev>0.01</stddev>
           </noise>
         </ray>
-        <plugin name="gazebo_ros_head_hokuyo_controller" filename="libgazebo_ros_gpu_laser.so">
-          <topicName>/rrbot/laser/scan</topicName>
-          <frameName>hokuyo_link</frameName>
+        <plugin name="gazebo_ros_head_hokuyo_controller" filename="libgazebo_ros_laser.so">
+          <topicName>${topic_name}</topicName>
+          <frameName>${frame_name}</frameName>
         </plugin>
       </sensor>
-    </gazebo-->
+    </gazebo>
+  </xacro:macro>
+  <xacro:macro name="camera" >
     <!-- camera -->
     <!--gazebo reference="camera_link">

File: aero_description/typeF/robots/aero.urdf.xacro (robot description, xacro)
@@ -15,5 +15,43 @@
  <xacro:aero-upper/>
  <xacro:aero-wheels base_link="base_link"/>
+ <xacro:gazebo_laser_sensor link_name="wheels_base_laser_link" frame_name="wheels_base_laser_link" />
  <xacro:gazebo_trajectory_controller />
  <xacro:gazebo_base_controller base_frame="base_link" />
+ <gazebo>
+   <plugin name="mimic_updater" filename="libmimic_plugin.so">
+     <!-- lifter -->
+     <mimic joint="knee_joint"  offset="0.0" multiplier="-1.0"
+            P="1000" I="0.0" D="1" i_max="0" i_min="0"
+            command_max="200" command_min="-200"> knee_joint_dummy</mimic>
+     <mimic joint="ankle_joint"  offset="0.0" multiplier="1.0"
+            P="1000" I="0.0" D="1" i_max="0" i_min="0"
+            command_max="200" command_min="-200"> ankle_joint_dummy</mimic>
+     <mimic joint="knee_joint"  offset="0.0" multiplier="-1.0"
+            P="3000" I="0.0" D="3" i_max="0" i_min="0"
+            command_max="1000" command_min="-1000"> knee_joint_mimic</mimic>
+     <mimic joint="ankle_joint"  offset="0.0" multiplier="-1.0"
+            P="3000" I="0.0" D="3" i_max="0" i_min="0"
+            command_max="1000" command_min="-1000"> ankle_joint_mimic</mimic>
+     <!-- lhand -->
+     <mimic joint="l_thumb_joint"  offset="0.0" multiplier="-1.0"
+            P="30" I="0.0" D="0.03" i_max="0" i_min="0"
+            command_max="50" command_min="-50"> l_indexbase_joint </mimic>
+     <mimic joint="l_thumb_joint"  offset="-0.2" multiplier="-0.3"
+            P="30" I="0.0" D="0.03" i_max="0" i_min="0"
+            command_max="50" command_min="-50"> l_indexmid_joint </mimic>
+     <mimic joint="l_thumb_joint"  offset="-0.2" multiplier="-0.3"
+            P="30" I="0.0" D="0.03" i_max="0" i_min="0"
+            command_max="50" command_min="-50"> l_indexend_joint </mimic>
+     <!-- rhand -->
+     <mimic joint="r_thumb_joint"  offset="0.0" multiplier="-1.0"
+            P="30" I="0.0" D="0.03" i_max="0" i_min="0"
+            command_max="50" command_min="-50"> r_indexbase_joint </mimic>
+     <mimic joint="r_thumb_joint"  offset="0.2" multiplier="-0.3"
+            P="30" I="0.0" D="0.03" i_max="0" i_min="0"
+            command_max="50" command_min="-50"> r_indexmid_joint </mimic>
+     <mimic joint="r_thumb_joint"  offset="0.2" multiplier="-0.3"
+            P="30" I="0.0" D="0.03" i_max="0" i_min="0"
+            command_max="50" command_min="-50"> r_indexend_joint </mimic>
+   </plugin>
+ </gazebo>
 </robot>

Commit message: [aero_description] update xacro for gazebo

File: aero_description/common_urdf/gazebo.xacro (robot description, xacro)
@@ -45,5 +45,5 @@
     </gazebo>
   </xacro:macro>
-  <xacro:macro name="gazebo_laser_sensor" params="link_name frame_name topic_name:=lider_scan" >
+  <xacro:macro name="gazebo_laser_sensor" params="link_name frame_name topic_name:=scan" >
     <!-- hokuyo -->
     <gazebo reference="${frame_name}">
@@ -85,11 +85,40 @@
     </gazebo>
   </xacro:macro>
-  <xacro:macro name="camera" >
+  <xacro:macro name="gazebo_depth_camera"
+               params="link_name frame_name camera_name:=camera" >
+    <gazebo>
+      <plugin name="${link_name}_controller" filename="libgazebo_ros_openni_kinect.so">
+        <baseline>0.14</baseline>
+        <alwaysOn>true</alwaysOn>
+        <updateRate>10.0</updateRate>
+        <cameraName>${camera_name}</cameraName>
+        <imageTopicName>/${camera_name}/image_raw</imageTopicName>
+        <cameraInfoTopicName>/${camera_name}/camera_info</cameraInfoTopicName>
+        <depthImageTopicName>/${camera_name}/depth/image_raw</depthImageTopicName>
+        <depthImageInfoTopicName>/${camera_name}/depth/camera_info</depthImageInfoTopicName>
+        <pointCloudTopicName>/${camera_name}/depth/points</pointCloudTopicName>
+        <frameName>${frame_name}</frameName>
+        <pointCloudCutoff>0.2</pointCloudCutoff>
+        <distortionK1>0.000000</distortionK1>
+        <distortionK2>0.000000</distortionK2>
+        <distortionK3>0.000000</distortionK3>
+        <distortionT1>0.000000</distortionT1>
+        <distortionT2>0.000000</distortionT2>
+        <CxPrime>0</CxPrime>
+        <Cx>0</Cx>
+        <Cy>0</Cy>
+        <focalLength>0</focalLength>
+        <hackBaseline>0</hackBaseline>
+      </plugin>
+    </gazebo>
+  </xacro:macro>
+  <xacro:macro name="gazebo_camera"
+               params="link_name frame_name topic_name:=camera" >
     <!-- camera -->
-    <!--gazebo reference="camera_link">
+    <gazebo reference="${link_name}">
       <sensor type="camera" name="camera1">
-        <update_rate>30.0</update_rate>
+        <update_rate>15.0</update_rate>
         <camera name="head">
-          <horizontal_fov>1.3962634</horizontal_fov>
+          <horizontal_fov>1.7</horizontal_fov> <!-- -->
           <image>
             <width>800</width>
@@ -103,7 +132,7 @@
           <noise>
             <type>gaussian</type>
-                 Noise is sampled independently per pixel on each frame.
+                 <!--Noise is sampled independently per pixel on each frame.
                  That pixel's noise value is added to each of its color
-                 channels, which at that point lie in the range [0,1].
+                 channels, which at that point lie in the range [0,1]. -->
             <mean>0.0</mean>
             <stddev>0.007</stddev>
@@ -113,11 +142,11 @@
           <alwaysOn>true</alwaysOn>
           <updateRate>0.0</updateRate>
-          <cameraName>rrbot/camera1</cameraName>
+          <cameraName>${camera_name}</cameraName>
           <imageTopicName>image_raw</imageTopicName>
           <cameraInfoTopicName>camera_info</cameraInfoTopicName>
-          <frameName>camera_link_optical</frameName>
-               setting hackBaseline to anything but 0.0 will cause a misalignment
+          <frameName>${frame_name}</frameName>
+               <!--setting hackBaseline to anything but 0.0 will cause a misalignment
                between the gazebo sensor image and the frame it is supposed to
-               be attached to
+               be attached to-->
           <hackBaseline>0.0</hackBaseline>
           <distortionK1>0.0</distortionK1>
@@ -132,5 +161,5 @@
         </plugin>
       </sensor>
-    </gazebo-->
+    </gazebo>
   </xacro:macro>
 </robot>

Commit message: [aero_description] add camera settings to typeF

File: aero_description/common_urdf/gazebo.xacro (robot description, xacro)
@@ -47,5 +47,5 @@
   <xacro:macro name="gazebo_laser_sensor" params="link_name frame_name topic_name:=scan" >
     <!-- hokuyo -->
-    <gazebo reference="${frame_name}">
+    <gazebo reference="${link_name}">
       <sensor type="ray" name="head_hokuyo_sensor">
         <pose>0 0 0 0 0 0</pose>
@@ -62,5 +62,5 @@
           </scan>
           <range>
-            <min>0.10</min>
+            <min>0.5</min>
             <max>30.0</max>
             <resolution>0.01</resolution>
@@ -87,32 +87,53 @@
   <xacro:macro name="gazebo_depth_camera"
                params="link_name frame_name camera_name:=camera" >
-    <gazebo>
-      <plugin name="${link_name}_controller" filename="libgazebo_ros_openni_kinect.so">
-        <baseline>0.14</baseline>
-        <alwaysOn>true</alwaysOn>
-        <updateRate>10.0</updateRate>
-        <cameraName>${camera_name}</cameraName>
-        <imageTopicName>/${camera_name}/image_raw</imageTopicName>
-        <cameraInfoTopicName>/${camera_name}/camera_info</cameraInfoTopicName>
-        <depthImageTopicName>/${camera_name}/depth/image_raw</depthImageTopicName>
-        <depthImageInfoTopicName>/${camera_name}/depth/camera_info</depthImageInfoTopicName>
-        <pointCloudTopicName>/${camera_name}/depth/points</pointCloudTopicName>
-        <frameName>${frame_name}</frameName>
-        <pointCloudCutoff>0.2</pointCloudCutoff>
-        <distortionK1>0.000000</distortionK1>
-        <distortionK2>0.000000</distortionK2>
-        <distortionK3>0.000000</distortionK3>
-        <distortionT1>0.000000</distortionT1>
-        <distortionT2>0.000000</distortionT2>
-        <CxPrime>0</CxPrime>
-        <Cx>0</Cx>
-        <Cy>0</Cy>
-        <focalLength>0</focalLength>
-        <hackBaseline>0</hackBaseline>
-      </plugin>
+    <gazebo reference="${link_name}">
+      <sensor type="depth" name="camera1">
+        <update_rate>1</update_rate>
+        <camera name="head">
+          <!--
+               <noise>
+               <type>gaussian</type>
+               <mean>0.0</mean>
+               <stddev>0.007</stddev>
+               </noise>
+          -->
+          <horizontal_fov>1.7</horizontal_fov>
+          <image>
+            <width>640</width>
+            <height>480</height>
+            <format>R8G8B8</format>
+          </image>
+          <clip>
+            <near>0.15</near>
+            <far>300</far>
+          </clip>
+        </camera>
+        <plugin name="camera_controller" filename="libgazebo_ros_depth_camera.so">
+          <alwaysOn>true</alwaysOn>
+          <!-- Keep this zero, update_rate will control the frame rate -->
+          <updateRate>0.0</updateRate>
+          <cameraName>${camera_name}</cameraName>
+          <imageTopicName>image_raw</imageTopicName>
+          <cameraInfoTopicName>camera_info</cameraInfoTopicName>
+          <depthImageTopicName>depth/image_raw</depthImageTopicName>
+          <!-- neither camera info is getting published, frame_id is empty
+               in points and both image headers -->
+          <depthImageCameraInfoTopicName>depth/camera_info</depthImageCameraInfoTopicName>
+          <pointCloudTopicName>points</pointCloudTopicName>
+          <frameName>${frame_name}</frameName>
+          <!-- TODO(lucasw) is this used by depth camera at all? -->
+          <hackBaseline>0.07</hackBaseline>
+          <pointCloudCutoff>0.001</pointCloudCutoff>
+          <distortionK1>0.0</distortionK1>
+          <distortionK2>0.0</distortionK2>
+          <distortionK3>0.0</distortionK3>
+          <distortionT1>0.0</distortionT1>
+          <distortionT2>0.0</distortionT2>
+        </plugin>
+      </sensor>
     </gazebo>
   </xacro:macro>
   <xacro:macro name="gazebo_camera"
-               params="link_name frame_name topic_name:=camera" >
+               params="link_name frame_name camera_name:=camera" >
     <!-- camera -->
     <gazebo reference="${link_name}">
@@ -127,5 +148,5 @@
           </image>
           <clip>
-            <near>0.02</near>
+            <near>0.15</near>
             <far>300</far>
           </clip>

File: aero_description/typeF/robots/aero.urdf.xacro (robot description, xacro)
@@ -15,5 +15,21 @@
  <xacro:aero-upper/>
  <xacro:aero-wheels base_link="base_link"/>
- <xacro:gazebo_laser_sensor link_name="wheels_base_laser_link" frame_name="wheels_base_laser_link" />
+ <!-- camera -->
+ <link name="camera_frame" />
+ <link name="camera_optical_frame" />
+ <joint name="camera_setting" type="fixed" >
+   <parent link="head_link" />
+   <child  link="camera_frame" />
+   <origin xyz="0 0.035 0.09" rpy="0 0.15 0" />
+ </joint>
+ <joint name="camera_optical" type="fixed" >
+   <parent link="camera_frame" />
+   <child  link="camera_optical_frame" />
+   <origin xyz="0 0 0" rpy="-1.570796326795 0 -1.570796326795" />
+ </joint>
+ <xacro:gazebo_camera link_name="camera_frame"
+                      frame_name="camera_optical_frame" />
+ <xacro:gazebo_laser_sensor link_name="wheels_base_laser_link"
+                            frame_name="wheels_base_laser_link" />
  <xacro:gazebo_trajectory_controller />
  <xacro:gazebo_base_controller base_frame="base_link" />

Commit message: [aero_gazebo] use velocity feedback

File: aero_description/common_urdf/gazebo.xacro (robot description, xacro)
@@ -7,5 +7,5 @@
     </gazebo>
   </xacro:macro>
-  <xacro:macro name="gazebo_joint_reference" params="joint_name implicitspringdamper:=0.4" >
+  <xacro:macro name="gazebo_joint_reference" params="joint_name implicitspringdamper:=0" >
     <gazebo reference="${joint_name}">
       <implicitSpringDamper>${implicitspringdamper}</implicitSpringDamper>
@@ -18,10 +18,12 @@
         <!-- dupricated in kinetic -->
         <!--hardwareInterface>hardware_interface/EffortJointInterface</hardwareInterface-->
-        <hardwareInterface>EffortJointInterface</hardwareInterface>
+        <!--hardwareInterface>EffortJointInterface</hardwareInterface-->
+        <hardwareInterface>VelocityJointInterface</hardwareInterface>
       </joint>
       <actuator name="${joint_name}_motor">
         <!-- dupricated in kinetic -->
         <!--hardwareInterface>hardware_interface/EffortJointInterface</hardwareInterface-->
-        <hardwareInterface>EffortJointInterface</hardwareInterface>
+        <!--hardwareInterface>EffortJointInterface</hardwareInterface-->
+        <hardwareInterface>VelocityJointInterface</hardwareInterface>
         <mechanicalReduction>1</mechanicalReduction>
       </actuator>
