Commit message: [aero_shop] fix limit of mimic joints for typeC_lifter

File: aero_shop/typeC_lifter/urdf/lifter.urdf.xacro (robot description, xacro)
@@ -148,5 +148,5 @@
       <origin xyz="0 0 0.055" rpy="0 0 0"/>
     </joint>
-    <joint name="knee_joint_mimic" type="continuous">
+    <joint name="knee_joint_mimic" type="revolute">
       <parent link="leg_thigh_link"/>
       <child link="leg_base_link"/>
@@ -154,4 +154,5 @@
       <axis   xyz="0 -1 0"/>
       <mimic joint="knee_joint" multiplier="-1" offset="0"/>
+      <limit effort="10000" upper="1.5707" lower="0" velocity="1.5"/> <!-- just invert of knee_joint -->
     </joint>
     <joint name="knee_joint" type="revolute"> <!-- rename "knee_joint_thigh_dummy" -->
@@ -168,5 +169,5 @@
       <origin xyz="0 0 0.05" rpy="0 0 0"/>
       <axis   xyz="0 -1 0"/>
-      <limit effort="4000" lower="0" upper="1.5707" velocity="1.5" />
+      <limit effort="10000" lower="0" upper="1.5707" velocity="1.5" />
       <dynamics damping="0.2" friction="0" />
     </joint>
@@ -174,5 +175,5 @@
 <!--- mimic joints -->
 <!-- requried -->
-    <joint name="ankle_joint_mimic" type="continuous">
+    <joint name="ankle_joint_mimic" type="revolute">
       <parent link="leg_shank_link"/>
       <child  link="leg_knee_link"/>
@@ -180,4 +181,5 @@
       <axis   xyz="0 -1 0"/>
       <mimic joint="ankle_joint" multiplier="-1" offset="0" />
+      <limit effort="10000" upper="0" lower="-1.5707" velocity="1.5" /> <!-- just invert of ankle_joint -->
     </joint>
 <!-- redundant -->

Commit message: use collision dir for collision geometries

File: aero_shop/typeC_lifter/urdf/lifter.urdf.xacro (robot description, xacro)
@@ -28,5 +28,5 @@
         <origin xyz="0 0 0" rpy="0 -0 0"/>
         <geometry>
-          <mesh filename="package://aero_description/meshes/typeC_lifter/lifter_base.dae" scale="1 1 1" />
+          <mesh filename="package://aero_description/meshes/typeC_lifter/collision/lifter_base.dae" scale="1 1 1" />
         </geometry>
       </collision>
@@ -48,5 +48,5 @@
         <origin xyz="0.0 0.0 0" rpy="3.1415 -0 0"/>
         <geometry>
-          <mesh filename="package://aero_description/meshes/typeC_lifter/lifter_bone.dae" scale="1 1 1" />
+          <mesh filename="package://aero_description/meshes/typeC_lifter/collision/lifter_bone.dae" scale="1 1 1" />
         </geometry>
       </collision>
@@ -70,5 +70,5 @@
         <origin xyz="0.0 0.0 0" rpy="3.1415 -0 0"/>
         <geometry>
-          <mesh filename="package://aero_description/meshes/typeC_lifter/lifter_knee.dae" scale="1 1 1" />
+          <mesh filename="package://aero_description/meshes/typeC_lifter/collision/lifter_knee.dae" scale="1 1 1" />
         </geometry>
       </collision>
@@ -92,5 +92,5 @@
         <origin xyz="0 0 0.25" rpy="0 0 0"/>
         <geometry>
-          <mesh filename="package://aero_description/meshes/typeC_lifter/lifter_bone.dae" scale="1 1 1" />
+          <mesh filename="package://aero_description/meshes/typeC_lifter/collision/lifter_bone.dae" scale="1 1 1" />
         </geometry>
       </collision>
@@ -113,5 +113,5 @@
         <origin xyz="0 0 0.05" rpy="3.1415920 0 0"/>
         <geometry>
-          <mesh filename="package://aero_description/meshes/typeC_lifter/lifter_base.dae" scale="1 1 1" />
+          <mesh filename="package://aero_description/meshes/typeC_lifter/collision/lifter_base.dae" scale="1 1 1" />
         </geometry>
       </collision>
@@ -133,5 +133,5 @@
         <origin xyz="0 0 0" rpy="0 -0 0"/>
         <geometry>
-          <mesh filename="package://aero_description/meshes/typeC_lifter/lifter_top.dae" scale="1 1 1" />
+          <mesh filename="package://aero_description/meshes/typeC_lifter/collision/lifter_top.dae" scale="1 1 1" />
         </geometry>
       </collision>

File: aero_shop/typeF_upperbody/urdf/aero_upper_typef.urdf.xacro (robot description, xacro)
@@ -20,5 +20,5 @@
       <origin xyz="0 0 0" rpy="0 -0 0"/>
       <geometry>
-        <mesh filename="package://aero_description/meshes/typeF_upperbody/WAIST_LINK0_mesh.dae" scale="1 1 1" />
+        <mesh filename="package://aero_description/meshes/typeF_upperbody/collision/WAIST_LINK0_mesh.dae" scale="1 1 1" />
       </geometry>
     </collision> </xacro:unless>
@@ -40,5 +40,5 @@
       <origin xyz="0 0 0" rpy="0 -0 0"/>
       <geometry>
-        <mesh filename="package://aero_description/meshes/typeF_upperbody/WAIST_LINK1_mesh.dae" scale="1 1 1" />
+        <mesh filename="package://aero_description/meshes/typeF_upperbody/collision/WAIST_LINK1_mesh.dae" scale="1 1 1" />
       </geometry>
     </collision> </xacro:unless>
@@ -72,5 +72,5 @@
       <origin xyz="0 0 0" rpy="0 -0 0"/>
       <geometry>
-        <mesh filename="package://aero_description/meshes/typeF_upperbody/WAIST_LINK3_mesh.dae" scale="1 1 1" />
+        <mesh filename="package://aero_description/meshes/typeF_upperbody/collision/WAIST_LINK3_mesh.dae" scale="1 1 1" />
       </geometry>
     </collision> </xacro:unless>
@@ -92,5 +92,5 @@
       <origin xyz="0 0 0" rpy="-0.174532925 -0 0"/>
       <geometry>
-        <mesh filename="package://aero_description/meshes/typeF_upperbody/LARM_LINK1_mesh.dae" scale="1 1 1" />
+        <mesh filename="package://aero_description/meshes/typeF_upperbody/collision/LARM_LINK1_mesh.dae" scale="1 1 1" />
       </geometry>
     </collision> </xacro:unless>
@@ -115,5 +115,5 @@
       <origin xyz="0 0 0" rpy="0 -0 0"/>
       <geometry>
-        <mesh filename="package://aero_description/meshes/typeF_upperbody/LARM_LINK2_mesh.dae" scale="1 1 1" />
+        <mesh filename="package://aero_description/meshes/typeF_upperbody/collision/LARM_LINK2_mesh.dae" scale="1 1 1" />
       </geometry>
     </collision> </xacro:unless>
@@ -136,5 +136,5 @@
       <origin xyz="0 0 0" rpy="0 -0 0"/>
       <geometry>
-        <mesh filename="package://aero_description/meshes/typeF_upperbody/LARM_LINK3_mesh.dae" scale="1 1 1" />
+        <mesh filename="package://aero_description/meshes/typeF_upperbody/collision/LARM_LINK3_mesh.dae" scale="1 1 1" />
       </geometry>
     </collision> </xacro:unless>
@@ -159,5 +159,5 @@
       <origin xyz="-0.035 0 -0.035" rpy="0 -0 0"/>
       <geometry>
-        <mesh filename="package://aero_description/meshes/typeF_upperbody/LARM_LINK4_mesh.dae" scale="1 1 1" />
+        <mesh filename="package://aero_description/meshes/typeF_upperbody/collision/LARM_LINK4_mesh.dae" scale="1 1 1" />
       </geometry>
     </collision> </xacro:unless>
@@ -182,5 +182,5 @@
       <origin xyz="0 0 0" rpy="0 0 -1.5707963267948966"/>
       <geometry>
-        <mesh filename="package://aero_description/meshes/typeF_upperbody/LARM_LINK5_mesh.dae" scale="1 1 1" />
+        <mesh filename="package://aero_description/meshes/typeF_upperbody/collision/LARM_LINK5_mesh.dae" scale="1 1 1" />
       </geometry>
     </collision> </xacro:unless>
@@ -211,5 +211,5 @@
       <origin xyz="0 0 0" rpy="0 -0 0"/>
       <geometry>
-        <mesh filename="package://aero_description/meshes/typeF_upperbody/NECK_LINK1_mesh.dae" scale="1 1 1" />
+        <mesh filename="package://aero_description/meshes/typeF_upperbody/collision/NECK_LINK1_mesh.dae" scale="1 1 1" />
       </geometry>
     </collision> </xacro:unless>
@@ -232,5 +232,5 @@
       <origin xyz="0 0 0" rpy="0 -0 0"/>
       <geometry>
-        <mesh filename="package://aero_description/meshes/typeF_upperbody/NECK_LINK2_mesh.dae" scale="1 1 1" />
+        <mesh filename="package://aero_description/meshes/typeF_upperbody/collision/NECK_LINK2_mesh.dae" scale="1 1 1" />
       </geometry>
     </collision> </xacro:unless>
@@ -252,5 +252,5 @@
       <origin xyz="0 0 0" rpy="0 -0 0"/>
       <geometry>
-        <mesh filename="package://aero_description/meshes/typeF_upperbody/NECK_LINK3_mesh.dae" scale="1 1 1" />
+        <mesh filename="package://aero_description/meshes/typeF_upperbody/collision/NECK_LINK3_mesh.dae" scale="1 1 1" />
       </geometry>
     </collision> </xacro:unless>
@@ -272,5 +272,5 @@
       <origin xyz="0 0 0" rpy="0.174532925 -0 0"/>
       <geometry>
-        <mesh filename="package://aero_description/meshes/typeF_upperbody/RARM_LINK1_mesh.dae" scale="1 1 1" />
+        <mesh filename="package://aero_description/meshes/typeF_upperbody/collision/RARM_LINK1_mesh.dae" scale="1 1 1" />
       </geometry>
     </collision> </xacro:unless>
@@ -294,5 +294,5 @@
       <origin xyz="0 0 0" rpy="0 -0 0"/>
       <geometry>
-        <mesh filename="package://aero_description/meshes/typeF_upperbody/RARM_LINK2_mesh.dae" scale="1 1 1" />
+        <mesh filename="package://aero_description/meshes/typeF_upperbody/collision/RARM_LINK2_mesh.dae" scale="1 1 1" />
       </geometry>
     </collision> </xacro:unless>
@@ -315,5 +315,5 @@
       <origin xyz="0 0 0" rpy="0 -0 0"/>
       <geometry>
-        <mesh filename="package://aero_description/meshes/typeF_upperbody/RARM_LINK3_mesh.dae" scale="1 1 1" />
+        <mesh filename="package://aero_description/meshes/typeF_upperbody/collision/RARM_LINK3_mesh.dae" scale="1 1 1" />
       </geometry>
     </collision> </xacro:unless>
@@ -338,5 +338,5 @@
       <origin xyz="-0.035 0 -0.035" rpy="0 -0 0"/>
       <geometry>
-        <mesh filename="package://aero_description/meshes/typeF_upperbody/RARM_LINK4_mesh.dae" scale="1 1 1" />
+        <mesh filename="package://aero_description/meshes/typeF_upperbody/collision/RARM_LINK4_mesh.dae" scale="1 1 1" />
       </geometry>
     </collision> </xacro:unless>
@@ -361,5 +361,5 @@
       <origin xyz="0 0 0" rpy="0 0 1.5707963267948966"/>
       <geometry>
-        <mesh filename="package://aero_description/meshes/typeF_upperbody/RARM_LINK5_mesh.dae" scale="1 1 1" />
+        <mesh filename="package://aero_description/meshes/typeF_upperbody/collision/RARM_LINK5_mesh.dae" scale="1 1 1" />
       </geometry>
     </collision> </xacro:unless>
