Commit message: fix joint limit and veclocity limit

File: aero_shop/typeF_upperbody/urdf/aero_upper_typef.urdf.xacro (robot description, xacro)
@@ -415,5 +415,6 @@
     <origin xyz="0 0 0.010" rpy="0 -0 0 "/>
     <axis   xyz="0 0 1"/>
-    <limit lower="-1.5707" upper="1.5707" effort="100" velocity="0.5" />
+    <!-- from -120 to 120 degrees-->
+    <limit lower="-1.5707" upper="1.5707" effort="100" velocity="0.9" />
     <dynamics damping="0.2" friction="0" />
   </joint>
@@ -431,5 +432,6 @@
     <origin xyz="0 0 0.1355" rpy="0 -0 0 "/>
     <axis   xyz="0 1 0"/>
-    <limit lower="0" upper="0.4014" effort="100" velocity="0.5" />
+    <!-- from -5 to 30 degrees-->
+    <limit lower="-0.0872" upper="0.5235" effort="100" velocity="0.3" />
     <dynamics damping="0.2" friction="0" />
   </joint>
@@ -447,5 +449,6 @@
     <origin xyz="0 0 0" rpy="0 -0 0 "/>
     <axis   xyz="1 0 0"/>
-    <limit lower="-0.017" upper="0.017" effort="100" velocity="0.5" />
+    <!-- from -1 to 1 degrees-->
+    <limit lower="-0.017" upper="0.017" effort="100" velocity="0.3" />
     <dynamics damping="0.2" friction="0" />
   </joint>
@@ -463,5 +466,6 @@
     <origin xyz="-0.01815 0.1342 0.3049" rpy="0 -0 0 "/>
     <axis   xyz="0 0.984808 -0.173648"/>
-    <limit lower="-1.50" upper="0" effort="100" velocity="0.5" />
+    <!-- from -88 to 15 degrees-->
+    <limit lower="-1.535" upper="0.261" effort="100" velocity="2.2" />
     <dynamics damping="0.2" friction="0" />
   </joint>
@@ -479,5 +483,6 @@
     <origin xyz="0 0.05978 0.028046" rpy="0 -0 0 "/>
     <axis   xyz="1 0 0"/>
-    <limit lower="0" upper="1.5707" effort="100" velocity="0.5" />
+    <!-- from 0 to 90 degrees-->
+    <limit lower="0" upper="1.5707" effort="100" velocity="2.3" />
     <dynamics damping="0.2" friction="0" />
   </joint>
@@ -495,5 +500,6 @@
     <origin xyz="0 -0.010 -0.127" rpy="0 -0 0 "/>
     <axis   xyz="0 0 1"/>
-    <limit lower="-1.5707" upper="0.785398" effort="100" velocity="0.5" />
+    <!-- from -180 to 45 degrees-->
+    <limit lower="-1.5707" upper="0.785398" effort="100" velocity="3.0" />
     <dynamics damping="0.2" friction="0" />
   </joint>
@@ -511,5 +517,6 @@
     <origin xyz="0.035 0 -0.1625" rpy="0 -0 0 "/>
     <axis   xyz="0 1 0"/>
-    <limit lower="-2.44246" upper="0" effort="100" velocity="0.5" />
+    <!-- from -140 to 0 degrees-->
+    <limit lower="-2.44246" upper="0" effort="100" velocity="2.3" />
     <dynamics damping="0.2" friction="0" />
   </joint>
@@ -527,5 +534,6 @@
     <origin xyz="-0.035 0 -0.070" rpy="0 -0 0 "/>
     <axis   xyz="0 0 1"/>
-    <limit lower="-1.5707" upper="1.5707" effort="100" velocity="0.5" />
+    <!-- from -180 to 180 degrees-->
+    <limit lower="-1.5707" upper="1.5707" effort="100" velocity="5.6" />
     <dynamics damping="0.2" friction="0" />
   </joint>
@@ -543,5 +551,6 @@
     <origin xyz="0 0 -0.1955" rpy="0 -0 0 "/>
     <axis   xyz="0 1 0"/>
-    <limit lower="-0.15" upper="0.15" effort="100" velocity="0.5" />
+    <!-- from -9 to 9 degrees-->
+    <limit lower="-0.15" upper="0.15" effort="100" velocity="2.2" />
     <dynamics damping="0.2" friction="0" />
   </joint>
@@ -559,5 +568,6 @@
     <origin xyz="0 0 0" rpy="0 -0 0 "/>
     <axis   xyz="1 0 0"/>
-    <limit lower="-0.698132" upper="0.698132" effort="100" velocity="0.5" />
+    <!-- from -75 to 40 degrees-->
+    <limit lower="-1.309" upper="-0.698132" effort="100" velocity="2.2" />
     <dynamics damping="0.2" friction="0" />
   </joint>
@@ -623,5 +633,6 @@
     <origin xyz="-0.01815 -0.1342 0.3049" rpy="0 -0 0 "/>
     <axis   xyz="0 0.984808 0.173648"/>
-    <limit lower="-1.50" upper="0" effort="100" velocity="0.5" />
+    <!-- from -15 to 88 degrees-->
+    <limit lower="-0.261" upper="-1.535" effort="100" velocity="2.2" />
     <dynamics damping="0.2" friction="0" />
   </joint>
@@ -639,5 +650,6 @@
     <origin xyz="0 -0.059778 0.028046" rpy="0 -0 0 "/>
     <axis   xyz="1 0 0"/>
-    <limit lower="-1.5707" upper="0" effort="100" velocity="0.5" />
+    <!-- from -90 to 0 degrees-->
+    <limit lower="-1.5707" upper="0" effort="100" velocity="2.3" />
     <dynamics damping="0.2" friction="0" />
   </joint>
@@ -655,5 +667,6 @@
     <origin xyz="0 0.010 -0.127" rpy="0 -0 0 "/>
     <axis   xyz="0 0 1"/>
-    <limit lower="-0.785398" upper="1.5707" effort="100" velocity="0.5" />
+    <!-- from -45 to 180 degrees-->
+    <limit lower="-0.785398" upper="1.5707" effort="100" velocity="3.0" />
     <dynamics damping="0.2" friction="0" />
   </joint>
@@ -671,5 +684,6 @@
     <origin xyz="0.035 0 -0.1625" rpy="0 -0 0 "/>
     <axis   xyz="0 1 0"/>
-    <limit lower="-2.44246" upper="0" effort="100" velocity="0.5" />
+    <!-- from 0 to 140 degrees-->
+    <limit lower="0" upper="2.44246" effort="100" velocity="2.3" />
     <dynamics damping="0.2" friction="0" />
   </joint>
@@ -687,5 +701,6 @@
     <origin xyz="-0.035 0 -0.070" rpy="0 -0 0 "/>
     <axis   xyz="0 0 1"/>
-    <limit lower="-1.5707" upper="1.5707" effort="100" velocity="0.5" />
+    <!-- from -180 to 180 degrees-->
+    <limit lower="-1.5707" upper="1.5707" effort="100" velocity="5.6" />
     <dynamics damping="0.2" friction="0" />
   </joint>
@@ -703,5 +718,6 @@
     <origin xyz="0 0 -0.1955" rpy="0 -0 0 "/>
     <axis   xyz="0 1 0"/>
-    <limit lower="-0.15" upper="0.15" effort="100" velocity="0.5" />
+    <!-- from -9 to 9 degrees-->
+    <limit lower="-0.15" upper="0.15" effort="100" velocity="2.2" />
     <dynamics damping="0.2" friction="0" />
   </joint>
@@ -719,5 +735,6 @@
     <origin xyz="0 0 0" rpy="0 -0 0 "/>
     <axis   xyz="1 0 0"/>
-    <limit lower="-0.698132" upper="0.698132" effort="100" velocity="0.5" />
+    <!-- from -40 to 75 degrees-->
+    <limit lower="-0.698132" upper="1.309" effort="100" velocity="2.2" />
     <dynamics damping="0.2" friction="0" />
   </joint>

Commit message: fix wrong joint limit

File: aero_shop/typeF_upperbody/urdf/aero_upper_typef.urdf.xacro (robot description, xacro)
@@ -569,5 +569,5 @@
     <axis   xyz="1 0 0"/>
     <!-- from -75 to 40 degrees-->
-    <limit lower="-1.309" upper="-0.698132" effort="100" velocity="2.2" />
+    <limit lower="-1.309" upper="0.698132" effort="100" velocity="2.2" />
     <dynamics damping="0.2" friction="0" />
   </joint>
@@ -634,5 +634,5 @@
     <axis   xyz="0 0.984808 0.173648"/>
     <!-- from -15 to 88 degrees-->
-    <limit lower="-0.261" upper="-1.535" effort="100" velocity="2.2" />
+    <limit lower="-0.261" upper="1.535" effort="100" velocity="2.2" />
     <dynamics damping="0.2" friction="0" />
   </joint>

Commit message: loosen waist_yaw limit from +-90 to +-120

File: aero_shop/typeF_upperbody/urdf/aero_upper_typef.urdf.xacro (robot description, xacro)
@@ -416,5 +416,5 @@
     <axis   xyz="0 0 1"/>
     <!-- from -120 to 120 degrees-->
-    <limit lower="-1.5707" upper="1.5707" effort="100" velocity="0.9" />
+    <limit lower="-2.0" upper="2.0" effort="100" velocity="0.9" />
     <dynamics damping="0.2" friction="0" />
   </joint>

Commit message: fix r_shoulder_p_joint limit

File: aero_shop/typeF_upperbody/urdf/aero_upper_typef.urdf.xacro (robot description, xacro)
@@ -633,6 +633,6 @@
     <origin xyz="-0.01815 -0.1342 0.3049" rpy="0 -0 0 "/>
     <axis   xyz="0 0.984808 0.173648"/>
-    <!-- from -15 to 88 degrees-->
-    <limit lower="-0.261" upper="1.535" effort="100" velocity="2.2" />
+    <!-- from -88 to 15 degrees-->
+    <limit lower="-1.535" upper="0.261" effort="100" velocity="2.2" />
     <dynamics damping="0.2" friction="0" />
   </joint>
@@ -684,6 +684,6 @@
     <origin xyz="0.035 0 -0.1625" rpy="0 -0 0 "/>
     <axis   xyz="0 1 0"/>
-    <!-- from 0 to 140 degrees-->
-    <limit lower="0" upper="2.44246" effort="100" velocity="2.3" />
+    <!-- from -140 to 0 degrees-->
+    <limit lower="-2.44246" upper="0" effort="100" velocity="2.3" />
     <dynamics damping="0.2" friction="0" />
   </joint>

Commit message: update neck joint limits

File: aero_shop/typeF_upperbody/urdf/aero_upper_typef.urdf.xacro (robot description, xacro)
@@ -585,5 +585,5 @@
     <origin xyz="0 0 0.3535" rpy="0 -0 0 "/>
     <axis   xyz="0 0 1"/>
-    <limit lower="-1.5707" upper="1.5707" effort="100" velocity="0.5" />
+    <limit lower="-2.1" upper="2.1" effort="100" velocity="0.5" />
     <dynamics damping="0.2" friction="0" />
   </joint>

Commit message: fix waist_yaw speed

File: aero_shop/typeF_upperbody/urdf/aero_upper_typef.urdf.xacro (robot description, xacro)
@@ -416,5 +416,5 @@
     <axis   xyz="0 0 1"/>
     <!-- from -120 to 120 degrees-->
-    <limit lower="-2.0" upper="2.0" effort="100" velocity="0.9" />
+    <limit lower="-2.0" upper="2.0" effort="100" velocity="0.5" />
     <dynamics damping="0.2" friction="0" />
   </joint>
@@ -484,5 +484,5 @@
     <axis   xyz="1 0 0"/>
     <!-- from 0 to 90 degrees-->
-    <limit lower="0" upper="1.5707" effort="100" velocity="2.3" />
+    <limit lower="0" upper="1.5707" effort="100" velocity="1.5" />
     <dynamics damping="0.2" friction="0" />
   </joint>
@@ -651,5 +651,5 @@
     <axis   xyz="1 0 0"/>
     <!-- from -90 to 0 degrees-->
-    <limit lower="-1.5707" upper="0" effort="100" velocity="2.3" />
+    <limit lower="-1.5707" upper="0" effort="100" velocity="1.5" />
     <dynamics damping="0.2" friction="0" />
   </joint>

Commit message: [aero_shop, typeF_upperbody] add dummy collision objects for avoiding elbow collision

File: aero_shop/typeF_upperbody/urdf/aero_upper_typef.urdf.xacro (robot description, xacro)
@@ -130,4 +130,10 @@
         <mesh filename="package://aero_description/meshes/typeF_upperbody/LARM_LINK3_mesh.dae" scale="1 1 1" />
       </geometry>
+    </collision>
+    <collision>
+      <origin rpy="0 2.8415926535897931 0" xyz="0.015 0 -0.13"/>
+      <geometry>
+        <mesh filename="package://aero_description/meshes/typeF_upperbody/elbow_pad.dae" scale="1 1 1"/>
+      </geometry>
     </collision> </xacro:unless>
     <inertial>
@@ -153,4 +159,10 @@
         <mesh filename="package://aero_description/meshes/typeF_upperbody/LARM_LINK4_mesh.dae" scale="1 1 1" />
       </geometry>
+    </collision>
+    <collision>
+      <origin rpy="0 0 3.1415926535897931" xyz="-0.010 0 -0.035"/>
+      <geometry>
+        <mesh filename="package://aero_description/meshes/typeF_upperbody/elbow_pad.dae" scale="1 1 1"/>
+      </geometry>
     </collision> </xacro:unless>
     <inertial>
@@ -305,4 +317,10 @@
         <mesh filename="package://aero_description/meshes/typeF_upperbody/RARM_LINK3_mesh.dae" scale="1 1 1" />
       </geometry>
+    </collision>
+    <collision>
+      <origin rpy="0 2.8415926535897931 0" xyz="0.015 0 -0.13"/>
+      <geometry>
+        <mesh filename="package://aero_description/meshes/typeF_upperbody/elbow_pad.dae" scale="1 1 1"/>
+      </geometry>
     </collision> </xacro:unless>
     <inertial>
@@ -327,4 +345,10 @@
       <geometry>
         <mesh filename="package://aero_description/meshes/typeF_upperbody/RARM_LINK4_mesh.dae" scale="1 1 1" />
+      </geometry>
+    </collision>
+    <collision>
+      <origin rpy="0 0 3.1415926535897931" xyz="-0.010 0 -0.035"/>
+      <geometry>
+        <mesh filename="package://aero_description/meshes/typeF_upperbody/elbow_pad.dae" scale="1 1 1"/>
       </geometry>
     </collision> </xacro:unless>

Commit message: update csv and angle limit

File: aero_shop/typeF_upperbody/urdf/aero_upper_typef.urdf.xacro (robot description, xacro)
@@ -386,5 +386,5 @@
     <axis   xyz="0 0 1"/>
     <!-- from -120 to 120 degrees-->
-    <limit lower="-2.0" upper="2.0" effort="500" velocity="0.5" />
+    <limit lower="-2.09" upper="2.09" effort="500" velocity="0.5" />
     <dynamics damping="0.2" friction="0" />
   </joint>
@@ -395,6 +395,6 @@
     <origin xyz="0 0 0.1355" rpy="0 -0 0 "/>
     <axis   xyz="0 1 0"/>
-    <!-- from -5 to 30 degrees-->
-    <limit lower="-0.0872" upper="0.5235" effort="2000" velocity="0.3" />
+    <!-- from -5 to 35 degrees-->
+    <limit lower="-0.087" upper="0.61" effort="2000" velocity="0.3" />
     <dynamics damping="0.2" friction="0" />
   </joint>
@@ -446,5 +446,5 @@
     <axis   xyz="0 1 0"/>
     <!-- from -140 to 0 degrees-->
-    <limit lower="-2.44246" upper="0" effort="100" velocity="1.0" />
+    <limit lower="-2.44346" upper="0" effort="100" velocity="1.0" />
     <dynamics damping="0.2" friction="0" />
   </joint>
@@ -465,6 +465,6 @@
     <origin xyz="0 0 -0.1955" rpy="0 -0 0 "/>
     <axis   xyz="0 1 0"/>
-    <!-- from -9 to 9 degrees-->
-    <limit lower="-0.15" upper="0.15" effort="100" velocity="1.3" />
+    <!-- from -5 to 5 degrees-->
+    <limit lower="-0.087" upper="0.087" effort="100" velocity="1.3" />
     <dynamics damping="0.2" friction="0" />
   </joint>
@@ -475,6 +475,6 @@
     <origin xyz="0 0 0" rpy="0 -0 0 "/>
     <axis   xyz="1 0 0"/>
-    <!-- from -75 to 40 degrees-->
-    <limit lower="-1.309" upper="0.698132" effort="100" velocity="1.3" />
+    <!-- from -85 to 25 degrees-->
+    <limit lower="-1.484" upper="0.436" effort="100" velocity="1.3" />
     <dynamics damping="0.2" friction="0" />
   </joint>
@@ -485,5 +485,6 @@
     <origin xyz="0 0 0.3535" rpy="0 -0 0 "/>
     <axis   xyz="0 0 1"/>
-    <limit lower="-2.1" upper="2.1" effort="100" velocity="0.5" />
+    <!-- from -120 to 120 degrees-->
+    <limit lower="-2.09" upper="2.09" effort="100" velocity="0.5" />
     <dynamics damping="0.2" friction="0" />
   </joint>
@@ -494,5 +495,6 @@
     <origin xyz="0 0 0.1045" rpy="0 -0 0 "/>
     <axis   xyz="0 1 0"/>
-    <limit lower="0" upper="0.610864" effort="100" velocity="0.5" />
+    <!-- from -15 to 55 degrees-->
+    <limit lower="-0.262" upper="0.96" effort="100" velocity="0.5" />
     <dynamics damping="0.2" friction="0" />
   </joint>
@@ -503,5 +505,6 @@
     <origin xyz="0 0 0" rpy="0 -0 0 "/>
     <axis   xyz="1 0 0"/>
-    <limit lower="-0.122173" upper="0.122173" effort="100" velocity="0.5" />
+    <!-- from -5 to 5 degrees-->
+    <limit lower="-0.087" upper="0.087" effort="100" velocity="0.5" />
     <dynamics damping="0.2" friction="0" />
   </joint>
@@ -543,5 +546,5 @@
     <axis   xyz="0 1 0"/>
     <!-- from -140 to 0 degrees-->
-    <limit lower="-2.44246" upper="0" effort="100" velocity="1.0" />
+    <limit lower="-2.44346" upper="0" effort="100" velocity="1.0" />
     <dynamics damping="0.2" friction="0" />
   </joint>
@@ -562,6 +565,6 @@
     <origin xyz="0 0 -0.1955" rpy="0 -0 0 "/>
     <axis   xyz="0 1 0"/>
-    <!-- from -9 to 9 degrees-->
-    <limit lower="-0.15" upper="0.15" effort="100" velocity="1.3" />
+    <!-- from -5 to 5 degrees-->
+    <limit lower="-0.087" upper="0.087" effort="100" velocity="1.3" />
     <dynamics damping="0.2" friction="0" />
   </joint>
@@ -572,6 +575,6 @@
     <origin xyz="0 0 0" rpy="0 -0 0 "/>
     <axis   xyz="1 0 0"/>
-    <!-- from -40 to 75 degrees-->
-    <limit lower="-0.698132" upper="1.309" effort="100" velocity="1.3" />
+    <!-- from -25 to 85 degrees-->
+    <limit lower="-0.436" upper="1.484" effort="100" velocity="1.3" />
     <dynamics damping="0.2" friction="0" />
   </joint>

Commit message: Update aero_upper_typef.urdf.xacro
change elbow joint's limit from 2.44 to 3.0

File: aero_shop/typeF_upperbody/urdf/aero_upper_typef.urdf.xacro (robot description, xacro)
@@ -445,6 +445,6 @@
     <origin xyz="0.035 0 -0.1625" rpy="0 -0 0 "/>
     <axis   xyz="0 1 0"/>
-    <!-- from -140 to 0 degrees-->
-    <limit lower="-2.44346" upper="0" effort="100" velocity="1.0" />
+    <!-- from -171 to 0 degrees-->
+    <limit lower="-3.0" upper="0" effort="100" velocity="1.0" />
     <dynamics damping="0.2" friction="0" />
   </joint>
@@ -545,6 +545,6 @@
     <origin xyz="0.035 0 -0.1625" rpy="0 -0 0 "/>
     <axis   xyz="0 1 0"/>
-    <!-- from -140 to 0 degrees-->
-    <limit lower="-2.44346" upper="0" effort="100" velocity="1.0" />
+    <!-- from -171 to 0 degrees-->
+    <limit lower="-3.0" upper="0" effort="100" velocity="1.0" />
     <dynamics damping="0.2" friction="0" />
   </joint>

Commit message: updat velocity of each joints

File: aero_shop/typeF_upperbody/urdf/aero_upper_typef.urdf.xacro (robot description, xacro)
@@ -386,5 +386,5 @@
     <axis   xyz="0 0 1"/>
     <!-- from -120 to 120 degrees-->
-    <limit lower="-2.09" upper="2.09" effort="500" velocity="0.5" />
+    <limit lower="-2.09" upper="2.09" effort="500" velocity="0.6" />
     <dynamics damping="0.2" friction="0" />
   </joint>
@@ -396,5 +396,5 @@
     <axis   xyz="0 1 0"/>
     <!-- from -5 to 35 degrees-->
-    <limit lower="-0.087" upper="0.61" effort="2000" velocity="0.3" />
+    <limit lower="-0.087" upper="0.61" effort="2000" velocity="0.5" />
     <dynamics damping="0.2" friction="0" />
   </joint>
@@ -406,5 +406,5 @@
     <axis   xyz="1 0 0"/>
     <!-- from -1 to 1 degrees-->
-    <limit lower="-0.017" upper="0.017" effort="2000" velocity="0.3" />
+    <limit lower="-0.017" upper="0.017" effort="2000" velocity="0.4" />
     <dynamics damping="0.2" friction="0" />
   </joint>
@@ -416,5 +416,5 @@
     <axis   xyz="0 0.984808 -0.173648"/>
     <!-- from -88 to 15 degrees-->
-    <limit lower="-1.535" upper="0.261" effort="200" velocity="0.5" />
+    <limit lower="-1.535" upper="0.261" effort="200" velocity="0.4" />
     <dynamics damping="0.2" friction="0" />
   </joint>
@@ -436,5 +436,5 @@
     <axis   xyz="0 0 1"/>
     <!-- from -180 to 45 degrees-->
-    <limit lower="-1.5707" upper="0.785398" effort="100" velocity="0.5" />
+    <limit lower="-1.5707" upper="0.785398" effort="100" velocity="1.2" />
     <dynamics damping="0.2" friction="0" />
   </joint>
@@ -446,5 +446,5 @@
     <axis   xyz="0 1 0"/>
     <!-- from -171 to 0 degrees-->
-    <limit lower="-3.0" upper="0" effort="100" velocity="1.0" />
+    <limit lower="-3.0" upper="0" effort="100" velocity="1.2" />
     <dynamics damping="0.2" friction="0" />
   </joint>
@@ -456,5 +456,5 @@
     <axis   xyz="0 0 1"/>
     <!-- from -180 to 180 degrees-->
-    <limit lower="-1.5707" upper="1.5707" effort="100" velocity="1.5" />
+    <limit lower="-1.5707" upper="1.5707" effort="100" velocity="1.3" />
     <dynamics damping="0.2" friction="0" />
   </joint>
@@ -466,5 +466,5 @@
     <axis   xyz="0 1 0"/>
     <!-- from -5 to 5 degrees-->
-    <limit lower="-0.087" upper="0.087" effort="100" velocity="1.3" />
+    <limit lower="-0.087" upper="0.087" effort="100" velocity="0.9" />
     <dynamics damping="0.2" friction="0" />
   </joint>
@@ -476,5 +476,5 @@
     <axis   xyz="1 0 0"/>
     <!-- from -85 to 25 degrees-->
-    <limit lower="-1.484" upper="0.436" effort="100" velocity="1.3" />
+    <limit lower="-1.484" upper="0.436" effort="100" velocity="2.1" />
     <dynamics damping="0.2" friction="0" />
   </joint>
@@ -486,5 +486,5 @@
     <axis   xyz="0 0 1"/>
     <!-- from -120 to 120 degrees-->
-    <limit lower="-2.09" upper="2.09" effort="100" velocity="0.5" />
+    <limit lower="-2.09" upper="2.09" effort="100" velocity="1.6" />
     <dynamics damping="0.2" friction="0" />
   </joint>
@@ -496,5 +496,5 @@
     <axis   xyz="0 1 0"/>
     <!-- from -15 to 55 degrees-->
-    <limit lower="-0.262" upper="0.96" effort="100" velocity="0.5" />
+    <limit lower="-0.262" upper="0.96" effort="100" velocity="2.1" />
     <dynamics damping="0.2" friction="0" />
   </joint>
@@ -506,5 +506,5 @@
     <axis   xyz="1 0 0"/>
     <!-- from -5 to 5 degrees-->
-    <limit lower="-0.087" upper="0.087" effort="100" velocity="0.5" />
+    <limit lower="-0.087" upper="0.087" effort="100" velocity="0.9" />
     <dynamics damping="0.2" friction="0" />
   </joint>
@@ -516,5 +516,5 @@
     <axis   xyz="0 0.984808 0.173648"/>
     <!-- from -88 to 15 degrees-->
-    <limit lower="-1.535" upper="0.261" effort="200" velocity="0.5" />
+    <limit lower="-1.535" upper="0.261" effort="200" velocity="0.4" />
     <dynamics damping="0.2" friction="0" />
   </joint>
@@ -536,5 +536,5 @@
     <axis   xyz="0 0 1"/>
     <!-- from -45 to 180 degrees-->
-    <limit lower="-0.785398" upper="1.5707" effort="100" velocity="0.5" />
+    <limit lower="-0.785398" upper="1.5707" effort="100" velocity="1.2" />
     <dynamics damping="0.2" friction="0" />
   </joint>
@@ -546,5 +546,5 @@
     <axis   xyz="0 1 0"/>
     <!-- from -171 to 0 degrees-->
-    <limit lower="-3.0" upper="0" effort="100" velocity="1.0" />
+    <limit lower="-3.0" upper="0" effort="100" velocity="1.2" />
     <dynamics damping="0.2" friction="0" />
   </joint>
@@ -556,5 +556,5 @@
     <axis   xyz="0 0 1"/>
     <!-- from -180 to 180 degrees-->
-    <limit lower="-1.5707" upper="1.5707" effort="100" velocity="1.5" />
+    <limit lower="-1.5707" upper="1.5707" effort="100" velocity="1.3" />
     <dynamics damping="0.2" friction="0" />
   </joint>
@@ -566,5 +566,5 @@
     <axis   xyz="0 1 0"/>
     <!-- from -5 to 5 degrees-->
-    <limit lower="-0.087" upper="0.087" effort="100" velocity="1.3" />
+    <limit lower="-0.087" upper="0.087" effort="100" velocity="0.9" />
     <dynamics damping="0.2" friction="0" />
   </joint>
@@ -576,5 +576,5 @@
     <axis   xyz="1 0 0"/>
     <!-- from -25 to 85 degrees-->
-    <limit lower="-0.436" upper="1.484" effort="100" velocity="1.3" />
+    <limit lower="-0.436" upper="1.484" effort="100" velocity="2.1" />
     <dynamics damping="0.2" friction="0" />
   </joint>
