Commit message: [aero_robot_jsk] fix urdf for using in gazebo, there is no effect to real robot

File: aero_shop/hand_yaw/urdf/hand_yaw.urdf.xacro (robot description, xacro)
@@ -26,6 +26,10 @@
     <inertial>
       <mass value="0.183" />
-      <origin xyz="0 0 -0.0875" rpy="0 -0 0"/>
-      <inertia ixx="0.000601" ixy="0" ixz="0" iyy="0.00055" iyz="0" izz="0.000102"/>
+      <!-- original version -->
+      <!--origin xyz="0 0 -0.0875" rpy="0 -0 0"/>
+      <inertia ixx="0.000601" ixy="0" ixz="0" iyy="0.00055" iyz="0" izz="0.000102"/-->
+      <!-- just fixed for gazebo / aim to increase z axis inertia-->
+      <origin xyz="0 0.014 -0.02" rpy="0 -0 0"/>
+      <inertia ixx="0.000601" ixy="0" ixz="0" iyy="0.00055" iyz="0" izz="0.0014" />
     </inertial>
   </link>
@@ -42,7 +46,5 @@
     <dynamics damping="0.2" friction="0" />
   </joint>
-  <gazebo reference="${prefix}_hand_yaw_joint">
-    <implicitSpringDamper>0.4</implicitSpringDamper>
-  </gazebo>
+  <xacro:gazebo_transmission joint_name="${prefix}_hand_y_joint" />
   </xacro:macro>
 </robot>

Commit message: [aero_robot_jsk] fix minor

File: aero_shop/hand_yaw/urdf/hand_yaw.urdf.xacro (robot description, xacro)
@@ -7,6 +7,6 @@
   <xacro:include filename="$(find aero_description)/urdf/common.xacro" />
   <property name="M_PI" value="3.1415926535897931" />
+  <xacro:macro name="hand_yaw" params="prefix:=r reflect:=1 hand_link disable_mesh:=false">
   <!-- ============================   hand_yaw   ============================ -->
-  <xacro:macro name="hand_yaw" params="prefix:=r reflect:=1 hand_link disable_mesh:=false">
     <!-- prefix is "r" or "l" -->
     <!-- reflect=1 is rightside, reflect=-1 is leftside -->

Commit message: [aero_shop] fix inertia for gazebo

File: aero_shop/hand_yaw/urdf/hand_yaw.urdf.xacro (robot description, xacro)
@@ -31,5 +31,5 @@
       <!-- just fixed for gazebo / aim to increase z axis inertia-->
       <origin xyz="0 0.014 -0.02" rpy="0 -0 0"/>
-      <inertia ixx="0.003" ixy="0" ixz="0" iyy="0.003" iyz="0" izz="0.005" />
+      <inertia ixx="0.0005" ixy="0" ixz="0" iyy="0.0005" iyz="0" izz="0.0007" />
     </inertial>
   </link>

File: aero_shop/typeF_upperbody/urdf/aero_upper_typef.urdf.xacro (robot description, xacro)
@@ -46,5 +46,7 @@
       <mass value="1.257" />
       <origin xyz="0 0 0.042" rpy="0 -0 0"/>
-      <inertia ixx="0.034" ixy="0" ixz="0" iyy="0.034" iyz="0" izz="0.018"/>
+      <!-- inertia ixx="0.034" ixy="0" ixz="0" iyy="0.034" iyz="0" izz="0.018"/ -->
+      <!-- just fixed for gazebo / reduce inertia-->
+      <inertia ixx="0.01" ixy="0" ixz="0" iyy="0.01" iyz="0" izz="0.007"/>
     </inertial>
   </link>
@@ -54,5 +56,7 @@
       <mass value="0.1" />
       <origin xyz="0 0 0" rpy="0 -0 0"/>
-      <inertia ixx="0.01" ixy="0" ixz="0" iyy="0.01" iyz="0" izz="0.01"/>
+      <!--inertia ixx="0.01" ixy="0" ixz="0" iyy="0.01" iyz="0" izz="0.01"/-->
+      <!-- just fixed for gazebo / reduce inertia-->
+      <inertia ixx="0.003" ixy="0" ixz="0" iyy="0.003" iyz="0" izz="0.003"/>
     </inertial>
   </link>
@@ -93,6 +97,9 @@
     <inertial>
       <mass value="0.242" />
-      <origin xyz="0 0.02 0" rpy="0 -0 0"/>
-      <inertia ixx="0.000228" ixy="0" ixz="0" iyy="0.000148" iyz="0" izz="0.000263"/>
+      <!--origin xyz="0 0.02 0" rpy="0 -0 0"/>
+      <inertia ixx="0.000228" ixy="0" ixz="0" iyy="0.000148" iyz="0" izz="0.000263"/-->
+      <!-- just fixed for gazebo / increase inertia-->
+      <origin xyz="0 0.02 0.015" rpy="0 -0 0"/>
+      <inertia ixx="0.00133" ixy="0" ixz="0" iyy="0.001" iyz="0" izz="0.00133"/>
     </inertial>
   </link>
@@ -113,5 +120,6 @@
     <inertial>
       <mass value="0.744" />
-      <origin xyz="0 0.01 0" rpy="0 -0 0"/>
+      <!--origin xyz="0 0.01 0" rpy="0 -0 0"/-->
+      <origin xyz="0 -0.01 -0.06" rpy="0 -0 0"/>
       <inertia ixx="0.000841" ixy="0" ixz="0" iyy="0.000835" iyz="0" izz="0.000304"/>
     </inertial>
@@ -180,5 +188,6 @@
       <mass value="0.132" />
       <origin xyz="0.006 0 -0.0738" rpy="0 -0 0"/>
-      <inertia ixx="0.00276" ixy="0" ixz="0" iyy="0.00286" iyz="0" izz="0.004"/>
+      <!--inertia ixx="0.00276" ixy="0" ixz="0" iyy="0.00286" iyz="0" izz="0.004"/-->
+      <inertia ixx="0.0007" ixy="0" ixz="0" iyy="0.0007" iyz="0" izz="0.0004"/>
     </inertial>
   </link>
@@ -268,6 +277,8 @@
     <inertial>
       <mass value="0.242" />
-      <origin xyz="0 -0.02 0" rpy="0 -0 0"/>
-      <inertia ixx="0.000228" ixy="0" ixz="0" iyy="0.000148" iyz="0" izz="0.000263"/>
+      <!--origin xyz="0 -0.02 0" rpy="0 -0 0"/>
+      <inertia ixx="0.000228" ixy="0" ixz="0" iyy="0.000148" iyz="0" izz="0.000263"/-->
+      <origin xyz="0 -0.02 0.015" rpy="0 -0 0"/>
+      <inertia ixx="0.00133" ixy="0" ixz="0" iyy="0.001" iyz="0" izz="0.00133"/>
     </inertial>
   </link>
@@ -288,5 +299,6 @@
     <inertial>
       <mass value="0.744" />
-      <origin xyz="0 -0.01 0" rpy="0 -0 0"/>
+      <!--origin xyz="0 -0.01 0" rpy="0 -0 0"/-->
+      <origin xyz="0 0.01 -0.06" rpy="0 -0 0"/>
       <inertia ixx="0.000841" ixy="0" ixz="0" iyy="0.000835" iyz="0" izz="0.000305"/>
     </inertial>
@@ -355,5 +367,6 @@
       <mass value="0.132" />
       <origin xyz="0.006 0 -0.0738" rpy="0 -0 0"/>
-      <inertia ixx="0.00276" ixy="0" ixz="0" iyy="0.00286" iyz="0" izz="0.004"/>
+      <!--inertia ixx="0.00276" ixy="0" ixz="0" iyy="0.00286" iyz="0" izz="0.004"/-->
+      <inertia ixx="0.0007" ixy="0" ixz="0" iyy="0.0007" iyz="0" izz="0.0004"/>
     </inertial>
   </link>
@@ -403,5 +416,5 @@
     <axis   xyz="0 0.984808 -0.173648"/>
     <!-- from -88 to 15 degrees-->
-    <limit lower="-1.535" upper="0.261" effort="100" velocity="0.5" />
+    <limit lower="-1.535" upper="0.261" effort="200" velocity="0.5" />
     <dynamics damping="0.2" friction="0" />
   </joint>
@@ -500,5 +513,5 @@
     <axis   xyz="0 0.984808 0.173648"/>
     <!-- from -88 to 15 degrees-->
-    <limit lower="-1.535" upper="0.261" effort="100" velocity="0.5" />
+    <limit lower="-1.535" upper="0.261" effort="200" velocity="0.5" />
     <dynamics damping="0.2" friction="0" />
   </joint>

Commit message: fix hand yaw limits

File: aero_shop/hand_yaw/urdf/hand_yaw.urdf.xacro (robot description, xacro)
@@ -43,5 +43,5 @@
     <origin xyz="0 0 -0.04" rpy="0 0 0"/>
     <axis   xyz="0 0 1"/>
-    <limit lower="-2.0" upper="2.0" effort="100" velocity="3.1" />
+    <limit lower="-3.2" upper="3.2" effort="100" velocity="3.1" />
     <dynamics damping="0.2" friction="0" />
   </joint>
